File: FuseBox/USB_SPI.kicad_sch (KiCad schematic)
At the start: 1 part, among them U5 FT2232HPQTRAY

Commit message: changes
Parts:
- added C47, C48, C49, C50, C51, C54, C56: 100n, symbol Device:C
- added C52, C53: 20p, symbol Device:C
- added C55: 10u, symbol Device:C
- added R25, R40: 2k2, symbol Device:R
- added R26: 12k, symbol Device:R
- added R27, R28, R29, R30, R31, R32, R33, R34, R35, R36, R37, R38, R39: 0, symbol Device:R
- added R41, R42, R43: 10k, symbol Device:R
- added U6: 93LC56CIMS, Custom:93LC56CIMS, symbol Custom:93LC56CIMS
- added X2: STDCSU212M, Custom:STDCSU212M, symbol Custom:STDCSU212M
Connections:
- net at U5.1 (EECLK): now also R42.1, U6.2 (CLK)
- net +3V3: now reaches U5.10 (VCCIO)
- net +3V3: now also U5.26 (VCCIO), U5.30 (VREGIN), U5.39 (VCCIO), U5.51 (VCCIO), C47.1, C48.1, C49.1, C50.1, C51.1, C56.2, R25.1, R41.2, R42.2, R43.2, U6.6 (ORG), U6.8 (VCC)
- net at U5.11 (ADBUS2): now also R29.1
- net at U5.13 (ADBUS4): now also R30.1
- net at U5.15 (ADBUS6): now also R31.1
- net at U5.16 (ADBUS7): now also R32.1
- net at U5.2 (EEDATA): now also R40.2, R41.1, U6.3 (DI)
- net VCCFT_1V8: now reaches U5.25 (VCORE)
- net VCCFT_1V8: now also U5.31 (VREGOUT), U5.44 (VCORE), U5.66 (VCORE), U5.8 (VCORE), C54.1, C55.1
- net at U5.27 (OSCI): now also C52.2, X2.1
- net at U5.28 (OSCO): now also C53.2, X2.2
- net GND: now reaches U5.29 (GND)
- net GND: now also U5.3 (TEST), U5.9 (GND), C47.2, C48.2, C49.2, C50.2, C51.2, C52.1, C53.1, C54.2, C55.2, C56.1, R26.1, U6.5 (VSS)
- net at U5.34 (BDBUS0): now also R33.1
- net at U5.35 (BDBUS1): now also R34.1
- net at U5.36 (BDBUS2): now also R35.1
- net at U5.37 (BDBUS3): now also R36.1
- net at U5.38 (BDBUS4): now also R37.1
- net at U5.4 (RESET#): now also R25.2
- net at U5.40 (BDBUS5): now also R38.1
- net at U5.41 (BDBUS6): now also R39.1
- net at U5.6 (ADBUS0): now also R27.1
- net at U5.60 (REF): now also R26.2
- net at U5.68 (EECS): now also R43.1, U6.1 (CS)
- net at U5.7 (ADBUS1): now also R28.1
- new net: R40.1, U6.4 (DO)
- new net CTSn: R36.2
- new net DCDn: R39.2
- new net DSRn: R38.2
- new net DTRn: R37.2
- new net FPGA_CDONE: R31.2
- new net FPGA_CREST: R32.2
- new net FPGA_SCK: R27.2
- new net FPGA_SPI_MISO: R29.2
- new net FPGA_SPI_MOSI: R28.2
- new net FPGA_SS: R30.2
- new net RS232_RX_TTL: R33.2
- new net RS232_TX_TTL: R34.2
- new net RTSn: R35.2
- no-connect marks 0 -> 22
Other:
- moved on the sheet: U5

Commit message: some foo
Connections:
- net at R40.2, U5.2 (EEDATA), U6.3 (DI): no longer R41.1
- net at R40.1, U6.4 (DO): now also R41.1
Changed lines of the file:
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@@
+	)
+	(junction
+		(at 62.23 93.98)
+		(diameter 0)
+		(color 0 0 0 0)
 	)
 	(junction
@@
 	)
 	(junction
-		(at 62.23 91.44)
-		(diameter 0)
-		(color 0 0 0 0)
-	)
-	(junction
 		(at 231.14 33.02)
 		(diameter 0)
@@
 	)
 	(no_connect
-		(at 22.86 88.9)
+		(at 27.94 88.9)
 	)
 	(no_connect
@@
 	(wire
 		(pts
-			(xy 60.96 91.44) (xy 62.23 91.44)
+			(xy 60.96 91.44) (xy 96.52 91.44)
 		)
 		(stroke
@@
 	(wire
 		(pts
-			(xy 62.23 91.44) (xy 62.23 102.87)
-		)
-		(stroke
-			(width 0)
-			(type default)
-		)
-	)
-	(wire
-		(pts
 			(xy 231.14 33.02) (xy 243.84 33.02)
 		)
@@
 	(wire
 		(pts
+			(xy 62.23 93.98) (xy 82.55 93.98)
+		)
+		(stroke
+			(width 0)
+			(type default)
+		)
+	)
+	(wire
+		(pts
 			(xy 76.2 66.04) (xy 87.63 66.04)
 		)
@@
 	(wire
 		(pts
-			(xy 22.86 88.9) (xy 27.94 88.9)
-		)
-		(stroke
-			(width 0)
-			(type default)
-		)
-	)
-	(wire
-		(pts
 			(xy 19.05 110.49) (xy 27.94 110.49)
 		)
@@
 	(wire
 		(pts
-			(xy 62.23 91.44) (xy 96.52 91.44)
-		)
-		(stroke
-			(width 0)
-			(type default)
-		)
-	)
-	(wire
-		(pts
 			(xy 139.7 33.02) (xy 139.7 38.1)
 		)
@@
 	(wire
 		(pts
+			(xy 62.23 93.98) (xy 62.23 102.87)
+		)
+		(stroke
+			(width 0)
+			(type default)
+		)
+	)
+	(wire
+		(pts
 			(xy 92.71 44.45) (xy 92.71 48.26)
 		)
@@
 	(wire
 		(pts
-			(xy 60.96 93.98) (xy 82.55 93.98)
+			(xy 60.96 93.98) (xy 62.23 93.98)
 		)
 		(stroke
@@
 		(on_board yes)
 		(dnp no)
-		(fields_autoplaced yes)
 		(property "Reference" "C56"
-			(at 22.86 100.3299 0)
+			(at 22.098 100.33 0)
 			(effects
 				(font
@@
 		)
 		(property "Value" "100n"
-			(at 22.86 102.8699 0)
-			(effects
-				(font
+			(at 22.098 102.87 0)
+			(effects
+				(font
