File: FuseBox/ICE40HX.kicad_sch (KiCad schematic)
At the start: 59 parts, among them J10 901301150, J11 901301150, J6 901301150, J8 61301611121, J9 901301150, U4 ICE40HX8KCT256

Commit message: finished schematic
Parts:
- C16, C17, C18, C19, C20, C21, C22, C23, C24, C25, C26, C27, C28, C29, C30, C31, C32, C33, C34, C35, C36, C37, C38, C39, C40, C41, C42, C43, C44, C45, C46: footprint (none) -> Capacitor_SMD:C_0603_1608Metric_Pad1.08x0.95mm_HandSolder
- R18, R19, R20, R21, R22, R23, R24, R25, R26: footprint (none) -> Resistor_SMD:R_0603_1608Metric_Pad0.98x0.95mm_HandSolder
Connections:
- net at U4.B16 (IOR_165): now also J9.48; no longer J9.44
- net at U4.C16 (IOR_161): now also J9.46; no longer J9.42
- net at U4.D14 (IOR_167): now also J9.50; no longer J9.46
- net at U4.D15 (IOR_157): now also J9.43; no longer J9.39
- net at U4.D16 (IOR_153): now also J9.39; no longer J9.35
- net at U4.E13 (IOR_166): now also J9.49; no longer J9.45
- net at U4.E14 (IOR_160): now also J9.45; no longer J9.41
- net at U4.E16 (IOR_151): now also J9.37; no longer J9.33
- net at U4.F11 (IOR_158): now also J9.44; no longer J9.40
- net at U4.F12 (IOR_156): now also J9.42; no longer J9.38
- net at U4.F13 (IOR_162): now also J9.47; no longer J9.43
- net at U4.F14 (IOR_155): now also J9.41; no longer J9.37
- net at U4.F15 (IOR_149): now also J9.35; no longer J9.31
- net at U4.F16 (IOR_147): now also J9.33; no longer J9.29
- net at U4.G10 (IOR_146): now also J9.32; no longer J9.28
- net at U4.G11 (IOR_148): now also J9.34; no longer J9.30
- net at U4.G12 (IOR_154): now also J9.40; no longer J9.36
- net at U4.G13 (IOR_152): now also J9.38; no longer J9.34
- net at U4.G14 (IOR_150): now also J9.36; no longer J9.32
- net at U4.G15 (IOR_145): now also J9.31; no longer J9.27
- net at U4.G16 (IOR_143): now also J9.29; no longer J9.25
- net at U4.H12 (IOR_144): now also J9.30; no longer J9.26
- net at U4.H13 (IOR_139): now also J9.27; no longer J9.23
- net at U4.H14 (IOR_142): now also J9.28; no longer J9.24
- net at U4.J10 (IOR_122): now also J9.14; no longer J9.10
- net at U4.J11 (IOR_126): now also J9.16; no longer J9.12
- net at U4.J12 (IOR_136): now also J9.24; no longer J9.20
- net at U4.J13 (IOR_137): now also J9.25; no longer J9.21
- net at U4.J14 (IOR_134): now also J9.23; no longer J9.19
- net at U4.J15 (IOR_130): now also J9.20; no longer J9.16
- net at U4.J16 (IOR_138): now also J9.26; no longer J9.22
- net at U4.K12 (IOR_120): now also J9.12; no longer J9.8
- net at U4.K13 (IOR_128): now also J9.18; no longer J9.14
- net at U4.K14 (IOR_129): now also J9.19; no longer J9.15
- net at U4.K15 (IOR_131): now also J9.21; no longer J9.17
- net at U4.K16 (IOR_133): now also J9.22; no longer J9.18
- net at U4.L12 (IOR_116): now also J9.8; no longer J9.4
- net at U4.L13 (IOR_118): now also J9.10; no longer J9.6
- net at U4.L14 (IOR_119): now also J9.11; no longer J9.7
- net at U4.L16 (IOR_127): now also J9.17; no longer J9.13
- net at U4.M13 (IOR_114): now also J9.6; no longer J9.2
- net at U4.M14 (IOR_115): now also J9.7; no longer J9.3
- net at U4.M15 (IOR_123): now also J9.15; no longer J9.11
- net at U4.M16 (IOR_121): now also J9.13; no longer J9.9
- net at U4.N16 (IOR_117): now also J9.9; no longer J9.5
- net at U4.P14 (IOR_111): now also J9.3
- net at U4.P16 (IOR_113): now also J9.5; no longer J9.1
- net at U4.R14 (IOR_109): now also J9.1
- net ICE_B1_110: no longer names the net of U4.R15 (IOR_110)
- net ICE_B1_110: now also J9.2
- net ICE_B1_112: no longer names the net of U4.P15 (IOR_112)
- net ICE_B1_112: now also J9.4
- no-connect marks 20 -> 16

Commit message: changes
Parts:
- D6: value D -> CDSU4148; footprint (none) -> Diode_SMD:D_0603_1608Metric_Pad1.05x0.95mm_HandSolder
- TP12, TP13, TP14, TP15, TP16, TP17, TP18, TP19, TP20, TP21, TP22, TP23: footprint (none) -> TestPoint:TestPoint_Pad_D3.0mm
Connections:
- no-connect marks 16 -> 26
Changed lines of the file:
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@@
 	)
 	(no_connect
+		(at 237.49 101.6)
+	)
+	(no_connect
+		(at 46.99 158.75)
+	)
+	(no_connect
 		(at 289.56 158.75)
 	)
@@
 	)
 	(no_connect
+		(at 46.99 156.21)
+	)
+	(no_connect
 		(at 260.35 208.28)
 	)
 	(no_connect
+		(at 237.49 135.89)
+	)
+	(no_connect
+		(at 237.49 138.43)
+	)
+	(no_connect
+		(at 327.66 158.75)
+	)
+	(no_connect
+		(at 327.66 156.21)
+	)
+	(no_connect
 		(at 289.56 148.59)
 	)
 	(no_connect
+		(at 142.24 156.21)
+	)
+	(no_connect
 		(at 260.35 215.9)
 	)
 	(no_connect
+		(at 237.49 99.06)
+	)
+	(no_connect
+		(at 142.24 158.75)
+	)
+	(no_connect
 		(at 289.56 151.13)
 	)
@@
 			)
 		)
-		(property "Footprint" ""
+		(property "Footprint" "TestPoint:TestPoint_Pad_D3.0mm"
 			(at 62.23 212.09 0)
 			(effects
@@
 			)
 		)
-		(property "Footprint" ""
+		(property "Footprint" "TestPoint:TestPoint_Pad_D3.0mm"
 			(at 33.02 91.44 0)
 			(effects
@@
 			)
 		)
-		(property "Footprint" ""
+		(property "Footprint" "TestPoint:TestPoint_Pad_D3.0mm"
 			(at 223.52 91.44 0)
 			(effects
@@
 			)
 		)
-		(property "Footprint" ""
+		(property "Footprint" "TestPoint:TestPoint_Pad_D3.0mm"
 			(at 153.67 212.09 0)
 			(effects
@@
 			)
 		)
-		(property "Footprint" ""
+		(property "Footprint" "TestPoint:TestPoint_Pad_D3.0mm"
 			(at 33.02 73.66 0)
 			(effects
@@
 			)
 		)
-		(property "Value" "D"
+		(property "Value" "CDSU4148"
 			(at 367.03 191.008 0)
 			(effects
@@
 			)
 		)
-		(property "Footprint" ""
+		(property "Footprint" "Diode_SMD:D_0603_1608Metric_Pad1.05x0.95mm_HandSolder"
 			(at 367.03 187.96 0)
 			(effects
@@
 			)
 		)
-		(property "Footprint" ""
+		(property "Footprint" "TestPoint:TestPoint_Pad_D3.0mm"
 			(at 44.45 212.09 0)
 			(effects
@@
 			)
 		)
-		(property "Footprint" ""
+		(property "Footprint" "TestPoint:TestPoint_Pad_D3.0mm"
 			(at 223.52 73.66 0)
 			(effects
@@
 			)
 		)
-		(property "Footprint" ""
+		(property "Footprint" "TestPoint:TestPoint_Pad_D3.0mm"
 			(at 135.89 212.09 0)
 			(effects
@@
 			)
 		)
-		(property "Footprint" ""
+		(property "Footprint" "TestPoint:TestPoint_Pad_D3.0mm"
 			(at 62.23 251.46 0)
 			(effects
@@
 			)
 		)
-		(property "Footprint" ""
+		(property "Footprint" "TestPoint:TestPoint_Pad_D3.0mm"
 			(at 44.45 251.46 0)
 			(effects
@@
 			)
 		)
-		(property "Footprint" ""
+		(property "Footprint" "TestPoint:TestPoint_Pad_D3.0mm"
 			(at 135.89 251.46 0)
 			(effects
@@
 			)
 		)
-		(property "Footprint" ""
+		(property "Footprint" "TestPoint:TestPoint_Pad_D3.0mm"
 			(at 153.67 251.46 0)
 			(effects

Commit message: fpga decoupling
Parts:
- removed TP12, TP13, TP16, TP17, TP18, TP19, TP20, TP21: TestPoint, TestPoint:TestPoint_Pad_D3.0mm, symbol Connector:TestPoint
Connections:
- net at U4.L10 (IOB_85): no longer J10.29
- net at U4.L11 (IOB_99): no longer J10.39
- net at U4.L9 (IOB_74): no longer J10.20
- net at U4.M11 (IOB_93): no longer J10.36
- net at U4.M12 (IOB_101): no longer J10.41
- net at U4.M7 (IOB_64): no longer J10.12
- net at U4.M8 (IOB_68): no longer J10.15
- net at U4.M9 (IOB_80): no longer J10.26
- net at U4.N10 (IOB_87): no longer J10.31
- net at U4.N12 (IOB_98): no longer J10.38
- net at U4.N5 (IOB_56): no longer J10.5
- net at U4.N6 (IOB_52): no longer J10.1
- net at U4.N7 (IOB_66): no longer J10.13
- net at U4.N9 (IOB_78): no longer J10.24
- net at U4.P10 (IOB_86): no longer J10.30
- net at U4.P4 (IOB_54): no longer J10.3
- net at U4.P5 (IOB_58): no longer J10.7
- net at U4.P6 (IOB_67): no longer J10.14
- net at U4.P7 (IOB_77): no longer J10.23
- net at U4.P8 (IOB_72): no longer J10.18
- net at U4.P9 (IOB_83): no longer J10.27
- net at U4.R10 (IOB_84): no longer J10.28
- net at U4.R16 (IOB_102): no longer J10.42
- net at U4.R2 (IOB_55): no longer J10.4
- net at U4.R3 (IOB_59): no longer J10.8
- net at U4.R4 (IOB_63): no longer J10.11
- net at U4.R5 (IOB_60): no longer J10.9
- net at U4.R6 (IOB_71): no longer J10.17
- net at U4.T1 (IOB_53): no longer J10.2
- net ICE_B2_88: now reaches U4.T10 (IOB_88)
- net ICE_B2_88: now also J10.27; no longer J10.32
- net at J10.33: no longer U4.T11 (IOB_89)
- net at J10.37: no longer U4.T13 (IOB_94)
- net at J10.35: no longer U4.T14 (IOB_92)
- net ICE_B2_100: now reaches J10.34
- net ICE_B2_100: now also U4.T16 (IOB_100); no longer U4.T15 (IOB_91)
- net at J10.40: no longer U4.T16 (IOB_100)
- net at U4.T2 (IOB_57): no longer J10.6
- net at U4.T3 (IOB_61): no longer J10.10
- net at U4.T5 (IOB_69): no longer J10.16
- net at U4.T6 (IOB_73): no longer J10.19
- net at U4.T7 (IOB_75): no longer J10.21
- net at J10.22: no longer U4.T8 (IOB_76)
- net ICE_B2_76: now reaches J10.25
- net ICE_B2_76: now also U4.T8 (IOB_76); no longer U4.T9 (IOB_79)
- new net ICE_B2_79: J10.28, U4.T9 (IOB_79)
- new net ICE_B2_89: J10.30, U4.T11 (IOB_89)
- new net ICE_B2_91: J10.31, U4.T15 (IOB_91)
- new net ICE_B2_92: J10.32, U4.T14 (IOB_92)
- new net ICE_B2_94: J10.29, U4.T13 (IOB_94)
Other:
- moved on the sheet: J10
