File: FuseBox/ICE40HX.kicad_sch (KiCad schematic)
At the start: 51 parts, among them J10 901301150, J11 901301150, J6 901301150, J8 61301611121, J9 901301150, U4 ICE40HX8KCT256

Commit message: bank 2 done
Connections:
- net ICE_B2_100: now also J10.32; no longer J10.34
- net ICE_B2_79: now also J10.26; no longer J10.28
- net ICE_B2_89: now also J10.28; no longer J10.30
- net ICE_B2_92: now also J10.30; no longer J10.32
- net at J11.1: no longer U4.E4 (IOL_1A)
- net at J11.10: no longer U4.D1 (IOL_5B)
- net at J11.11: no longer U4.G4 (IOL_6A)
- net at J11.12: no longer U4.E3 (IOL_6B)
- net at J11.13: no longer U4.H5 (IOL_7A)
- net at J11.14: no longer U4.E2 (IOL_7B)
- net at J11.15: no longer U4.G3 (IOL_8A)
- net at J11.16: no longer U4.F3 (IOL_8B)
- net at J11.17: no longer U4.H3 (IOL_9A)
- net at J11.18: no longer U4.F2 (IOL_9B)
- net at J11.19: no longer U4.H6 (IOL_10A)
- net at J11.2: no longer U4.B2 (IOL_1B)
- net at J11.20: no longer U4.F1 (IOL_10B)
- net at J11.21: no longer U4.H4 (IOL_11A)
- net at J11.22: no longer U4.G2 (IOL_11B)
- net at J11.23: no longer U4.J4 (IOL_12A)
- net at J11.24: no longer U4.H2 (IOL_12B)
- net at J11.25: no longer U4.J5 (IOL_13A)
- net at J11.26: no longer U4.H1 (IOL_14B)
- net at J11.27: no longer U4.J2 (IOL_15A)
- net at J11.28: no longer U4.J1 (IOL_15B)
- net at J11.29: no longer U4.K1 (IOL_16A)
- net at J11.3: no longer U4.F5 (IOL_2A)
- net at J11.30: no longer U4.K3 (IOL_16B)
- net at J11.31: no longer U4.L4 (IOL_17A)
- net at J11.32: no longer U4.L1 (IOL_17B)
- net at J11.33: no longer U4.K4 (IOL_18A)
- net at J11.34: no longer U4.M1 (IOL_18B)
- net at J11.35: no longer U4.L6 (IOL_19A)
- net at J11.36: no longer U4.L3 (IOL_19B)
- net at J11.37: no longer U4.K5 (IOL_20A)
- net at J11.38: no longer U4.M2 (IOL_20B)
- net at J11.39: no longer U4.L7 (IOL_21A)
- net at J11.4: no longer U4.B1 (IOL_2B)
- net at J11.40: no longer U4.N2 (IOL_21B)
- net at J11.41: no longer U4.M6 (IOL_22A)
- net at J11.42: no longer U4.M3 (IOL_22B)
- net at J11.43: no longer U4.L5 (IOL_23A)
- net at J11.44: no longer U4.N3 (IOL_23B)
- net at J11.45: no longer U4.P1 (IOL_24A)
- net at J11.46: no longer U4.M4 (IOL_24B)
- net at J11.47: no longer U4.P2 (IOL_25A)
- net at J11.48: no longer U4.M5 (IOL_25B)
- net at J11.49: no longer U4.R1 (IOL_26A)
- net at J11.5: no longer U4.C1 (IOL_3A)
- net at J11.50: no longer U4.N4 (IOL_26B)
- net at J11.6: no longer U4.C2 (IOL_3B)
- net at J11.7: no longer U4.F4 (IOL_4A)
- net at J11.8: no longer U4.D2 (IOL_4B)
- net at J11.9: no longer U4.G5 (IOL_5A)
- net at U4.A1 (IOT_220): no longer J6.43
- net at U4.A10 (IOT_186): no longer J6.18
- net at U4.A11 (IOT_187): no longer J6.19
- net at U4.A15 (IOT_177): no longer J6.9
- net at U4.A16 (IOT_176): no longer J6.8
- net at U4.A2 (IOT_218): no longer J6.41
- net at U4.A5 (IOT_213): no longer J6.37
- net at U4.A6 (IOT_211): no longer J6.35
- net at U4.A7 (IOT_205): no longer J6.29
- net at U4.A9 (IOT_194): no longer J6.24
- net at U4.B10 (IOT_183): no longer J6.15
- net at U4.B11 (IOT_184): no longer J6.16
- net at U4.B12 (IOT_182): no longer J6.14
- net at U4.B13 (IOT_178): no longer J6.10
- net at U4.B14 (IOT_171): no longer J6.4
- net at U4.B15 (IOT_169): no longer J6.2
- net at U4.B3 (IOT_223): no longer J6.46
- net at U4.B4 (IOT_216): no longer J6.40
- net at U4.B5 (IOT_214): no longer J6.38
- net at U4.B6 (IOT_208): no longer J6.32
- net at U4.B7 (IOT_207): no longer J6.31
- net at U4.B8 (IOT_203): no longer J6.28
- net at U4.B9 (IOT_199): no longer J6.26
- net at U4.C10 (IOT_185): no longer J6.17
- net at U4.C11 (IOT_180): no longer J6.12
- net at U4.C12 (IOT_172): no longer J6.5
- net at U4.C13 (IOT_174): no longer J6.7
- net at U4.C14 (IOT_168): no longer J6.1
- net at U4.C3 (IOT_227): no longer J6.50
- net at U4.C4 (IOT_222): no longer J6.45
- net at U4.C5 (IOT_221): no longer J6.44
- net at U4.C6 (IOT_209): no longer J6.33
- net at U4.C7 (IOT_206): no longer J6.30
- net at U4.C9 (IOT_191): no longer J6.21
- net at U4.D10 (IOT_190): no longer J6.20
- net at U4.D11 (IOT_181): no longer J6.13
- net at U4.D13 (IOT_170): no longer J6.3
- net at U4.D3 (IOT_226): no longer J6.49
- net at U4.D4 (IOT_224): no longer J6.47
- net at U4.D5 (IOT_219): no longer J6.42
- net at U4.D6 (IOT_212): no longer J6.36
- net at U4.D7 (IOT_210): no longer J6.34
- net at U4.D8 (IOT_200): no longer J6.27
- net at U4.D9 (IOT_193): no longer J6.23
- net at U4.E10 (IOT_179): no longer J6.11
- net at U4.E11 (IOT_173): no longer J6.6
- net at U4.E5 (IOT_225): no longer J6.48
- net at U4.E6 (IOT_215): no longer J6.39
- net at U4.E9 (IOT_192): no longer J6.22
- net at U4.F9 (IOT_196): no longer J6.25
- net at U4.B16 (IOR_165): no longer J9.48
- net at U4.C16 (IOR_161): no longer J9.46
- net at U4.D14 (IOR_167): no longer J9.50
- net at U4.D15 (IOR_157): no longer J9.43
- net at U4.D16 (IOR_153): no longer J9.39
- net at U4.E13 (IOR_166): no longer J9.49
- net at U4.E14 (IOR_160): no longer J9.45
- net at U4.E16 (IOR_151): no longer J9.37
- net at U4.F11 (IOR_158): no longer J9.44
- net at U4.F12 (IOR_156): no longer J9.42
- net at U4.F13 (IOR_162): no longer J9.47
- net at U4.F14 (IOR_155): no longer J9.41
- net at U4.F15 (IOR_149): no longer J9.35
- net at U4.F16 (IOR_147): no longer J9.33
- net at U4.G10 (IOR_146): no longer J9.32
- net at U4.G11 (IOR_148): no longer J9.34
- net at U4.G12 (IOR_154): no longer J9.40
- net at U4.G13 (IOR_152): no longer J9.38
- net at U4.G14 (IOR_150): no longer J9.36
- net at U4.G15 (IOR_145): no longer J9.31
- net at U4.G16 (IOR_143): no longer J9.29
- net at U4.H12 (IOR_144): no longer J9.30
- net at U4.H13 (IOR_139): no longer J9.27
- net at U4.H14 (IOR_142): no longer J9.28
- net at U4.J10 (IOR_122): no longer J9.14
- net at U4.J11 (IOR_126): no longer J9.16
- net at U4.J12 (IOR_136): no longer J9.24
- net at U4.J13 (IOR_137): no longer J9.25
- net at U4.J14 (IOR_134): no longer J9.23
- net at U4.J15 (IOR_130): no longer J9.20
- net at U4.J16 (IOR_138): no longer J9.26
- net at U4.K12 (IOR_120): no longer J9.12
- net at U4.K13 (IOR_128): no longer J9.18
- net at U4.K14 (IOR_129): no longer J9.19
- net at U4.K15 (IOR_131): no longer J9.21
- net at U4.K16 (IOR_133): no longer J9.22
- net at U4.L12 (IOR_116): no longer J9.8
- net at U4.L13 (IOR_118): no longer J9.10
- net at U4.L14 (IOR_119): no longer J9.11
- net at U4.L16 (IOR_127): no longer J9.17
- net at U4.M13 (IOR_114): no longer J9.6
- net at U4.M14 (IOR_115): no longer J9.7
- net at U4.M15 (IOR_123): no longer J9.15
- net at U4.M16 (IOR_121): no longer J9.13
- net at U4.N16 (IOR_117): no longer J9.9
- net at U4.P14 (IOR_111): no longer J9.3
- net at U4.P15 (IOR_112): no longer J9.4
- net at U4.P16 (IOR_113): no longer J9.5
- net at U4.R14 (IOR_109): no longer J9.1
- net at U4.R15 (IOR_110): no longer J9.2
- net ICE_B2_85: now reaches U4.L10 (IOB_85)
- net ICE_B2_85: now also J10.4
- net ICE_B2_99: now reaches U4.L11 (IOB_99)
- net ICE_B2_99: now also J10.40
- net ICE_B2_74: now reaches U4.L9 (IOB_74)
- net ICE_B2_74: now also J10.5
- net ICE_B2_93: now reaches U4.M11 (IOB_93)
- net ICE_B2_93: now also J10.37
- net ICE_B2_101: now reaches U4.M12 (IOB_101)
- net ICE_B2_101: now also J10.41
- net ICE_B2_64: now reaches U4.M7 (IOB_64)
- net ICE_B2_64: now also J10.1
- net ICE_B2_68: now reaches U4.M8 (IOB_68)
- net ICE_B2_68: now also J10.3
- net ICE_B2_80: now reaches U4.M9 (IOB_80)
- net ICE_B2_80: now also J10.2
- net ICE_B2_87: now reaches U4.N10 (IOB_87)
- net ICE_B2_87: now also J10.36
- net ICE_B2_98: now reaches U4.N12 (IOB_98)
- net ICE_B2_98: now also J10.39
- net ICE_B2_56: now reaches U4.N5 (IOB_56)
- net ICE_B2_56: now also J10.7
- net ICE_B2_52: now reaches U4.N6 (IOB_52)
- net ICE_B2_52: now also J10.9
- net ICE_B2_66: now reaches U4.N7 (IOB_66)
- net ICE_B2_66: now also J10.11
- net ICE_B2_78: now reaches U4.N9 (IOB_78)
- net ICE_B2_78: now also J10.34
- net ICE_B2_86: now reaches U4.P10 (IOB_86)
- net ICE_B2_86: now also J10.35
- net ICE_B2_54: now reaches U4.P4 (IOB_54)
- net ICE_B2_54: now also J10.6
- net ICE_B2_58: now reaches U4.P5 (IOB_58)
- net ICE_B2_58: now also J10.8
- net ICE_B2_67: now reaches U4.P6 (IOB_67)
- net ICE_B2_67: now also J10.10
- net ICE_B2_77: now reaches U4.P7 (IOB_77)
- net ICE_B2_77: now also J10.12
- net ICE_B2_72: now reaches U4.P8 (IOB_72)
- net ICE_B2_72: now also J10.13
- net ICE_B2_83: now reaches U4.P9 (IOB_83)
- net ICE_B2_83: now also J10.33
- net ICE_B2_84: now reaches U4.R10 (IOB_84)
- net ICE_B2_84: now also J10.38
- net ICE_B2_102: now reaches U4.R16 (IOB_102)
- net ICE_B2_102: now also J10.42
- net ICE_B2_55: now reaches U4.R2 (IOB_55)
- net ICE_B2_55: now also J10.15
- net ICE_B2_59: now reaches U4.R3 (IOB_59)
- net ICE_B2_59: now also J10.17
- net ICE_B2_63: now reaches U4.R4 (IOB_63)
- net ICE_B2_63: now also J10.19
- net ICE_B2_60: now reaches U4.R5 (IOB_60)
- net ICE_B2_60: now also J10.20
- net ICE_B2_71: now reaches U4.R6 (IOB_71)
- net ICE_B2_71: now also J10.22
- net ICE_B2_53: now reaches U4.T1 (IOB_53)
- net ICE_B2_53: now also J10.14
- net ICE_B2_57: now reaches U4.T2 (IOB_57)
- net ICE_B2_57: now also J10.16
- net ICE_B2_61: now reaches U4.T3 (IOB_61)
- net ICE_B2_61: now also J10.18
- net ICE_B2_69: now reaches U4.T5 (IOB_69)
- net ICE_B2_69: now also J10.21
- net ICE_B2_73: now reaches U4.T6 (IOB_73)
- net ICE_B2_73: now also J10.23
- net ICE_B2_75: now reaches U4.T7 (IOB_75)
- net ICE_B2_75: now also J10.24
Other:
- moved on the sheet: J10, J11

Commit message: bank L done
Parts:
- removed TP14, TP15, TP22, TP23: TestPoint, TestPoint:TestPoint_Pad_D3.0mm, symbol Connector:TestPoint
Connections:
- net ICE_B3_2A: now reaches J11.1
- net ICE_B3_2A: now also U4.F5 (IOL_2A)
- net ICE_B3_8A: now reaches J11.10
- net ICE_B3_8A: now also U4.G3 (IOL_8A)
- net ICE_B3_11A: now reaches J11.11
- net ICE_B3_11A: now also U4.H4 (IOL_11A)
- net ICE_B3_9A: now reaches J11.12
- net ICE_B3_9A: now also U4.H3 (IOL_9A)
- net ICE_B3_1B: now reaches J11.13
- net ICE_B3_1B: now also U4.B2 (IOL_1B)
- net ICE_B3_2B: now reaches J11.14
- net ICE_B3_2B: now also U4.B1 (IOL_2B)
- net ICE_B3_3B: now reaches J11.15
- net ICE_B3_3B: now also U4.C2 (IOL_3B)
- net ICE_B3_3A: now reaches J11.16
- net ICE_B3_3A: now also U4.C1 (IOL_3A)
- net ICE_B3_4B: now reaches J11.17
- net ICE_B3_4B: now also U4.D2 (IOL_4B)
- net ICE_B3_5B: now reaches J11.18
- net ICE_B3_5B: now also U4.D1 (IOL_5B)
- net ICE_B3_7B: now reaches J11.19
- net ICE_B3_7B: now also U4.E2 (IOL_7B)
- net ICE_B3_4A: now reaches J11.2
- net ICE_B3_4A: now also U4.F4 (IOL_4A)
- net ICE_B3_9B: now reaches J11.20
- net ICE_B3_9B: now also U4.F2 (IOL_9B)
- net ICE_B3_10B: now reaches J11.21
- net ICE_B3_10B: now also U4.F1 (IOL_10B)
- net ICE_B3_11B: now reaches J11.22
- net ICE_B3_11B: now also U4.G2 (IOL_11B)
- net ICE_B3_12B: now reaches J11.23
- net ICE_B3_12B: now also U4.H2 (IOL_12B)
- net ICE_B3_14B: now reaches J11.24
- net ICE_B3_14B: now also U4.H1 (IOL_14B)
- net ICE_B3_15A: now reaches J11.25
- net ICE_B3_15A: now also U4.J2 (IOL_15A)
- net ICE_B3_15B: now reaches J11.26
- net ICE_B3_15B: now also U4.J1 (IOL_15B)
- net ICE_B3_17B: now reaches J11.27
- net ICE_B3_17B: now also U4.L1 (IOL_17B)
- net ICE_B3_16A: now reaches J11.28
- net ICE_B3_16A: now also U4.K1 (IOL_16A)
- net ICE_B3_20B: now reaches J11.29
- net ICE_B3_20B: now also U4.M2 (IOL_20B)
- net ICE_B3_5A: now reaches J11.3
- net ICE_B3_5A: now also U4.G5 (IOL_5A)
- net ICE_B3_18B: now reaches J11.30
- net ICE_B3_18B: now also U4.M1 (IOL_18B)
- net ICE_B3_24A: now reaches J11.31
- net ICE_B3_24A: now also U4.P1 (IOL_24A)
- net ICE_B3_21B: now reaches J11.32
- net ICE_B3_21B: now also U4.N2 (IOL_21B)
- net ICE_B3_26A: now reaches J11.33
- net ICE_B3_26A: now also U4.R1 (IOL_26A)
- net ICE_B3_25A: now reaches J11.34
- net ICE_B3_25A: now also U4.P2 (IOL_25A)
- net ICE_B3_12A: now reaches J11.35
- net ICE_B3_12A: now also U4.J4 (IOL_12A)
- net ICE_B3_10A: now reaches J11.36
- net ICE_B3_10A: now also U4.H6 (IOL_10A)
- net ICE_B3_16B: now reaches J11.37
- net ICE_B3_16B: now also U4.K3 (IOL_16B)
- net ICE_B3_13A: now reaches J11.38
- net ICE_B3_13A: now also U4.J5 (IOL_13A)
- net ICE_B3_19B: now reaches J11.39
- net ICE_B3_19B: now also U4.L3 (IOL_19B)
- net ICE_B3_7A: now reaches J11.4
- net ICE_B3_7A: now also U4.H5 (IOL_7A)
- net ICE_B3_18A: now reaches J11.40
- net ICE_B3_18A: now also U4.K4 (IOL_18A)
- net ICE_B3_22B: now reaches J11.41
- net ICE_B3_22B: now also U4.M3 (IOL_22B)
- net ICE_B3_17A: now reaches J11.42
- net ICE_B3_17A: now also U4.L4 (IOL_17A)
- net ICE_B3_26B: now reaches J11.43
- net ICE_B3_26B: now also U4.N4 (IOL_26B)
- net ICE_B3_23B: now reaches J11.44
- net ICE_B3_23B: now also U4.N3 (IOL_23B)
- net ICE_B3_23A: now reaches J11.45
- net ICE_B3_23A: now also U4.L5 (IOL_23A)
- net ICE_B3_19A: now reaches J11.46
- net ICE_B3_19A: now also U4.L6 (IOL_19A)
- net ICE_B3_25B: now reaches J11.47
- net ICE_B3_25B: now also U4.M5 (IOL_25B)
- net ICE_B3_24B: now reaches J11.48
- net ICE_B3_24B: now also U4.M4 (IOL_24B)
- net ICE_B3_21A: now reaches J11.49
- net ICE_B3_21A: now also U4.L7 (IOL_21A)
- net ICE_B3_20A: now reaches J11.5
- net ICE_B3_20A: now also U4.K5 (IOL_20A)
- net ICE_B3_22A: now reaches J11.50
- net ICE_B3_22A: now also U4.M6 (IOL_22A)
- net ICE_B3_1A: now reaches J11.6
- net ICE_B3_1A: now also U4.E4 (IOL_1A)
- net ICE_B3_6B: now reaches J11.7
- net ICE_B3_6B: now also U4.E3 (IOL_6B)
- net ICE_B3_8B: now reaches J11.8
- net ICE_B3_8B: now also U4.F3 (IOL_8B)
- net ICE_B3_6A: now reaches J11.9
- net ICE_B3_6A: now also U4.G4 (IOL_6A)
Other:
- moved on the sheet: C34, C35, J10, J11, R24, R25, R26

Commit message: more traces
Connections:
- net ICE_B2_100: now also J10.34; no longer J10.32
- net ICE_B2_102: now also J10.33; no longer J10.42
- net ICE_B2_68: now also J10.2; no longer J10.3
- net ICE_B2_74: now also J10.4; no longer J10.5
- net ICE_B2_78: now also J10.35; no longer J10.34
- net ICE_B2_80: now also J10.3; no longer J10.2
- net ICE_B2_83: now also J10.36; no longer J10.33
- net ICE_B2_84: now also J10.28; no longer J10.38
- net ICE_B2_85: now also J10.5; no longer J10.4
- net ICE_B2_86: now also J10.38; no longer J10.35
- net ICE_B2_87: now also J10.37; no longer J10.36
- net ICE_B2_89: now also J10.30; no longer J10.28
- net ICE_B2_92: now also J10.32; no longer J10.30
- net ICE_B2_93: now also J10.40; no longer J10.37
- net ICE_B2_98: now also J10.42; no longer J10.39
- net ICE_B2_99: now also J10.39; no longer J10.40
- net ICE_T_220: now reaches U4.A1 (IOT_220)
- net ICE_T_220: now also J6.35
- net ICE_T_186: now reaches U4.A10 (IOT_186)
- net ICE_T_186: now also J6.22
- net ICE_T_187: now reaches U4.A11 (IOT_187)
- net ICE_T_187: now also J6.20
- net ICE_T_177: now reaches U4.A15 (IOT_177)
- net ICE_T_177: now also J6.15
- net ICE_T_176: now reaches U4.A16 (IOT_176)
- net ICE_T_176: now also J6.13
- net ICE_T_218: now reaches U4.A2 (IOT_218)
- net ICE_T_218: now also J6.36
- net ICE_T_213: now reaches U4.A5 (IOT_213)
- net ICE_T_213: now also J6.32
- net ICE_T_211: now reaches U4.A6 (IOT_211)
- net ICE_T_211: now also J6.30
- net ICE_T_205: now reaches U4.A7 (IOT_205)
- net ICE_T_205: now also J6.28
- net ICE_T_194: now reaches U4.A9 (IOT_194)
- net ICE_T_194: now also J6.24
- net ICE_T_183: now reaches U4.B10 (IOT_183)
- net ICE_T_183: now also J6.21
- net ICE_T_184: now reaches U4.B11 (IOT_184)
- net ICE_T_184: now also J6.19
- net ICE_T_182: now reaches U4.B12 (IOT_182)
- net ICE_T_182: now also J6.18
- net ICE_T_178: now reaches U4.B13 (IOT_178)
- net ICE_T_178: now also J6.17
- net ICE_T_171: now reaches U4.B14 (IOT_171)
- net ICE_T_171: now also J6.16
- net ICE_T_169: now reaches U4.B15 (IOT_169)
- net ICE_T_169: now also J6.14
- net ICE_T_223: now reaches U4.B3 (IOT_223)
- net ICE_T_223: now also J6.33
- net ICE_T_216: now reaches U4.B4 (IOT_216)
- net ICE_T_216: now also J6.34
- net ICE_T_214: now reaches U4.B5 (IOT_214)
- net ICE_T_214: now also J6.31
- net ICE_T_208: now reaches U4.B6 (IOT_208)
- net ICE_T_208: now also J6.29
- net ICE_T_207: now reaches U4.B7 (IOT_207)
- net ICE_T_207: now also J6.27
- net ICE_T_203: now reaches U4.B8 (IOT_203)
- net ICE_T_203: now also J6.26
- net ICE_T_199: now reaches U4.B9 (IOT_199)
- net ICE_T_199: now also J6.23
- net ICE_T_200: now reaches U4.D8 (IOT_200)
- net ICE_T_200: now also J6.25
- net ICE_R_165: now reaches U4.B16 (IOR_165)
- net ICE_R_165: now also J9.35
- net ICE_R_161: now reaches U4.C16 (IOR_161)
- net ICE_R_161: now also J9.36
- net ICE_R_157: now reaches U4.D15 (IOR_157)
- net ICE_R_157: now also J9.33
- net ICE_R_153: now reaches U4.D16 (IOR_153)
- net ICE_R_153: now also J9.34
- net ICE_R_160: now reaches U4.E14 (IOR_160)
- net ICE_R_160: now also J9.31
- net ICE_R_151: now reaches U4.E16 (IOR_151)
- net ICE_R_151: now also J9.32
- net ICE_R_149: now reaches U4.F15 (IOR_149)
- net ICE_R_149: now also J9.29
- net ICE_R_147: now reaches U4.F16 (IOR_147)
- net ICE_R_147: now also J9.30
- net ICE_R_145: now reaches U4.G15 (IOR_145)
- net ICE_R_145: now also J9.27
- net ICE_R_143: now reaches U4.G16 (IOR_143)
- net ICE_R_143: now also J9.28
- net ICE_R_130: now reaches U4.J15 (IOR_130)
- net ICE_R_130: now also J9.25
- net ICE_R_138: now reaches U4.J16 (IOR_138)
- net ICE_R_138: now also J9.26
- net ICE_R_131: now reaches U4.K15 (IOR_131)
- net ICE_R_131: now also J9.23
- net ICE_R_133: now reaches U4.K16 (IOR_133)
- net ICE_R_133: now also J9.24
- net ICE_R_119: now reaches U4.L14 (IOR_119)
- net ICE_R_119: now also J9.21
- net ICE_R_127: now reaches U4.L16 (IOR_127)
- net ICE_R_127: now also J9.22
- net ICE_R_123: now reaches U4.M15 (IOR_123)
- net ICE_R_123: now also J9.19
- net ICE_R_121: now reaches U4.M16 (IOR_121)
- net ICE_R_121: now also J9.20
- net ICE_R_117: now reaches U4.N16 (IOR_117)
- net ICE_R_117: now also J9.18
- net ICE_R_112: now reaches U4.P15 (IOR_112)
- net ICE_R_112: now also J9.16
- net ICE_R_113: now reaches U4.P16 (IOR_113)
- net ICE_R_113: now also J9.17
Other:
- moved on the sheet: J6, J9, R20

Commit message: added again some traces
Connections:
- net ICE_R_167: now reaches U4.D14 (IOR_167)
- net ICE_R_167: now also J9.44
- net ICE_R_166: now reaches U4.E13 (IOR_166)
- net ICE_R_166: now also J9.41
- net ICE_R_158: now reaches U4.F11 (IOR_158)
- net ICE_R_158: now also J9.48
- net ICE_R_156: now reaches U4.F12 (IOR_156)
- net ICE_R_156: now also J9.46
- net ICE_R_162: now reaches U4.F13 (IOR_162)
- net ICE_R_162: now also J9.42
- net ICE_R_155: now reaches U4.F14 (IOR_155)
- net ICE_R_155: now also J9.39
- net ICE_R_146: now reaches U4.G10 (IOR_146)
- net ICE_R_146: now also J9.45
- net ICE_R_154: now reaches U4.G12 (IOR_154)
- net ICE_R_154: now also J9.43
- net ICE_R_152: now reaches U4.G13 (IOR_152)
- net ICE_R_152: now also J9.40
- net ICE_R_150: now reaches U4.G14 (IOR_150)
- net ICE_R_150: now also J9.37
- net ICE_R_142: now reaches U4.H14 (IOR_142)
- net ICE_R_142: now also J9.38
- net ICE_R_122: now reaches U4.J10 (IOR_122)
- net ICE_R_122: now also J9.3
- net ICE_R_126: now reaches U4.J11 (IOR_126)
- net ICE_R_126: now also J9.2
- net ICE_R_136: now reaches U4.J12 (IOR_136)
- net ICE_R_136: now also J9.1
- net ICE_R_137: now reaches U4.J13 (IOR_137)
- net ICE_R_137: now also J9.14
- net ICE_R_134: now reaches U4.J14 (IOR_134)
- net ICE_R_134: now also J9.15
- net ICE_R_120: now reaches U4.K12 (IOR_120)
- net ICE_R_120: now also J9.4
- net ICE_R_128: now reaches U4.K13 (IOR_128)
- net ICE_R_128: now also J9.12
- net ICE_R_129: now reaches U4.K14 (IOR_129)
- net ICE_R_129: now also J9.13
- net ICE_R_116: now reaches U4.L12 (IOR_116)
- net ICE_R_116: now also J9.10
- net ICE_R_118: now reaches U4.L13 (IOR_118)
- net ICE_R_118: now also J9.11
- net ICE_R_114: now reaches U4.M13 (IOR_114)
- net ICE_R_114: now also J9.8
- net ICE_R_115: now reaches U4.M14 (IOR_115)
- net ICE_R_115: now also J9.9
- net ICE_R_111: now reaches U4.P14 (IOR_111)
- net ICE_R_111: now also J9.7
- net ICE_R_109: now reaches U4.R14 (IOR_109)
- net ICE_R_109: now also J9.6
- net ICE_R_110: now reaches U4.R15 (IOR_110)
- net ICE_R_110: now also J9.5
