File: FuseBox/FUSEBOX.kicad_pcb (KiCad board)
At the start: 2 copper layers, 6 parts, among them J1 UJ31CHG2SMTTR, J2 61301611121, U1 TPS61040DBVR, U2 LT3030EFETRPBF, U3 STM32F407VGTx

Commit message: changes
Parts:
- added C1: 10u, Capacitor_SMD:C_0603_1608Metric_Pad1.08x0.95mm_HandSolder, F.Cu at (-68.0, 34.2)
- added C10: 10u, Capacitor_SMD:C_0603_1608Metric_Pad1.08x0.95mm_HandSolder, F.Cu at (-63.6, 36.7)
- added C11: 22u, Capacitor_SMD:C_0603_1608Metric_Pad1.08x0.95mm_HandSolder, F.Cu at (-63.6, 39.2)
- added C12: 100n, Capacitor_SMD:C_0603_1608Metric_Pad1.08x0.95mm_HandSolder, F.Cu at (-63.6, 41.7)
- added C13: 4u7, Capacitor_SMD:C_0603_1608Metric_Pad1.08x0.95mm_HandSolder, F.Cu at (-63.6, 44.2)
- added C14: 22u, Capacitor_SMD:C_0603_1608Metric_Pad1.08x0.95mm_HandSolder, F.Cu at (-63.6, 46.7)
- added C15: 20p, Capacitor_SMD:C_0603_1608Metric_Pad1.08x0.95mm_HandSolder, F.Cu at (-72.4, 97.3)
- added C16: 100p, Capacitor_SMD:C_0603_1608Metric_Pad1.08x0.95mm_HandSolder, F.Cu at (-136.6, 140.4)
- added C17: 100p, Capacitor_SMD:C_0603_1608Metric_Pad1.08x0.95mm_HandSolder, F.Cu at (-136.6, 142.9)
- added C18: 100p, Capacitor_SMD:C_0603_1608Metric_Pad1.08x0.95mm_HandSolder, F.Cu at (-136.6, 145.4)
- added C19: 100p, Capacitor_SMD:C_0603_1608Metric_Pad1.08x0.95mm_HandSolder, F.Cu at (-136.6, 148.0)
- added C2: 30p, Capacitor_SMD:C_0603_1608Metric_Pad1.08x0.95mm_HandSolder, F.Cu at (-68.0, 36.7)
- added C20: 100n, Capacitor_SMD:C_0603_1608Metric_Pad1.08x0.95mm_HandSolder, F.Cu at (-136.6, 150.5)
- added C21: 10u, Capacitor_SMD:C_0603_1608Metric_Pad1.08x0.95mm_HandSolder, F.Cu at (-136.6, 153.0)
- added C22: 100p, Capacitor_SMD:C_0603_1608Metric_Pad1.08x0.95mm_HandSolder, F.Cu at (-136.6, 155.5)
- added C23: 100p, Capacitor_SMD:C_0603_1608Metric_Pad1.08x0.95mm_HandSolder, F.Cu at (-136.6, 158.0)
- added C24: 100p, Capacitor_SMD:C_0603_1608Metric_Pad1.08x0.95mm_HandSolder, F.Cu at (-132.3, 140.4)
- added C25: 100p, Capacitor_SMD:C_0603_1608Metric_Pad1.08x0.95mm_HandSolder, F.Cu at (-132.3, 142.9)
- added C26: 100p, Capacitor_SMD:C_0603_1608Metric_Pad1.08x0.95mm_HandSolder, F.Cu at (-132.3, 145.4)
- added C27: 100p, Capacitor_SMD:C_0603_1608Metric_Pad1.08x0.95mm_HandSolder, F.Cu at (-132.3, 148.0)
- added C28: 100p, Capacitor_SMD:C_0603_1608Metric_Pad1.08x0.95mm_HandSolder, F.Cu at (-132.3, 150.5)
- added C29: 100p, Capacitor_SMD:C_0603_1608Metric_Pad1.08x0.95mm_HandSolder, F.Cu at (-132.3, 153.0)
- added C3: 10u, Capacitor_SMD:C_0603_1608Metric_Pad1.08x0.95mm_HandSolder, F.Cu at (-68.0, 39.2)
- added C30: 100p, Capacitor_SMD:C_0603_1608Metric_Pad1.08x0.95mm_HandSolder, F.Cu at (-132.3, 155.5)
- added C31: 100p, Capacitor_SMD:C_0603_1608Metric_Pad1.08x0.95mm_HandSolder, F.Cu at (-132.3, 158.0)
- added C32: 100p, Capacitor_SMD:C_0603_1608Metric_Pad1.08x0.95mm_HandSolder, F.Cu at (-127.9, 140.4)
- added C33: 100p, Capacitor_SMD:C_0603_1608Metric_Pad1.08x0.95mm_HandSolder, F.Cu at (-127.9, 142.9)
- added C34: 100n, Capacitor_SMD:C_0603_1608Metric_Pad1.08x0.95mm_HandSolder, F.Cu at (-127.9, 145.4)
- added C35: 10u, Capacitor_SMD:C_0603_1608Metric_Pad1.08x0.95mm_HandSolder, F.Cu at (-127.9, 148.0)
- added C36: 10u, Capacitor_SMD:C_0603_1608Metric_Pad1.08x0.95mm_HandSolder, F.Cu at (-127.9, 150.5)
- added C37: 1u, Capacitor_SMD:C_0603_1608Metric_Pad1.08x0.95mm_HandSolder, F.Cu at (-127.9, 153.0)
- added C38: 100n, Capacitor_SMD:C_0603_1608Metric_Pad1.08x0.95mm_HandSolder, F.Cu at (-127.9, 155.5)
- added C39: 100n, Capacitor_SMD:C_0603_1608Metric_Pad1.08x0.95mm_HandSolder, F.Cu at (-127.9, 158.0)
- added C4: 20p, Capacitor_SMD:C_0603_1608Metric_Pad1.08x0.95mm_HandSolder, F.Cu at (-72.4, 94.8)
- added C40: 100n, Capacitor_SMD:C_0603_1608Metric_Pad1.08x0.95mm_HandSolder, F.Cu at (-123.6, 140.4)
- added C41: 100n, Capacitor_SMD:C_0603_1608Metric_Pad1.08x0.95mm_HandSolder, F.Cu at (-123.6, 142.9)
- added C42: 10n, Capacitor_SMD:C_0603_1608Metric_Pad1.08x0.95mm_HandSolder, F.Cu at (-123.6, 145.4)
- added C43: 10u, Capacitor_SMD:C_0603_1608Metric_Pad1.08x0.95mm_HandSolder, F.Cu at (-123.6, 148.0)
- added C44: 1u, Capacitor_SMD:C_0603_1608Metric_Pad1.08x0.95mm_HandSolder, F.Cu at (-123.6, 150.5)
- added C45: 100n, Capacitor_SMD:C_0603_1608Metric_Pad1.08x0.95mm_HandSolder, F.Cu at (-123.6, 153.0)
- added C46: 10n, Capacitor_SMD:C_0603_1608Metric_Pad1.08x0.95mm_HandSolder, F.Cu at (-123.6, 155.5)
- added C47: 100n, Capacitor_SMD:C_0603_1608Metric_Pad1.08x0.95mm_HandSolder, F.Cu at (-72.4, 99.8)
- added C48: 100n, Capacitor_SMD:C_0603_1608Metric_Pad1.08x0.95mm_HandSolder, F.Cu at (-72.4, 102.3)
- added C49: 100n, Capacitor_SMD:C_0603_1608Metric_Pad1.08x0.95mm_HandSolder, F.Cu at (-72.4, 104.8)
- added C5: 2u2, Capacitor_SMD:C_0603_1608Metric_Pad1.08x0.95mm_HandSolder, F.Cu at (-68.0, 41.7)
- added C50: 2p2, Capacitor_SMD:C_0603_1608Metric_Pad1.08x0.95mm_HandSolder, F.Cu at (-72.4, 107.3)
- added C51: 100n, Capacitor_SMD:C_0603_1608Metric_Pad1.08x0.95mm_HandSolder, F.Cu at (-72.4, 109.8)
- added C52: 100n, Capacitor_SMD:C_0603_1608Metric_Pad1.08x0.95mm_HandSolder, F.Cu at (-72.4, 112.3)
- added C53: 2p2, Capacitor_SMD:C_0603_1608Metric_Pad1.08x0.95mm_HandSolder, F.Cu at (-68.0, 94.8)
- added C54: 1u, Capacitor_SMD:C_0603_1608Metric_Pad1.08x0.95mm_HandSolder, F.Cu at (-68.0, 97.3)
- added C55: 1u, Capacitor_SMD:C_0603_1608Metric_Pad1.08x0.95mm_HandSolder, F.Cu at (-68.0, 99.8)
- added C56: 100n, Capacitor_SMD:C_0603_1608Metric_Pad1.08x0.95mm_HandSolder, F.Cu at (-68.0, 102.3)
- added C57: 100n, Capacitor_SMD:C_0603_1608Metric_Pad1.08x0.95mm_HandSolder, F.Cu at (-68.0, 104.8)
- added C58: 100n, Capacitor_SMD:C_0603_1608Metric_Pad1.08x0.95mm_HandSolder, F.Cu at (-68.0, 107.3)
- added C59: 100n, Capacitor_SMD:C_0603_1608Metric_Pad1.08x0.95mm_HandSolder, F.Cu at (-68.0, 109.8)
- added C6: 2u2, Capacitor_SMD:C_0603_1608Metric_Pad1.08x0.95mm_HandSolder, F.Cu at (-68.0, 44.2)
- added C60: 100n, Capacitor_SMD:C_0603_1608Metric_Pad1.08x0.95mm_HandSolder, F.Cu at (-68.0, 112.3)
- added C61: 1u, Capacitor_SMD:C_0603_1608Metric_Pad1.08x0.95mm_HandSolder, F.Cu at (-63.7, 94.8)
- added C7: 10u, Capacitor_SMD:C_0603_1608Metric_Pad1.08x0.95mm_HandSolder, F.Cu at (-68.0, 46.7)
- added C8: 10n, Capacitor_SMD:C_0603_1608Metric_Pad1.08x0.95mm_HandSolder, F.Cu at (-68.0, 49.3)
- added C9: 10n, Capacitor_SMD:C_0603_1608Metric_Pad1.08x0.95mm_HandSolder, F.Cu at (-63.6, 34.2)
- added D2: LED, LED_SMD:LED_0603_1608Metric, F.Cu at (-53.9, 51.8)
- added D3: LED, LED_SMD:LED_0603_1608Metric, F.Cu at (-53.9, 54.4)
- added D4: LED, LED_SMD:LED_0603_1608Metric, F.Cu at (-53.9, 57.0)
- added D5: LED, LED_SMD:LED_0603_1608Metric, F.Cu at (-53.9, 59.6)
- added D6: CDSU4148, Diode_SMD:D_0603_1608Metric_Pad1.05x0.95mm_HandSolder, F.Cu at (-143.3, 144.7)
- added FB1: 600R 500mA, Inductor_SMD:L_0603_1608Metric_Pad1.05x0.95mm_HandSolder, F.Cu at (-63.6, 49.3)
- added FB2: 600R 500mA, Inductor_SMD:L_0603_1608Metric_Pad1.05x0.95mm_HandSolder, F.Cu at (-59.3, 34.2)
- added FB3: 600R 500mA, Inductor_SMD:L_0603_1608Metric_Pad1.05x0.95mm_HandSolder, F.Cu at (-59.3, 36.7)
- added FB4: 600R 500mA, Inductor_SMD:L_0603_1608Metric_Pad1.05x0.95mm_HandSolder, F.Cu at (-59.3, 39.2)
- added FB5: 600R 500mA, Inductor_SMD:L_0603_1608Metric_Pad1.05x0.95mm_HandSolder, F.Cu at (-63.7, 97.3)
- added J10: 901301150, Custom:901301150, F.Cu at (145.5, 239.5)
- added J11: 901301150, Custom:901301150, F.Cu at (136.1, 168.9)
- added J12: 901301240, Custom:901301240, F.Cu at (373.1, 229.5)
- added J3: 702462004, Custom:702462004, F.Cu at (294.9, 203.9)
- added J4: 702462004, Custom:702462004, F.Cu at (245.0, 226.2)
- added J5: 702462004, Custom:702462004, F.Cu at (240.1, 242.5)
- added J6: 901301150, Custom:901301150, F.Cu at (206.4, 159.5)
- added J7: 702462004, Custom:702462004, F.Cu at (277.5, 242.5)
- added J8: 61301611121, Custom:61301611121, F.Cu at (220.6, 255.5)
- added J9: 901301150, Custom:901301150, F.Cu at (216.0, 230.0)
- added L1: 10u, Inductor_SMD:L_0603_1608Metric_Pad1.05x0.95mm_HandSolder, F.Cu at (-59.3, 41.7)
- added R1: 5k1, Resistor_SMD:R_0603_1608Metric_Pad0.98x0.95mm_HandSolder, F.Cu at (-59.3, 44.2)
- added R10: 100, Resistor_SMD:R_0603_1608Metric_Pad0.98x0.95mm_HandSolder, F.Cu at (-54.9, 49.3)
- added R11: 100m, Resistor_SMD:R_0603_1608Metric_Pad0.98x0.95mm_HandSolder, F.Cu at (-50.6, 34.2)
- added R12: 100, Resistor_SMD:R_0603_1608Metric_Pad0.98x0.95mm_HandSolder, F.Cu at (-50.6, 36.7)
- added R13: 100m, Resistor_SMD:R_0603_1608Metric_Pad0.98x0.95mm_HandSolder, F.Cu at (-50.6, 39.2)
- added R14: 1, Resistor_SMD:R_0603_1608Metric_Pad0.98x0.95mm_HandSolder, F.Cu at (-50.6, 41.7)
- added R15: 2k4, Resistor_SMD:R_0603_1608Metric_Pad0.98x0.95mm_HandSolder, F.Cu at (-50.6, 44.2)
- added R16: 825, Resistor_SMD:R_0603_1608Metric_Pad0.98x0.95mm_HandSolder, F.Cu at (-50.6, 46.7)
- added R17: 300, Resistor_SMD:R_0603_1608Metric_Pad0.98x0.95mm_HandSolder, F.Cu at (-50.6, 49.3)
- added R18: 1, Resistor_SMD:R_0603_1608Metric_Pad0.98x0.95mm_HandSolder, F.Cu at (-123.6, 158.0)
- added R19: 100, Resistor_SMD:R_0603_1608Metric_Pad0.98x0.95mm_HandSolder, F.Cu at (-119.2, 140.4)
- added R2: 5k1, Resistor_SMD:R_0603_1608Metric_Pad0.98x0.95mm_HandSolder, F.Cu at (-59.3, 46.7)
- added R20: 10k, Resistor_SMD:R_0603_1608Metric_Pad0.98x0.95mm_HandSolder, F.Cu at (-119.2, 142.9)
- added R21: 1, Resistor_SMD:R_0603_1608Metric_Pad0.98x0.95mm_HandSolder, F.Cu at (-119.2, 145.4)
- added R22: 1, Resistor_SMD:R_0603_1608Metric_Pad0.98x0.95mm_HandSolder, F.Cu at (-119.2, 148.0)
- added R23: 1, Resistor_SMD:R_0603_1608Metric_Pad0.98x0.95mm_HandSolder, F.Cu at (-119.2, 150.5)
- added R24: 100, Resistor_SMD:R_0603_1608Metric_Pad0.98x0.95mm_HandSolder, F.Cu at (-119.2, 153.0)
- added R25: 10k, Resistor_SMD:R_0603_1608Metric_Pad0.98x0.95mm_HandSolder, F.Cu at (-119.2, 155.5)
- added R26: 649, Resistor_SMD:R_0603_1608Metric_Pad0.98x0.95mm_HandSolder, F.Cu at (-119.2, 158.0)
- added R27: 0, Resistor_SMD:R_0603_1608Metric_Pad0.98x0.95mm_HandSolder, F.Cu at (-63.7, 99.8)
- added R28: 0, Resistor_SMD:R_0603_1608Metric_Pad0.98x0.95mm_HandSolder, F.Cu at (-63.7, 102.3)
- added R29: 10k, Resistor_SMD:R_0603_1608Metric_Pad0.98x0.95mm_HandSolder, F.Cu at (-123.1, 72.7)
- added R3: 873k3, Resistor_SMD:R_0603_1608Metric_Pad0.98x0.95mm_HandSolder, F.Cu at (-59.3, 49.3)
- added R30: 10k, Resistor_SMD:R_0603_1608Metric_Pad0.98x0.95mm_HandSolder, F.Cu at (-123.1, 75.2)
- added R31: 10k, Resistor_SMD:R_0603_1608Metric_Pad0.98x0.95mm_HandSolder, F.Cu at (-123.1, 77.7)
- added R32: 10k, Resistor_SMD:R_0603_1608Metric_Pad0.98x0.95mm_HandSolder, F.Cu at (-123.1, 80.2)
- added R33: 10k, Resistor_SMD:R_0603_1608Metric_Pad0.98x0.95mm_HandSolder, F.Cu at (-123.1, 82.7)
- added R34: 10k, Resistor_SMD:R_0603_1608Metric_Pad0.98x0.95mm_HandSolder, F.Cu at (-123.1, 85.2)
- added R35: 10k, Resistor_SMD:R_0603_1608Metric_Pad0.98x0.95mm_HandSolder, F.Cu at (-123.1, 87.8)
- added R36: 10k, Resistor_SMD:R_0603_1608Metric_Pad0.98x0.95mm_HandSolder, F.Cu at (-123.1, 90.3)
- added R37: 10k, Resistor_SMD:R_0603_1608Metric_Pad0.98x0.95mm_HandSolder, F.Cu at (-118.7, 72.7)
- added R38: 10k, Resistor_SMD:R_0603_1608Metric_Pad0.98x0.95mm_HandSolder, F.Cu at (-118.7, 75.2)
- added R39: 10k, Resistor_SMD:R_0603_1608Metric_Pad0.98x0.95mm_HandSolder, F.Cu at (-118.7, 77.7)
- added R4: 100k, Resistor_SMD:R_0603_1608Metric_Pad0.98x0.95mm_HandSolder, F.Cu at (-54.9, 34.2)
- added R40: 10k, Resistor_SMD:R_0603_1608Metric_Pad0.98x0.95mm_HandSolder, F.Cu at (-118.7, 80.2)
- added R41: 10k, Resistor_SMD:R_0603_1608Metric_Pad0.98x0.95mm_HandSolder, F.Cu at (-118.7, 82.7)
- added R42: 10k, Resistor_SMD:R_0603_1608Metric_Pad0.98x0.95mm_HandSolder, F.Cu at (-118.7, 85.2)
- added R43: 10k, Resistor_SMD:R_0603_1608Metric_Pad0.98x0.95mm_HandSolder, F.Cu at (-118.7, 87.8)
- added R44: 10k, Resistor_SMD:R_0603_1608Metric_Pad0.98x0.95mm_HandSolder, F.Cu at (-118.7, 90.3)
- added R45: 10k, Resistor_SMD:R_0603_1608Metric_Pad0.98x0.95mm_HandSolder, F.Cu at (-114.4, 72.7)
- added R46: 10k, Resistor_SMD:R_0603_1608Metric_Pad0.98x0.95mm_HandSolder, F.Cu at (-114.4, 75.2)
- added R47: 10k, Resistor_SMD:R_0603_1608Metric_Pad0.98x0.95mm_HandSolder, F.Cu at (-114.4, 77.7)
- added R48: 10k, Resistor_SMD:R_0603_1608Metric_Pad0.98x0.95mm_HandSolder, F.Cu at (-114.4, 80.2)
- added R49: 10k, Resistor_SMD:R_0603_1608Metric_Pad0.98x0.95mm_HandSolder, F.Cu at (-114.4, 82.7)
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Connections:
- net /USB_OTG_FS_DN renamed /USB_PWR/STM_USB_OTG_FS_DN
- net /USB_OTG_FS_DP renamed /USB_PWR/STM_USB_OTG_FS_DP
- J2 pad 1: unconnected-(J2-Pad1) -> /STM32F4/STM_A0
- J2 pad 10: unconnected-(J2-Pad10) -> /STM32F4/STM_A9
- J2 pad 11: unconnected-(J2-Pad11) -> /STM32F4/STM_A10
- J2 pad 12: unconnected-(J2-Pad12) -> /STM32F4/STM_A11
- J2 pad 13: unconnected-(J2-Pad13) -> /STM32F4/STM_A12
- J2 pad 14: unconnected-(J2-Pad14) -> /STM32F4/STM_A13
- J2 pad 15: unconnected-(J2-Pad15) -> /STM32F4/STM_A14
- J2 pad 16: unconnected-(J2-Pad16) -> /STM32F4/STM_A15
- J2 pad 2: unconnected-(J2-Pad2) -> /STM32F4/STM_A1
- J2 pad 3: unconnected-(J2-Pad3) -> /STM32F4/STM_A2
- J2 pad 4: unconnected-(J2-Pad4) -> /STM32F4/STM_A3
- J2 pad 5: unconnected-(J2-Pad5) -> /STM32F4/STM_A4
- J2 pad 6: unconnected-(J2-Pad6) -> /STM32F4/STM_A5
- J2 pad 7: unconnected-(J2-Pad7) -> /STM32F4/STM_A6
- J2 pad 8: unconnected-(J2-Pad8) -> /STM32F4/STM_A7
- J2 pad 9: unconnected-(J2-Pad9) -> /STM32F4/STM_A8
- U3 pad 1: unconnected-(U3-PE2-Pad1) -> /STM32F4/STM_E2
- U3 pad 10: Net-(U3-VSS-Pad10) -> GND
- U3 pad 100: unconnected-(U3-VDD-Pad100) -> VDD
- U3 pad 11: unconnected-(U3-VDD-Pad11) -> VDD
- U3 pad 12: unconnected-(U3-PH0-Pad12) -> Net-(U3-PH0)
- U3 pad 13: unconnected-(U3-PH1-Pad13) -> Net-(U3-PH1)
- U3 pad 14: unconnected-(U3-NRST-Pad14) -> Net-(U3-NRST)
- U3 pad 15: unconnected-(U3-PC0-Pad15) -> /STM32F4/STM_C0
- U3 pad 16: unconnected-(U3-PC1-Pad16) -> /STM32F4/STM_C1
- U3 pad 17: unconnected-(U3-PC2-Pad17) -> /STM32F4/STM_C2
- U3 pad 18: unconnected-(U3-PC3-Pad18) -> /STM32F4/STM_C3
- U3 pad 19: unconnected-(U3-VDD-Pad19) -> VDD
- U3 pad 2: unconnected-(U3-PE3-Pad2) -> /STM32F4/STM_E3
- U3 pad 20: unconnected-(U3-VSSA-Pad20) -> GND
- U3 pad 21: unconnected-(U3-VREF+-Pad21) -> VREF+
- U3 pad 22: unconnected-(U3-VDDA-Pad22) -> VDDA
- U3 pad 23: unconnected-(U3-PA0-Pad23) -> /STM32F4/STM_A0
- U3 pad 24: unconnected-(U3-PA1-Pad24) -> /STM32F4/STM_A1
- U3 pad 25: unconnected-(U3-PA2-Pad25) -> /STM32F4/STM_A2
- U3 pad 26: unconnected-(U3-PA3-Pad26) -> /STM32F4/STM_A3
- U3 pad 27: Net-(U3-VSS-Pad10) -> GND
- U3 pad 28: unconnected-(U3-VDD-Pad28) -> VDD
- U3 pad 29: unconnected-(U3-PA4-Pad29) -> /STM32F4/STM_A4
- U3 pad 3: unconnected-(U3-PE4-Pad3) -> /STM32F4/STM_E4
- U3 pad 30: unconnected-(U3-PA5-Pad30) -> /STM32F4/STM_A5
- U3 pad 31: unconnected-(U3-PA6-Pad31) -> /STM32F4/STM_A6
- U3 pad 32: unconnected-(U3-PA7-Pad32) -> /STM32F4/STM_A7
- U3 pad 33: unconnected-(U3-PC4-Pad33) -> /STM32F4/STM_C4
- U3 pad 34: unconnected-(U3-PC5-Pad34) -> /STM32F4/STM_C5
- U3 pad 35: unconnected-(U3-PB0-Pad35) -> /STM32F4/STM_B0
- U3 pad 36: unconnected-(U3-PB1-Pad36) -> /STM32F4/STM_B1
- U3 pad 37: unconnected-(U3-PB2-Pad37) -> /STM32F4/STM_B2
- U3 pad 38: unconnected-(U3-PE7-Pad38) -> /STM32F4/STM_E7
- U3 pad 39: unconnected-(U3-PE8-Pad39) -> /STM32F4/STM_E8
- U3 pad 4: unconnected-(U3-PE5-Pad4) -> /STM32F4/STM_E5
- U3 pad 40: unconnected-(U3-PE9-Pad40) -> /STM32F4/STM_E9
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Other:
- board outline added: 411.7 x 161.7 mm

Commit message: changes
Parts:
- moved R2 353.5 mm to (281.8, 139.9), turned to 90 degrees
- moved R1 348.9 mm to (276.2, 139.9), turned to 90 degrees
- moved J1 42.0 mm to (279.0, 129.5)
Other:
- copper layers 2 -> 6

Commit message: layout
Parts:
- moved +1V2 388.1 mm to (293.7, 147.9)
- moved VCC_1V2 384.0 mm to (288.7, 147.9)
- moved +3V3 383.5 mm to (293.7, 153.9)
- moved +1V22 380.5 mm to (283.7, 147.9)
- moved VCC_3V3 380.3 mm to (288.7, 153.9)
- moved GND 378.9 mm to (293.7, 142.0)
- moved +5V 377.1 mm to (278.7, 147.9)
- moved +3V31 375.9 mm to (283.7, 153.9)
- moved VBUS 373.8 mm to (273.7, 147.9)
- moved +12V 372.5 mm to (278.7, 153.9)
- moved VCC_12V 369.3 mm to (273.7, 153.9)
- moved C6 364.1 mm to (283.5, 139.2), turned to 90 degrees
- moved C5 356.7 mm to (275.4, 138.4)
- moved R5 355.3 mm to (285.2, 139.3), turned to -90 degrees
- moved C1 354.7 mm to (267.6, 149.1)
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- renumbered TP7 to +12V, TP5 to +1V2, TP3 to +1V22, TP10 to +3V3, TP8 to +3V31, TP2 to +5V, TP11 to GND, TP1 to VBUS, TP6 to VCC_12V, TP4 to VCC_1V2, TP9 to VCC_3V3
Connections:
- C12 pad 1: unconnected-(C12-Pad1) -> VCC_3V3
- R15 pad 2: unconnected-(R15-Pad2) -> +12V
- R17 pad 2: unconnected-(R17-Pad2) -> +1V2
Routing:
- net GND: track 0.00 -> 68.8 mm, vias 0 -> 22
- net +5V: track 0.00 -> 26.1 mm, vias 0 -> 2
- net +3V31: track 0.00 -> 13.6 mm
- net Net-(J1-CC2): track 0.00 -> 12.8 mm
- net Net-(U1-FB): track 0.00 -> 12.3 mm
- net +1V22: track 0.00 -> 12.1 mm
- net VBUS: track 0.00 -> 7.75 mm, vias 0 -> 1
- net VCC_12V: track 0.00 -> 7.23 mm
- net Net-(U2-PWRGD1): track 0.00 -> 6.10 mm
- net VCC_3V3: track 0.00 -> 5.66 mm
- net Net-(J1-CC1): track 0.00 -> 5.56 mm
- net Net-(U1-SW): track 0.00 -> 4.00 mm
- net +1V2: track 0.00 -> 3.90 mm, vias 0 -> 4
- net Net-(U2-BYP2): track 0.00 -> 3.83 mm
- net /USB_PWR/STM_USB_OTG_FS_DN: track 0.00 -> 3.74 mm, vias 0 -> 2
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- added copper zone on In3.Cu, net GND
Other:
- board text added: "U1"

Commit message: some bar
Parts:
- moved C5 1.16 mm to (276.6, 138.4)
- moved C6 1.16 mm to (284.7, 139.2)
- moved D2 1.16 mm to (288.1, 137.5)
- moved FB2 1.16 mm to (280.1, 139.3)
- moved J1 1.16 mm to (280.2, 129.5)
- moved R2 1.16 mm to (282.9, 139.3)
- moved R5 1.16 mm to (286.4, 139.3)
- moved R1 1.16 mm to (276.5, 140.1)
Routing:
- net +5V: track 26.1 -> 32.0 mm, vias 2 -> 7
- net VBUS: track 7.75 -> 9.76 mm, vias 1 -> 2
- added copper zone on In2.Cu, net +1V22
- added copper zone on In2.Cu, net +5V
- added copper zone on In2.Cu, net VBUS

Commit message: fpga decoupling
Parts:
- removed TP12, TP13, TP16, TP17, TP18, TP19, TP20, TP21: TestPoint, TestPoint:TestPoint_Pad_D3.0mm
- added TP1: TestPoint, TestPoint:TestPoint_Pad_D3.0mm, F.Cu at (2.02, 2.02)
- added TP10: TestPoint, TestPoint:TestPoint_Pad_D3.0mm, F.Cu at (12.1, 7.08)
- added TP11: TestPoint, TestPoint:TestPoint_Pad_D3.0mm, F.Cu at (12.1, 12.1)
- added TP2: TestPoint, TestPoint:TestPoint_Pad_D3.0mm, F.Cu at (2.02, 7.08)
- added TP3: TestPoint, TestPoint:TestPoint_Pad_D3.0mm, F.Cu at (2.02, 12.1)
- added TP4: TestPoint, TestPoint:TestPoint_Pad_D3.0mm, F.Cu at (2.02, 17.2)
- added TP5: TestPoint, TestPoint:TestPoint_Pad_D3.0mm, F.Cu at (7.08, 2.02)
- added TP6: TestPoint, TestPoint:TestPoint_Pad_D3.0mm, F.Cu at (7.08, 7.08)
- added TP7: TestPoint, TestPoint:TestPoint_Pad_D3.0mm, F.Cu at (7.08, 12.1)
- added TP8: TestPoint, TestPoint:TestPoint_Pad_D3.0mm, F.Cu at (7.08, 17.2)
- added TP9: TestPoint, TestPoint:TestPoint_Pad_D3.0mm, F.Cu at (12.1, 2.02)
- C16, C17, C18, C19, C22, C23, C24, C25, C26, C27, C28, C29, C30, C31, C32, C33, C36, C37, C38, C39, C40, C41, C42, C43, C44, C45, C46, R18, R21, R22, R23: moved to B.Cu
- moved C23 322.8 mm to (183.4, 199.6)
- moved C22 322.5 mm to (183.4, 194.8)
- moved C24 320.9 mm to (183.4, 198.0)
- moved C25 320.2 mm to (183.4, 196.4)
- moved C16 319.1 mm to (178.4, 191.3), turned to 90 degrees
- moved C26 317.8 mm to (180.0, 204.7), turned to -90 degrees
- moved C18 316.8 mm to (176.8, 191.3), turned to 90 degrees
- moved C28 315.4 mm to (178.4, 204.7), turned to -90 degrees
- moved C19 314.8 mm to (175.2, 191.3), turned to 90 degrees
- moved C17 314.0 mm to (173.6, 191.3), turned to 90 degrees
- moved C29 313.4 mm to (176.8, 204.7), turned to -90 degrees
- moved C27 312.7 mm to (175.2, 204.7), turned to -90 degrees
- moved C40 309.5 mm to (180.0, 200.6), turned to 90 degrees
- moved C39 308.5 mm to (178.0, 198.0), turned to 180 degrees
- moved R21 307.8 mm to (183.4, 201.2)
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Connections:
- J10 pad 1: Net-(U4D-IOB_52) -> unconnected-(J10-Pad1)
- J10 pad 10: Net-(U4D-IOB_61) -> unconnected-(J10-Pad10)
- J10 pad 11: Net-(U4D-IOB_63) -> unconnected-(J10-Pad11)
- J10 pad 12: Net-(U4D-IOB_64) -> unconnected-(J10-Pad12)
- J10 pad 13: Net-(U4D-IOB_66) -> unconnected-(J10-Pad13)
- J10 pad 14: Net-(U4D-IOB_67) -> unconnected-(J10-Pad14)
- J10 pad 15: Net-(U4D-IOB_68) -> unconnected-(J10-Pad15)
- J10 pad 16: Net-(U4D-IOB_69) -> unconnected-(J10-Pad16)
- J10 pad 17: Net-(U4D-IOB_71) -> unconnected-(J10-Pad17)
- J10 pad 18: Net-(U4D-IOB_72) -> unconnected-(J10-Pad18)
- J10 pad 19: Net-(U4D-IOB_73) -> unconnected-(J10-Pad19)
- J10 pad 2: Net-(U4D-IOB_53) -> unconnected-(J10-Pad2)
- J10 pad 20: Net-(U4D-IOB_74) -> unconnected-(J10-Pad20)
- J10 pad 21: Net-(U4D-IOB_75) -> unconnected-(J10-Pad21)
- J10 pad 22: Net-(U4D-IOB_76) -> unconnected-(J10-Pad22)
- J10 pad 23: Net-(U4D-IOB_77) -> unconnected-(J10-Pad23)
- J10 pad 24: Net-(U4D-IOB_78) -> unconnected-(J10-Pad24)
- J10 pad 25: Net-(U4D-IOB_79) -> /ICE40HX/ICE_B2_76
- J10 pad 26: Net-(U4D-IOB_80) -> unconnected-(J10-Pad26)
- J10 pad 27: Net-(U4D-IOB_83) -> /ICE40HX/ICE_B2_88
- J10 pad 28: Net-(U4D-IOB_84) -> /ICE40HX/ICE_B2_79
- J10 pad 29: Net-(U4D-IOB_85) -> /ICE40HX/ICE_B2_94
- J10 pad 3: Net-(U4D-IOB_54) -> unconnected-(J10-Pad3)
- J10 pad 30: Net-(U4D-IOB_86) -> /ICE40HX/ICE_B2_89
- J10 pad 31: Net-(U4D-IOB_87) -> /ICE40HX/ICE_B2_91
- J10 pad 32: Net-(U4D-IOB_88) -> /ICE40HX/ICE_B2_92
- J10 pad 33: Net-(U4D-IOB_89) -> unconnected-(J10-Pad33)
- J10 pad 34: Net-(U4D-IOB_91) -> /ICE40HX/ICE_B2_100
- J10 pad 35: Net-(U4D-IOB_92) -> unconnected-(J10-Pad35)
- J10 pad 36: Net-(U4D-IOB_93) -> unconnected-(J10-Pad36)
- J10 pad 37: Net-(U4D-IOB_94) -> unconnected-(J10-Pad37)
- J10 pad 38: Net-(U4D-IOB_98) -> unconnected-(J10-Pad38)
- J10 pad 39: Net-(U4D-IOB_99) -> unconnected-(J10-Pad39)
- J10 pad 4: Net-(U4D-IOB_55) -> unconnected-(J10-Pad4)
- J10 pad 40: Net-(U4D-IOB_100) -> unconnected-(J10-Pad40)
- J10 pad 41: Net-(U4D-IOB_101) -> unconnected-(J10-Pad41)
- J10 pad 42: Net-(U4D-IOB_102) -> unconnected-(J10-Pad42)
- J10 pad 5: Net-(U4D-IOB_56) -> unconnected-(J10-Pad5)
- J10 pad 6: Net-(U4D-IOB_57) -> unconnected-(J10-Pad6)
- J10 pad 7: Net-(U4D-IOB_58) -> unconnected-(J10-Pad7)
- J10 pad 8: Net-(U4D-IOB_59) -> unconnected-(J10-Pad8)
- J10 pad 9: Net-(U4D-IOB_60) -> unconnected-(J10-Pad9)
- U4 pad L10: Net-(U4D-IOB_85) -> unconnected-(U4D-IOB_85-PadL10)
- U4 pad L11: Net-(U4D-IOB_99) -> unconnected-(U4D-IOB_99-PadL11)
- U4 pad L9: Net-(U4D-IOB_74) -> unconnected-(U4D-IOB_74-PadL9)
- U4 pad M11: Net-(U4D-IOB_93) -> unconnected-(U4D-IOB_93-PadM11)
- U4 pad M12: Net-(U4D-IOB_101) -> unconnected-(U4D-IOB_101-PadM12)
- U4 pad M7: Net-(U4D-IOB_64) -> unconnected-(U4D-IOB_64-PadM7)
- U4 pad M8: Net-(U4D-IOB_68) -> unconnected-(U4D-IOB_68-PadM8)
- U4 pad M9: Net-(U4D-IOB_80) -> unconnected-(U4D-IOB_80-PadM9)
- U4 pad N10: Net-(U4D-IOB_87) -> unconnected-(U4D-IOB_87-PadN10)
- U4 pad N12: Net-(U4D-IOB_98) -> unconnected-(U4D-IOB_98-PadN12)
- U4 pad N5: Net-(U4D-IOB_56) -> unconnected-(U4D-IOB_56-PadN5)
- U4 pad N6: Net-(U4D-IOB_52) -> unconnected-(U4D-IOB_52-PadN6)
- U4 pad N7: Net-(U4D-IOB_66) -> unconnected-(U4D-IOB_66-PadN7)
- U4 pad N9: Net-(U4D-IOB_78) -> unconnected-(U4D-IOB_78-PadN9)
- U4 pad P10: Net-(U4D-IOB_86) -> unconnected-(U4D-IOB_86-PadP10)
- U4 pad P4: Net-(U4D-IOB_54) -> unconnected-(U4D-IOB_54-PadP4)
- U4 pad P5: Net-(U4D-IOB_58) -> unconnected-(U4D-IOB_58-PadP5)
- U4 pad P6: Net-(U4D-IOB_67) -> unconnected-(U4D-IOB_67-PadP6)
- U4 pad P7: Net-(U4D-IOB_77) -> unconnected-(U4D-IOB_77-PadP7)
- U4 pad P8: Net-(U4D-IOB_72) -> unconnected-(U4D-IOB_72-PadP8)
- U4 pad P9: Net-(U4D-IOB_83) -> unconnected-(U4D-IOB_83-PadP9)
- U4 pad R10: Net-(U4D-IOB_84) -> unconnected-(U4D-IOB_84-PadR10)
- U4 pad R16: Net-(U4D-IOB_102) -> unconnected-(U4D-IOB_102-PadR16)
- U4 pad R2: Net-(U4D-IOB_55) -> unconnected-(U4D-IOB_55-PadR2)
- U4 pad R3: Net-(U4D-IOB_59) -> unconnected-(U4D-IOB_59-PadR3)
- U4 pad R4: Net-(U4D-IOB_63) -> unconnected-(U4D-IOB_63-PadR4)
- U4 pad R5: Net-(U4D-IOB_60) -> unconnected-(U4D-IOB_60-PadR5)
- U4 pad R6: Net-(U4D-IOB_71) -> unconnected-(U4D-IOB_71-PadR6)
- U4 pad T1: Net-(U4D-IOB_53) -> unconnected-(U4D-IOB_53-PadT1)
- U4 pad T10: Net-(U4D-IOB_88) -> /ICE40HX/ICE_B2_88
- U4 pad T11: Net-(U4D-IOB_89) -> /ICE40HX/ICE_B2_89
- U4 pad T13: Net-(U4D-IOB_94) -> /ICE40HX/ICE_B2_94
- U4 pad T14: Net-(U4D-IOB_92) -> /ICE40HX/ICE_B2_92
- U4 pad T15: Net-(U4D-IOB_91) -> /ICE40HX/ICE_B2_91
- U4 pad T16: Net-(U4D-IOB_100) -> /ICE40HX/ICE_B2_100
- U4 pad T2: Net-(U4D-IOB_57) -> unconnected-(U4D-IOB_57-PadT2)
- U4 pad T3: Net-(U4D-IOB_61) -> unconnected-(U4D-IOB_61-PadT3)
- U4 pad T5: Net-(U4D-IOB_69) -> unconnected-(U4D-IOB_69-PadT5)
- U4 pad T6: Net-(U4D-IOB_73) -> unconnected-(U4D-IOB_73-PadT6)
- U4 pad T7: Net-(U4D-IOB_75) -> unconnected-(U4D-IOB_75-PadT7)
- U4 pad T8: Net-(U4D-IOB_76) -> /ICE40HX/ICE_B2_76
- U4 pad T9: Net-(U4D-IOB_79) -> /ICE40HX/ICE_B2_79
Routing:
- net GND: track 68.8 -> 112.5 mm, vias 22 -> 29
- net /ICE40HX/ICE_B2_100: track 0.00 -> 39.5 mm
- net /ICE40HX/ICE_B2_92: track 0.00 -> 39.1 mm
- net /ICE40HX/ICE_B2_89: track 0.00 -> 39.0 mm
- net /ICE40HX/ICE_B2_79: track 0.00 -> 38.6 mm
- net /ICE40HX/ICE_B2_91: track 0.00 -> 36.2 mm
- net /ICE40HX/ICE_B2_94: track 0.00 -> 35.8 mm
- net /ICE40HX/ICE_B2_88: track 0.00 -> 35.8 mm
- net /ICE40HX/ICE_B2_76: track 0.00 -> 35.7 mm
- net VCCIO0: track 0.57 -> 24.9 mm, vias 1 -> 5
- net VCCIO1: track 0.57 -> 24.5 mm, vias 1 -> 5
- net VCCIO3: track 1.13 -> 25.1 mm, vias 2 -> 6
- net VCCIO2: track 1.13 -> 23.8 mm, vias 2 -> 5
- net +1V2: track 3.90 -> 16.3 mm, vias 4 -> 8
- net +3V3: track 1.66 -> 13.8 mm, vias 0 -> 6
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- added copper zone on In2.Cu, net +1V2
- added copper zone on In2.Cu, net +3V3
- removed copper zone on In2.Cu, net +1V22
- removed copper zone on In2.Cu, net +5V
- removed copper zone on In2.Cu, net VBUS

Commit message: bank 2 done
Connections:
- J10 pad 1: unconnected-(J10-Pad1) -> /ICE40HX/ICE_B2_64
- J10 pad 10: unconnected-(J10-Pad10) -> /ICE40HX/ICE_B2_67
- J10 pad 11: unconnected-(J10-Pad11) -> /ICE40HX/ICE_B2_66
- J10 pad 12: unconnected-(J10-Pad12) -> /ICE40HX/ICE_B2_77
- J10 pad 13: unconnected-(J10-Pad13) -> /ICE40HX/ICE_B2_72
- J10 pad 14: unconnected-(J10-Pad14) -> /ICE40HX/ICE_B2_53
- J10 pad 15: unconnected-(J10-Pad15) -> /ICE40HX/ICE_B2_55
- J10 pad 16: unconnected-(J10-Pad16) -> /ICE40HX/ICE_B2_57
- J10 pad 17: unconnected-(J10-Pad17) -> /ICE40HX/ICE_B2_59
- J10 pad 18: unconnected-(J10-Pad18) -> /ICE40HX/ICE_B2_61
- J10 pad 19: unconnected-(J10-Pad19) -> /ICE40HX/ICE_B2_63
- J10 pad 2: unconnected-(J10-Pad2) -> /ICE40HX/ICE_B2_80
- J10 pad 20: unconnected-(J10-Pad20) -> /ICE40HX/ICE_B2_60
- J10 pad 21: unconnected-(J10-Pad21) -> /ICE40HX/ICE_B2_69
- J10 pad 22: unconnected-(J10-Pad22) -> /ICE40HX/ICE_B2_71
- J10 pad 23: unconnected-(J10-Pad23) -> /ICE40HX/ICE_B2_73
- J10 pad 24: unconnected-(J10-Pad24) -> /ICE40HX/ICE_B2_75
- J10 pad 26: unconnected-(J10-Pad26) -> /ICE40HX/ICE_B2_79
- J10 pad 28: /ICE40HX/ICE_B2_79 -> /ICE40HX/ICE_B2_89
- J10 pad 3: unconnected-(J10-Pad3) -> /ICE40HX/ICE_B2_68
- J10 pad 30: /ICE40HX/ICE_B2_89 -> /ICE40HX/ICE_B2_92
- J10 pad 32: /ICE40HX/ICE_B2_92 -> /ICE40HX/ICE_B2_100
- J10 pad 33: unconnected-(J10-Pad33) -> /ICE40HX/ICE_B2_83
- J10 pad 34: /ICE40HX/ICE_B2_100 -> /ICE40HX/ICE_B2_78
- J10 pad 35: unconnected-(J10-Pad35) -> /ICE40HX/ICE_B2_86
- J10 pad 36: unconnected-(J10-Pad36) -> /ICE40HX/ICE_B2_87
- J10 pad 37: unconnected-(J10-Pad37) -> /ICE40HX/ICE_B2_93
- J10 pad 38: unconnected-(J10-Pad38) -> /ICE40HX/ICE_B2_84
- J10 pad 39: unconnected-(J10-Pad39) -> /ICE40HX/ICE_B2_98
- J10 pad 4: unconnected-(J10-Pad4) -> /ICE40HX/ICE_B2_85
- J10 pad 40: unconnected-(J10-Pad40) -> /ICE40HX/ICE_B2_99
- J10 pad 41: unconnected-(J10-Pad41) -> /ICE40HX/ICE_B2_101
- J10 pad 42: unconnected-(J10-Pad42) -> /ICE40HX/ICE_B2_102
- J10 pad 5: unconnected-(J10-Pad5) -> /ICE40HX/ICE_B2_74
- J10 pad 6: unconnected-(J10-Pad6) -> /ICE40HX/ICE_B2_54
- J10 pad 7: unconnected-(J10-Pad7) -> /ICE40HX/ICE_B2_56
- J10 pad 8: unconnected-(J10-Pad8) -> /ICE40HX/ICE_B2_58
- J10 pad 9: unconnected-(J10-Pad9) -> /ICE40HX/ICE_B2_52
- J11 pad 1: Net-(U4E-IOL_1A) -> unconnected-(J11-Pad1)
- J11 pad 10: Net-(U4E-IOL_5B) -> unconnected-(J11-Pad10)
- J11 pad 11: Net-(U4E-IOL_6A) -> unconnected-(J11-Pad11)
- J11 pad 12: Net-(U4E-IOL_6B) -> unconnected-(J11-Pad12)
- J11 pad 13: Net-(U4E-IOL_7A) -> unconnected-(J11-Pad13)
- J11 pad 14: Net-(U4E-IOL_7B) -> unconnected-(J11-Pad14)
- J11 pad 15: Net-(U4E-IOL_8A) -> unconnected-(J11-Pad15)
- J11 pad 16: Net-(U4E-IOL_8B) -> unconnected-(J11-Pad16)
- J11 pad 17: Net-(U4E-IOL_9A) -> unconnected-(J11-Pad17)
- J11 pad 18: Net-(U4E-IOL_9B) -> unconnected-(J11-Pad18)
- J11 pad 19: Net-(U4E-IOL_10A) -> unconnected-(J11-Pad19)
- J11 pad 2: Net-(U4E-IOL_1B) -> unconnected-(J11-Pad2)
- J11 pad 20: Net-(U4E-IOL_10B) -> unconnected-(J11-Pad20)
- J11 pad 21: Net-(U4E-IOL_11A) -> unconnected-(J11-Pad21)
- J11 pad 22: Net-(U4E-IOL_11B) -> unconnected-(J11-Pad22)
- J11 pad 23: Net-(U4E-IOL_12A) -> unconnected-(J11-Pad23)
- J11 pad 24: Net-(U4E-IOL_12B) -> unconnected-(J11-Pad24)
- J11 pad 25: Net-(U4E-IOL_13A) -> unconnected-(J11-Pad25)
- J11 pad 26: Net-(U4E-IOL_14B) -> unconnected-(J11-Pad26)
- J11 pad 27: Net-(U4E-IOL_15A) -> unconnected-(J11-Pad27)
- J11 pad 28: Net-(U4E-IOL_15B) -> unconnected-(J11-Pad28)
- J11 pad 29: Net-(U4E-IOL_16A) -> unconnected-(J11-Pad29)
- J11 pad 3: Net-(U4E-IOL_2A) -> unconnected-(J11-Pad3)
- J11 pad 30: Net-(U4E-IOL_16B) -> unconnected-(J11-Pad30)
- J11 pad 31: Net-(U4E-IOL_17A) -> unconnected-(J11-Pad31)
- J11 pad 32: Net-(U4E-IOL_17B) -> unconnected-(J11-Pad32)
- J11 pad 33: Net-(U4E-IOL_18A) -> unconnected-(J11-Pad33)
- J11 pad 34: Net-(U4E-IOL_18B) -> unconnected-(J11-Pad34)
- J11 pad 35: Net-(U4E-IOL_19A) -> unconnected-(J11-Pad35)
- J11 pad 36: Net-(U4E-IOL_19B) -> unconnected-(J11-Pad36)
- J11 pad 37: Net-(U4E-IOL_20A) -> unconnected-(J11-Pad37)
- J11 pad 38: Net-(U4E-IOL_20B) -> unconnected-(J11-Pad38)
- J11 pad 39: Net-(U4E-IOL_21A) -> unconnected-(J11-Pad39)
- J11 pad 4: Net-(U4E-IOL_2B) -> unconnected-(J11-Pad4)
- J11 pad 40: Net-(U4E-IOL_21B) -> unconnected-(J11-Pad40)
- J11 pad 41: Net-(U4E-IOL_22A) -> unconnected-(J11-Pad41)
- J11 pad 42: Net-(U4E-IOL_22B) -> unconnected-(J11-Pad42)
- J11 pad 43: Net-(U4E-IOL_23A) -> unconnected-(J11-Pad43)
- J11 pad 44: Net-(U4E-IOL_23B) -> unconnected-(J11-Pad44)
- J11 pad 45: Net-(U4E-IOL_24A) -> unconnected-(J11-Pad45)
- J11 pad 46: Net-(U4E-IOL_24B) -> unconnected-(J11-Pad46)
- J11 pad 47: Net-(U4E-IOL_25A) -> unconnected-(J11-Pad47)
- J11 pad 48: Net-(U4E-IOL_25B) -> unconnected-(J11-Pad48)
- J11 pad 49: Net-(U4E-IOL_26A) -> unconnected-(J11-Pad49)
- J11 pad 5: Net-(U4E-IOL_3A) -> unconnected-(J11-Pad5)
- J11 pad 50: Net-(U4E-IOL_26B) -> unconnected-(J11-Pad50)
- J11 pad 6: Net-(U4E-IOL_3B) -> unconnected-(J11-Pad6)
- J11 pad 7: Net-(U4E-IOL_4A) -> unconnected-(J11-Pad7)
- J11 pad 8: Net-(U4E-IOL_4B) -> unconnected-(J11-Pad8)
- J11 pad 9: Net-(U4E-IOL_5A) -> unconnected-(J11-Pad9)
- J6 pad 1: Net-(U4B-IOT_168) -> unconnected-(J6-Pad1)
- J6 pad 10: Net-(U4B-IOT_178) -> unconnected-(J6-Pad10)
- J6 pad 11: Net-(U4B-IOT_179) -> unconnected-(J6-Pad11)
- J6 pad 12: Net-(U4B-IOT_180) -> unconnected-(J6-Pad12)
- J6 pad 13: Net-(U4B-IOT_181) -> unconnected-(J6-Pad13)
- J6 pad 14: Net-(U4B-IOT_182) -> unconnected-(J6-Pad14)
- J6 pad 15: Net-(U4B-IOT_183) -> unconnected-(J6-Pad15)
- J6 pad 16: Net-(U4B-IOT_184) -> unconnected-(J6-Pad16)
- J6 pad 17: Net-(U4B-IOT_185) -> unconnected-(J6-Pad17)
- J6 pad 18: Net-(U4B-IOT_186) -> unconnected-(J6-Pad18)
- J6 pad 19: Net-(U4B-IOT_187) -> unconnected-(J6-Pad19)
- J6 pad 2: Net-(U4B-IOT_169) -> unconnected-(J6-Pad2)
- J6 pad 20: Net-(U4B-IOT_190) -> unconnected-(J6-Pad20)
- J6 pad 21: Net-(U4B-IOT_191) -> unconnected-(J6-Pad21)
- J6 pad 22: Net-(U4B-IOT_192) -> unconnected-(J6-Pad22)
- J6 pad 23: Net-(U4B-IOT_193) -> unconnected-(J6-Pad23)
- J6 pad 24: Net-(U4B-IOT_194) -> unconnected-(J6-Pad24)
- J6 pad 25: Net-(U4B-IOT_196) -> unconnected-(J6-Pad25)
- J6 pad 26: Net-(U4B-IOT_199) -> unconnected-(J6-Pad26)
- J6 pad 27: Net-(U4B-IOT_200) -> unconnected-(J6-Pad27)
- J6 pad 28: Net-(U4B-IOT_203) -> unconnected-(J6-Pad28)
- J6 pad 29: Net-(U4B-IOT_205) -> unconnected-(J6-Pad29)
- J6 pad 3: Net-(U4B-IOT_170) -> unconnected-(J6-Pad3)
- J6 pad 30: Net-(U4B-IOT_206) -> unconnected-(J6-Pad30)
- J6 pad 31: Net-(U4B-IOT_207) -> unconnected-(J6-Pad31)
- J6 pad 32: Net-(U4B-IOT_208) -> unconnected-(J6-Pad32)
- J6 pad 33: Net-(U4B-IOT_209) -> unconnected-(J6-Pad33)
- J6 pad 34: Net-(U4B-IOT_210) -> unconnected-(J6-Pad34)
- J6 pad 35: Net-(U4B-IOT_211) -> unconnected-(J6-Pad35)
- J6 pad 36: Net-(U4B-IOT_212) -> unconnected-(J6-Pad36)
- J6 pad 37: Net-(U4B-IOT_213) -> unconnected-(J6-Pad37)
- J6 pad 38: Net-(U4B-IOT_214) -> unconnected-(J6-Pad38)
- J6 pad 39: Net-(U4B-IOT_215) -> unconnected-(J6-Pad39)
- J6 pad 4: Net-(U4B-IOT_171) -> unconnected-(J6-Pad4)
- J6 pad 40: Net-(U4B-IOT_216) -> unconnected-(J6-Pad40)
- J6 pad 41: Net-(U4B-IOT_218) -> unconnected-(J6-Pad41)
- J6 pad 42: Net-(U4B-IOT_219) -> unconnected-(J6-Pad42)
- J6 pad 43: Net-(U4B-IOT_220) -> unconnected-(J6-Pad43)
- J6 pad 44: Net-(U4B-IOT_221) -> unconnected-(J6-Pad44)
- J6 pad 45: Net-(U4B-IOT_222) -> unconnected-(J6-Pad45)
- J6 pad 46: Net-(U4B-IOT_223) -> unconnected-(J6-Pad46)
- J6 pad 47: Net-(U4B-IOT_224) -> unconnected-(J6-Pad47)
- J6 pad 48: Net-(U4B-IOT_225) -> unconnected-(J6-Pad48)
- J6 pad 49: Net-(U4B-IOT_226) -> unconnected-(J6-Pad49)
- J6 pad 5: Net-(U4B-IOT_172) -> unconnected-(J6-Pad5)
- J6 pad 50: Net-(U4B-IOT_227) -> unconnected-(J6-Pad50)
- J6 pad 6: Net-(U4B-IOT_173) -> unconnected-(J6-Pad6)
- J6 pad 7: Net-(U4B-IOT_174) -> unconnected-(J6-Pad7)
- J6 pad 8: Net-(U4B-IOT_176) -> unconnected-(J6-Pad8)
- J6 pad 9: Net-(U4B-IOT_177) -> unconnected-(J6-Pad9)
- J9 pad 1: Net-(U4C-IOR_109) -> unconnected-(J9-Pad1)
- J9 pad 10: Net-(U4C-IOR_118) -> unconnected-(J9-Pad10)
- J9 pad 11: Net-(U4C-IOR_119) -> unconnected-(J9-Pad11)
- J9 pad 12: Net-(U4C-IOR_120) -> unconnected-(J9-Pad12)
- J9 pad 13: Net-(U4C-IOR_121) -> unconnected-(J9-Pad13)
- J9 pad 14: Net-(U4C-IOR_122) -> unconnected-(J9-Pad14)
- J9 pad 15: Net-(U4C-IOR_123) -> unconnected-(J9-Pad15)
- J9 pad 16: Net-(U4C-IOR_126) -> unconnected-(J9-Pad16)
- J9 pad 17: Net-(U4C-IOR_127) -> unconnected-(J9-Pad17)
- J9 pad 18: Net-(U4C-IOR_128) -> unconnected-(J9-Pad18)
- J9 pad 19: Net-(U4C-IOR_129) -> unconnected-(J9-Pad19)
- J9 pad 2: Net-(U4C-IOR_110) -> unconnected-(J9-Pad2)
- J9 pad 20: Net-(U4C-IOR_130) -> unconnected-(J9-Pad20)
- J9 pad 21: Net-(U4C-IOR_131) -> unconnected-(J9-Pad21)
- J9 pad 22: Net-(U4C-IOR_133) -> unconnected-(J9-Pad22)
- J9 pad 23: Net-(U4C-IOR_134) -> unconnected-(J9-Pad23)
- J9 pad 24: Net-(U4C-IOR_136) -> unconnected-(J9-Pad24)
- J9 pad 25: Net-(U4C-IOR_137) -> unconnected-(J9-Pad25)
- J9 pad 26: Net-(U4C-IOR_138) -> unconnected-(J9-Pad26)
- J9 pad 27: Net-(U4C-IOR_139) -> unconnected-(J9-Pad27)
- J9 pad 28: Net-(U4C-IOR_142) -> unconnected-(J9-Pad28)
- J9 pad 29: Net-(U4C-IOR_143) -> unconnected-(J9-Pad29)
- J9 pad 3: Net-(U4C-IOR_111) -> unconnected-(J9-Pad3)
- J9 pad 30: Net-(U4C-IOR_144) -> unconnected-(J9-Pad30)
- J9 pad 31: Net-(U4C-IOR_145) -> unconnected-(J9-Pad31)
- J9 pad 32: Net-(U4C-IOR_146) -> unconnected-(J9-Pad32)
- J9 pad 33: Net-(U4C-IOR_147) -> unconnected-(J9-Pad33)
- J9 pad 34: Net-(U4C-IOR_148) -> unconnected-(J9-Pad34)
- J9 pad 35: Net-(U4C-IOR_149) -> unconnected-(J9-Pad35)
- J9 pad 36: Net-(U4C-IOR_150) -> unconnected-(J9-Pad36)
- J9 pad 37: Net-(U4C-IOR_151) -> unconnected-(J9-Pad37)
- J9 pad 38: Net-(U4C-IOR_152) -> unconnected-(J9-Pad38)
- J9 pad 39: Net-(U4C-IOR_153) -> unconnected-(J9-Pad39)
- J9 pad 4: Net-(U4C-IOR_112) -> unconnected-(J9-Pad4)
- J9 pad 40: Net-(U4C-IOR_154) -> unconnected-(J9-Pad40)
- J9 pad 41: Net-(U4C-IOR_155) -> unconnected-(J9-Pad41)
- J9 pad 42: Net-(U4C-IOR_156) -> unconnected-(J9-Pad42)
- J9 pad 43: Net-(U4C-IOR_157) -> unconnected-(J9-Pad43)
- J9 pad 44: Net-(U4C-IOR_158) -> unconnected-(J9-Pad44)
- J9 pad 45: Net-(U4C-IOR_160) -> unconnected-(J9-Pad45)
- J9 pad 46: Net-(U4C-IOR_161) -> unconnected-(J9-Pad46)
- J9 pad 47: Net-(U4C-IOR_162) -> unconnected-(J9-Pad47)
- J9 pad 48: Net-(U4C-IOR_165) -> unconnected-(J9-Pad48)
- J9 pad 49: Net-(U4C-IOR_166) -> unconnected-(J9-Pad49)
- J9 pad 5: Net-(U4C-IOR_113) -> unconnected-(J9-Pad5)
- J9 pad 50: Net-(U4C-IOR_167) -> unconnected-(J9-Pad50)
- J9 pad 6: Net-(U4C-IOR_114) -> unconnected-(J9-Pad6)
- J9 pad 7: Net-(U4C-IOR_115) -> unconnected-(J9-Pad7)
- J9 pad 8: Net-(U4C-IOR_116) -> unconnected-(J9-Pad8)
- J9 pad 9: Net-(U4C-IOR_117) -> unconnected-(J9-Pad9)
- U4 pad A1: Net-(U4B-IOT_220) -> unconnected-(U4B-IOT_220-PadA1)
- U4 pad A10: Net-(U4B-IOT_186) -> unconnected-(U4B-IOT_186-PadA10)
- U4 pad A11: Net-(U4B-IOT_187) -> unconnected-(U4B-IOT_187-PadA11)
- U4 pad A15: Net-(U4B-IOT_177) -> unconnected-(U4B-IOT_177-PadA15)
- U4 pad A16: Net-(U4B-IOT_176) -> unconnected-(U4B-IOT_176-PadA16)
- U4 pad A2: Net-(U4B-IOT_218) -> unconnected-(U4B-IOT_218-PadA2)
- U4 pad A5: Net-(U4B-IOT_213) -> unconnected-(U4B-IOT_213-PadA5)
- U4 pad A6: Net-(U4B-IOT_211) -> unconnected-(U4B-IOT_211-PadA6)
- U4 pad A7: Net-(U4B-IOT_205) -> unconnected-(U4B-IOT_205-PadA7)
- U4 pad A9: Net-(U4B-IOT_194) -> unconnected-(U4B-IOT_194-PadA9)
- U4 pad B1: Net-(U4E-IOL_2B) -> unconnected-(U4E-IOL_2B-PadB1)
- U4 pad B10: Net-(U4B-IOT_183) -> unconnected-(U4B-IOT_183-PadB10)
- U4 pad B11: Net-(U4B-IOT_184) -> unconnected-(U4B-IOT_184-PadB11)
- U4 pad B12: Net-(U4B-IOT_182) -> unconnected-(U4B-IOT_182-PadB12)
- U4 pad B13: Net-(U4B-IOT_178) -> unconnected-(U4B-IOT_178-PadB13)
- U4 pad B14: Net-(U4B-IOT_171) -> unconnected-(U4B-IOT_171-PadB14)
- U4 pad B15: Net-(U4B-IOT_169) -> unconnected-(U4B-IOT_169-PadB15)
- U4 pad B16: Net-(U4C-IOR_165) -> unconnected-(U4C-IOR_165-PadB16)
- U4 pad B2: Net-(U4E-IOL_1B) -> unconnected-(U4E-IOL_1B-PadB2)
- U4 pad B3: Net-(U4B-IOT_223) -> unconnected-(U4B-IOT_223-PadB3)
- U4 pad B4: Net-(U4B-IOT_216) -> unconnected-(U4B-IOT_216-PadB4)
- U4 pad B5: Net-(U4B-IOT_214) -> unconnected-(U4B-IOT_214-PadB5)
- U4 pad B6: Net-(U4B-IOT_208) -> unconnected-(U4B-IOT_208-PadB6)
- U4 pad B7: Net-(U4B-IOT_207) -> unconnected-(U4B-IOT_207-PadB7)
- U4 pad B8: Net-(U4B-IOT_203) -> unconnected-(U4B-IOT_203-PadB8)
- U4 pad B9: Net-(U4B-IOT_199) -> unconnected-(U4B-IOT_199-PadB9)
- U4 pad C1: Net-(U4E-IOL_3A) -> unconnected-(U4E-IOL_3A-PadC1)
- U4 pad C10: Net-(U4B-IOT_185) -> unconnected-(U4B-IOT_185-PadC10)
- U4 pad C11: Net-(U4B-IOT_180) -> unconnected-(U4B-IOT_180-PadC11)
- U4 pad C12: Net-(U4B-IOT_172) -> unconnected-(U4B-IOT_172-PadC12)
- U4 pad C13: Net-(U4B-IOT_174) -> unconnected-(U4B-IOT_174-PadC13)
- U4 pad C14: Net-(U4B-IOT_168) -> unconnected-(U4B-IOT_168-PadC14)
- U4 pad C16: Net-(U4C-IOR_161) -> unconnected-(U4C-IOR_161-PadC16)
- U4 pad C2: Net-(U4E-IOL_3B) -> unconnected-(U4E-IOL_3B-PadC2)
- U4 pad C3: Net-(U4B-IOT_227) -> unconnected-(U4B-IOT_227-PadC3)
- U4 pad C4: Net-(U4B-IOT_222) -> unconnected-(U4B-IOT_222-PadC4)
- U4 pad C5: Net-(U4B-IOT_221) -> unconnected-(U4B-IOT_221-PadC5)
- U4 pad C6: Net-(U4B-IOT_209) -> unconnected-(U4B-IOT_209-PadC6)
- U4 pad C7: Net-(U4B-IOT_206) -> unconnected-(U4B-IOT_206-PadC7)
- U4 pad C9: Net-(U4B-IOT_191) -> unconnected-(U4B-IOT_191-PadC9)
- U4 pad D1: Net-(U4E-IOL_5B) -> unconnected-(U4E-IOL_5B-PadD1)
- U4 pad D10: Net-(U4B-IOT_190) -> unconnected-(U4B-IOT_190-PadD10)
- U4 pad D11: Net-(U4B-IOT_181) -> unconnected-(U4B-IOT_181-PadD11)
- U4 pad D13: Net-(U4B-IOT_170) -> unconnected-(U4B-IOT_170-PadD13)
- U4 pad D14: Net-(U4C-IOR_167) -> unconnected-(U4C-IOR_167-PadD14)
- U4 pad D15: Net-(U4C-IOR_157) -> unconnected-(U4C-IOR_157-PadD15)
- U4 pad D16: Net-(U4C-IOR_153) -> unconnected-(U4C-IOR_153-PadD16)
- U4 pad D2: Net-(U4E-IOL_4B) -> unconnected-(U4E-IOL_4B-PadD2)
- U4 pad D3: Net-(U4B-IOT_226) -> unconnected-(U4B-IOT_226-PadD3)
- U4 pad D4: Net-(U4B-IOT_224) -> unconnected-(U4B-IOT_224-PadD4)
- U4 pad D5: Net-(U4B-IOT_219) -> unconnected-(U4B-IOT_219-PadD5)
- U4 pad D6: Net-(U4B-IOT_212) -> unconnected-(U4B-IOT_212-PadD6)
- U4 pad D7: Net-(U4B-IOT_210) -> unconnected-(U4B-IOT_210-PadD7)
- U4 pad D8: Net-(U4B-IOT_200) -> unconnected-(U4B-IOT_200-PadD8)
- U4 pad D9: Net-(U4B-IOT_193) -> unconnected-(U4B-IOT_193-PadD9)
- U4 pad E10: Net-(U4B-IOT_179) -> unconnected-(U4B-IOT_179-PadE10)
- U4 pad E11: Net-(U4B-IOT_173) -> unconnected-(U4B-IOT_173-PadE11)
- U4 pad E13: Net-(U4C-IOR_166) -> unconnected-(U4C-IOR_166-PadE13)
- U4 pad E14: Net-(U4C-IOR_160) -> unconnected-(U4C-IOR_160-PadE14)
- U4 pad E16: Net-(U4C-IOR_151) -> unconnected-(U4C-IOR_151-PadE16)
- U4 pad E2: Net-(U4E-IOL_7B) -> unconnected-(U4E-IOL_7B-PadE2)
- U4 pad E3: Net-(U4E-IOL_6B) -> unconnected-(U4E-IOL_6B-PadE3)
- U4 pad E4: Net-(U4E-IOL_1A) -> unconnected-(U4E-IOL_1A-PadE4)
- U4 pad E5: Net-(U4B-IOT_225) -> unconnected-(U4B-IOT_225-PadE5)
- U4 pad E6: Net-(U4B-IOT_215) -> unconnected-(U4B-IOT_215-PadE6)
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Routing:
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