File: FuseBox/FUSEBOX.kicad_pcb (KiCad board)
At the start: 6 copper layers, 411.7 x 161.7 mm, 187 parts, among them J1 UJ31CHG2SMTTR, J10 901301150, J11 901301150, J12 901301240, J2 702462004, J3 702462004, J4 702462004, J5 702462004, J6 901301150, J7 702462004, J8 61301611121, J9 901301150, U1 TPS61040DBVR, U10 EC11E183440C, U11 EC11E183440C, U12 EC11E183440C, U13 EC11E183440C, U14 EC11E183440C, U2 LT3030EFETRPBF, U3 STM32F407VGTx, U4 ICE40HX8KCT256, U5 EC11E183440C, U6 EC11E183440C, U7 EC11E183440C, U8 EC11E183440C, U9 EC11E183440C, X1 STDCSU18M

Commit message: bank L done
Parts:
- removed +12V, +1V2, +1V22, +3V3, +3V31, +5V, GND, TP14, TP15, TP22, TP23, VBUS, VCC_12V, VCC_1V2, VCC_3V3: TestPoint, TestPoint:TestPoint_Pad_D3.0mm
Connections:
- J11 pad 1: unconnected-(J11-Pad1) -> /ICE40HX/ICE_B3_2A
- J11 pad 10: unconnected-(J11-Pad10) -> /ICE40HX/ICE_B3_8A
- J11 pad 11: unconnected-(J11-Pad11) -> /ICE40HX/ICE_B3_11A
- J11 pad 12: unconnected-(J11-Pad12) -> /ICE40HX/ICE_B3_9A
- J11 pad 13: unconnected-(J11-Pad13) -> /ICE40HX/ICE_B3_1B
- J11 pad 14: unconnected-(J11-Pad14) -> /ICE40HX/ICE_B3_2B
- J11 pad 15: unconnected-(J11-Pad15) -> /ICE40HX/ICE_B3_3B
- J11 pad 16: unconnected-(J11-Pad16) -> /ICE40HX/ICE_B3_3A
- J11 pad 17: unconnected-(J11-Pad17) -> /ICE40HX/ICE_B3_4B
- J11 pad 18: unconnected-(J11-Pad18) -> /ICE40HX/ICE_B3_5B
- J11 pad 19: unconnected-(J11-Pad19) -> /ICE40HX/ICE_B3_7B
- J11 pad 2: unconnected-(J11-Pad2) -> /ICE40HX/ICE_B3_4A
- J11 pad 20: unconnected-(J11-Pad20) -> /ICE40HX/ICE_B3_9B
- J11 pad 21: unconnected-(J11-Pad21) -> /ICE40HX/ICE_B3_10B
- J11 pad 22: unconnected-(J11-Pad22) -> /ICE40HX/ICE_B3_11B
- J11 pad 23: unconnected-(J11-Pad23) -> /ICE40HX/ICE_B3_12B
- J11 pad 24: unconnected-(J11-Pad24) -> /ICE40HX/ICE_B3_14B
- J11 pad 25: unconnected-(J11-Pad25) -> /ICE40HX/ICE_B3_15A
- J11 pad 26: unconnected-(J11-Pad26) -> /ICE40HX/ICE_B3_15B
- J11 pad 27: unconnected-(J11-Pad27) -> /ICE40HX/ICE_B3_17B
- J11 pad 28: unconnected-(J11-Pad28) -> /ICE40HX/ICE_B3_16A
- J11 pad 29: unconnected-(J11-Pad29) -> /ICE40HX/ICE_B3_20B
- J11 pad 3: unconnected-(J11-Pad3) -> /ICE40HX/ICE_B3_5A
- J11 pad 30: unconnected-(J11-Pad30) -> /ICE40HX/ICE_B3_18B
- J11 pad 31: unconnected-(J11-Pad31) -> /ICE40HX/ICE_B3_24A
- J11 pad 32: unconnected-(J11-Pad32) -> /ICE40HX/ICE_B3_21B
- J11 pad 33: unconnected-(J11-Pad33) -> /ICE40HX/ICE_B3_26A
- J11 pad 34: unconnected-(J11-Pad34) -> /ICE40HX/ICE_B3_25A
- J11 pad 35: unconnected-(J11-Pad35) -> /ICE40HX/ICE_B3_12A
- J11 pad 36: unconnected-(J11-Pad36) -> /ICE40HX/ICE_B3_10A
- J11 pad 37: unconnected-(J11-Pad37) -> /ICE40HX/ICE_B3_16B
- J11 pad 38: unconnected-(J11-Pad38) -> /ICE40HX/ICE_B3_13A
- J11 pad 39: unconnected-(J11-Pad39) -> /ICE40HX/ICE_B3_19B
- J11 pad 4: unconnected-(J11-Pad4) -> /ICE40HX/ICE_B3_7A
- J11 pad 40: unconnected-(J11-Pad40) -> /ICE40HX/ICE_B3_18A
- J11 pad 41: unconnected-(J11-Pad41) -> /ICE40HX/ICE_B3_22B
- J11 pad 42: unconnected-(J11-Pad42) -> /ICE40HX/ICE_B3_17A
- J11 pad 43: unconnected-(J11-Pad43) -> /ICE40HX/ICE_B3_26B
- J11 pad 44: unconnected-(J11-Pad44) -> /ICE40HX/ICE_B3_23B
- J11 pad 45: unconnected-(J11-Pad45) -> /ICE40HX/ICE_B3_23A
- J11 pad 46: unconnected-(J11-Pad46) -> /ICE40HX/ICE_B3_19A
- J11 pad 47: unconnected-(J11-Pad47) -> /ICE40HX/ICE_B3_25B
- J11 pad 48: unconnected-(J11-Pad48) -> /ICE40HX/ICE_B3_24B
- J11 pad 49: unconnected-(J11-Pad49) -> /ICE40HX/ICE_B3_21A
- J11 pad 5: unconnected-(J11-Pad5) -> /ICE40HX/ICE_B3_20A
- J11 pad 50: unconnected-(J11-Pad50) -> /ICE40HX/ICE_B3_22A
- J11 pad 6: unconnected-(J11-Pad6) -> /ICE40HX/ICE_B3_1A
- J11 pad 7: unconnected-(J11-Pad7) -> /ICE40HX/ICE_B3_6B
- J11 pad 8: unconnected-(J11-Pad8) -> /ICE40HX/ICE_B3_8B
- J11 pad 9: unconnected-(J11-Pad9) -> /ICE40HX/ICE_B3_6A
- U4 pad B1: unconnected-(U4E-IOL_2B-PadB1) -> /ICE40HX/ICE_B3_2B
- U4 pad B2: unconnected-(U4E-IOL_1B-PadB2) -> /ICE40HX/ICE_B3_1B
- U4 pad C1: unconnected-(U4E-IOL_3A-PadC1) -> /ICE40HX/ICE_B3_3A
- U4 pad C2: unconnected-(U4E-IOL_3B-PadC2) -> /ICE40HX/ICE_B3_3B
- U4 pad D1: unconnected-(U4E-IOL_5B-PadD1) -> /ICE40HX/ICE_B3_5B
- U4 pad D2: unconnected-(U4E-IOL_4B-PadD2) -> /ICE40HX/ICE_B3_4B
- U4 pad E2: unconnected-(U4E-IOL_7B-PadE2) -> /ICE40HX/ICE_B3_7B
- U4 pad E3: unconnected-(U4E-IOL_6B-PadE3) -> /ICE40HX/ICE_B3_6B
- U4 pad E4: unconnected-(U4E-IOL_1A-PadE4) -> /ICE40HX/ICE_B3_1A
- U4 pad F1: unconnected-(U4E-IOL_10B-PadF1) -> /ICE40HX/ICE_B3_10B
- U4 pad F2: unconnected-(U4E-IOL_9B-PadF2) -> /ICE40HX/ICE_B3_9B
- U4 pad F3: unconnected-(U4E-IOL_8B-PadF3) -> /ICE40HX/ICE_B3_8B
- U4 pad F4: unconnected-(U4E-IOL_4A-PadF4) -> /ICE40HX/ICE_B3_4A
- U4 pad F5: unconnected-(U4E-IOL_2A-PadF5) -> /ICE40HX/ICE_B3_2A
- U4 pad G2: unconnected-(U4E-IOL_11B-PadG2) -> /ICE40HX/ICE_B3_11B
- U4 pad G3: unconnected-(U4E-IOL_8A-PadG3) -> /ICE40HX/ICE_B3_8A
- U4 pad G4: unconnected-(U4E-IOL_6A-PadG4) -> /ICE40HX/ICE_B3_6A
- U4 pad G5: unconnected-(U4E-IOL_5A-PadG5) -> /ICE40HX/ICE_B3_5A
- U4 pad H1: unconnected-(U4E-IOL_14B-PadH1) -> /ICE40HX/ICE_B3_14B
- U4 pad H2: unconnected-(U4E-IOL_12B-PadH2) -> /ICE40HX/ICE_B3_12B
- U4 pad H3: unconnected-(U4E-IOL_9A-PadH3) -> /ICE40HX/ICE_B3_9A
- U4 pad H4: unconnected-(U4E-IOL_11A-PadH4) -> /ICE40HX/ICE_B3_11A
- U4 pad H5: unconnected-(U4E-IOL_7A-PadH5) -> /ICE40HX/ICE_B3_7A
- U4 pad H6: unconnected-(U4E-IOL_10A-PadH6) -> /ICE40HX/ICE_B3_10A
- U4 pad J1: unconnected-(U4E-IOL_15B-PadJ1) -> /ICE40HX/ICE_B3_15B
- U4 pad J2: unconnected-(U4E-IOL_15A-PadJ2) -> /ICE40HX/ICE_B3_15A
- U4 pad J4: unconnected-(U4E-IOL_12A-PadJ4) -> /ICE40HX/ICE_B3_12A
- U4 pad J5: unconnected-(U4E-IOL_13A-PadJ5) -> /ICE40HX/ICE_B3_13A
- U4 pad K1: unconnected-(U4E-IOL_16A-PadK1) -> /ICE40HX/ICE_B3_16A
- U4 pad K3: unconnected-(U4E-IOL_16B-PadK3) -> /ICE40HX/ICE_B3_16B
- U4 pad K4: unconnected-(U4E-IOL_18A-PadK4) -> /ICE40HX/ICE_B3_18A
- U4 pad K5: unconnected-(U4E-IOL_20A-PadK5) -> /ICE40HX/ICE_B3_20A
- U4 pad L1: unconnected-(U4E-IOL_17B-PadL1) -> /ICE40HX/ICE_B3_17B
- U4 pad L3: unconnected-(U4E-IOL_19B-PadL3) -> /ICE40HX/ICE_B3_19B
- U4 pad L4: unconnected-(U4E-IOL_17A-PadL4) -> /ICE40HX/ICE_B3_17A
- U4 pad L5: unconnected-(U4E-IOL_23A-PadL5) -> /ICE40HX/ICE_B3_23A
- U4 pad L6: unconnected-(U4E-IOL_19A-PadL6) -> /ICE40HX/ICE_B3_19A
- U4 pad L7: unconnected-(U4E-IOL_21A-PadL7) -> /ICE40HX/ICE_B3_21A
- U4 pad M1: unconnected-(U4E-IOL_18B-PadM1) -> /ICE40HX/ICE_B3_18B
- U4 pad M2: unconnected-(U4E-IOL_20B-PadM2) -> /ICE40HX/ICE_B3_20B
- U4 pad M3: unconnected-(U4E-IOL_22B-PadM3) -> /ICE40HX/ICE_B3_22B
- U4 pad M4: unconnected-(U4E-IOL_24B-PadM4) -> /ICE40HX/ICE_B3_24B
- U4 pad M5: unconnected-(U4E-IOL_25B-PadM5) -> /ICE40HX/ICE_B3_25B
- U4 pad M6: unconnected-(U4E-IOL_22A-PadM6) -> /ICE40HX/ICE_B3_22A
- U4 pad N2: unconnected-(U4E-IOL_21B-PadN2) -> /ICE40HX/ICE_B3_21B
- U4 pad N3: unconnected-(U4E-IOL_23B-PadN3) -> /ICE40HX/ICE_B3_23B
- U4 pad N4: unconnected-(U4E-IOL_26B-PadN4) -> /ICE40HX/ICE_B3_26B
- U4 pad P1: unconnected-(U4E-IOL_24A-PadP1) -> /ICE40HX/ICE_B3_24A
- U4 pad P2: unconnected-(U4E-IOL_25A-PadP2) -> /ICE40HX/ICE_B3_25A
- U4 pad R1: unconnected-(U4E-IOL_26A-PadR1) -> /ICE40HX/ICE_B3_26A
Routing:
- net /ICE40HX/ICE_B3_22A: track 0.00 -> 53.3 mm, vias 0 -> 1
- net /ICE40HX/ICE_B3_21A: track 0.00 -> 52.4 mm, vias 0 -> 1
- net /ICE40HX/ICE_B3_19A: track 0.00 -> 52.1 mm, vias 0 -> 1
- net /ICE40HX/ICE_B3_7A: track 0.00 -> 51.2 mm, vias 0 -> 1
- net /ICE40HX/ICE_B3_24B: track 0.00 -> 51.0 mm, vias 0 -> 1
- net /ICE40HX/ICE_B3_4A: track 0.00 -> 50.8 mm, vias 0 -> 1
- net /ICE40HX/ICE_B3_25B: track 0.00 -> 49.6 mm, vias 0 -> 1
- net /ICE40HX/ICE_B3_20A: track 0.00 -> 49.3 mm, vias 0 -> 1
- net /ICE40HX/ICE_B3_2A: track 0.00 -> 49.1 mm, vias 0 -> 1
- net /ICE40HX/ICE_B3_5A: track 0.00 -> 48.7 mm, vias 0 -> 1
- net /ICE40HX/ICE_B3_1A: track 0.00 -> 48.4 mm, vias 0 -> 1
- net /ICE40HX/ICE_B3_23A: track 0.00 -> 48.3 mm, vias 0 -> 1
- net /ICE40HX/ICE_B3_17A: track 0.00 -> 47.8 mm, vias 0 -> 1
- net /ICE40HX/ICE_B3_10A: track 0.00 -> 47.6 mm, vias 0 -> 1
- net /ICE40HX/ICE_B3_23B: track 0.00 -> 47.4 mm, vias 0 -> 1
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