File: FuseBox/FUSEBOX.kicad_pcb (KiCad board)
At the start: 6 copper layers, 411.7 x 161.7 mm, 172 parts, among them J1 UJ31CHG2SMTTR, J10 901301150, J11 901301150, J12 901301240, J2 702462004, J3 702462004, J4 702462004, J5 702462004, J6 901301150, J7 702462004, J8 61301611121, J9 901301150, U1 TPS61040DBVR, U10 EC11E183440C, U11 EC11E183440C, U12 EC11E183440C, U13 EC11E183440C, U14 EC11E183440C, U2 LT3030EFETRPBF, U3 STM32F407VGTx, U4 ICE40HX8KCT256, U5 EC11E183440C, U6 EC11E183440C, U7 EC11E183440C, U8 EC11E183440C, U9 EC11E183440C, X1 STDCSU18M

Commit message: more traces
Connections:
- J10 pad 2: /ICE40HX/ICE_B2_80 -> /ICE40HX/ICE_B2_68
- J10 pad 28: /ICE40HX/ICE_B2_89 -> /ICE40HX/ICE_B2_84
- J10 pad 3: /ICE40HX/ICE_B2_68 -> /ICE40HX/ICE_B2_80
- J10 pad 30: /ICE40HX/ICE_B2_92 -> /ICE40HX/ICE_B2_89
- J10 pad 32: /ICE40HX/ICE_B2_100 -> /ICE40HX/ICE_B2_92
- J10 pad 33: /ICE40HX/ICE_B2_83 -> /ICE40HX/ICE_B2_102
- J10 pad 34: /ICE40HX/ICE_B2_78 -> /ICE40HX/ICE_B2_100
- J10 pad 35: /ICE40HX/ICE_B2_86 -> /ICE40HX/ICE_B2_78
- J10 pad 36: /ICE40HX/ICE_B2_87 -> /ICE40HX/ICE_B2_83
- J10 pad 37: /ICE40HX/ICE_B2_93 -> /ICE40HX/ICE_B2_87
- J10 pad 38: /ICE40HX/ICE_B2_84 -> /ICE40HX/ICE_B2_86
- J10 pad 39: /ICE40HX/ICE_B2_98 -> /ICE40HX/ICE_B2_99
- J10 pad 4: /ICE40HX/ICE_B2_85 -> /ICE40HX/ICE_B2_74
- J10 pad 40: /ICE40HX/ICE_B2_99 -> /ICE40HX/ICE_B2_93
- J10 pad 42: /ICE40HX/ICE_B2_102 -> /ICE40HX/ICE_B2_98
- J10 pad 5: /ICE40HX/ICE_B2_74 -> /ICE40HX/ICE_B2_85
- J6 pad 13: unconnected-(J6-Pad13) -> /ICE40HX/ICE_T_176
- J6 pad 14: unconnected-(J6-Pad14) -> /ICE40HX/ICE_T_169
- J6 pad 15: unconnected-(J6-Pad15) -> /ICE40HX/ICE_T_177
- J6 pad 16: unconnected-(J6-Pad16) -> /ICE40HX/ICE_T_171
- J6 pad 17: unconnected-(J6-Pad17) -> /ICE40HX/ICE_T_178
- J6 pad 18: unconnected-(J6-Pad18) -> /ICE40HX/ICE_T_182
- J6 pad 19: unconnected-(J6-Pad19) -> /ICE40HX/ICE_T_184
- J6 pad 20: unconnected-(J6-Pad20) -> /ICE40HX/ICE_T_187
- J6 pad 21: unconnected-(J6-Pad21) -> /ICE40HX/ICE_T_183
- J6 pad 22: unconnected-(J6-Pad22) -> /ICE40HX/ICE_T_186
- J6 pad 23: unconnected-(J6-Pad23) -> /ICE40HX/ICE_T_199
- J6 pad 24: unconnected-(J6-Pad24) -> /ICE40HX/ICE_T_194
- J6 pad 25: unconnected-(J6-Pad25) -> /ICE40HX/ICE_T_200
- J6 pad 26: unconnected-(J6-Pad26) -> /ICE40HX/ICE_T_203
- J6 pad 27: unconnected-(J6-Pad27) -> /ICE40HX/ICE_T_207
- J6 pad 28: unconnected-(J6-Pad28) -> /ICE40HX/ICE_T_205
- J6 pad 29: unconnected-(J6-Pad29) -> /ICE40HX/ICE_T_208
- J6 pad 30: unconnected-(J6-Pad30) -> /ICE40HX/ICE_T_211
- J6 pad 31: unconnected-(J6-Pad31) -> /ICE40HX/ICE_T_214
- J6 pad 32: unconnected-(J6-Pad32) -> /ICE40HX/ICE_T_213
- J6 pad 33: unconnected-(J6-Pad33) -> /ICE40HX/ICE_T_223
- J6 pad 34: unconnected-(J6-Pad34) -> /ICE40HX/ICE_T_216
- J6 pad 35: unconnected-(J6-Pad35) -> /ICE40HX/ICE_T_220
- J6 pad 36: unconnected-(J6-Pad36) -> /ICE40HX/ICE_T_218
- J9 pad 16: unconnected-(J9-Pad16) -> /ICE40HX/ICE_R_112
- J9 pad 17: unconnected-(J9-Pad17) -> /ICE40HX/ICE_R_113
- J9 pad 18: unconnected-(J9-Pad18) -> /ICE40HX/ICE_R_117
- J9 pad 19: unconnected-(J9-Pad19) -> /ICE40HX/ICE_R_123
- J9 pad 20: unconnected-(J9-Pad20) -> /ICE40HX/ICE_R_121
- J9 pad 21: unconnected-(J9-Pad21) -> /ICE40HX/ICE_R_119
- J9 pad 22: unconnected-(J9-Pad22) -> /ICE40HX/ICE_R_127
- J9 pad 23: unconnected-(J9-Pad23) -> /ICE40HX/ICE_R_131
- J9 pad 24: unconnected-(J9-Pad24) -> /ICE40HX/ICE_R_133
- J9 pad 25: unconnected-(J9-Pad25) -> /ICE40HX/ICE_R_130
- J9 pad 26: unconnected-(J9-Pad26) -> /ICE40HX/ICE_R_138
- J9 pad 27: unconnected-(J9-Pad27) -> /ICE40HX/ICE_R_145
- J9 pad 28: unconnected-(J9-Pad28) -> /ICE40HX/ICE_R_143
- J9 pad 29: unconnected-(J9-Pad29) -> /ICE40HX/ICE_R_149
- J9 pad 30: unconnected-(J9-Pad30) -> /ICE40HX/ICE_R_147
- J9 pad 31: unconnected-(J9-Pad31) -> /ICE40HX/ICE_R_160
- J9 pad 32: unconnected-(J9-Pad32) -> /ICE40HX/ICE_R_151
- J9 pad 33: unconnected-(J9-Pad33) -> /ICE40HX/ICE_R_157
- J9 pad 34: unconnected-(J9-Pad34) -> /ICE40HX/ICE_R_153
- J9 pad 35: unconnected-(J9-Pad35) -> /ICE40HX/ICE_R_165
- J9 pad 36: unconnected-(J9-Pad36) -> /ICE40HX/ICE_R_161
- U4 pad A1: unconnected-(U4B-IOT_220-PadA1) -> /ICE40HX/ICE_T_220
- U4 pad A10: unconnected-(U4B-IOT_186-PadA10) -> /ICE40HX/ICE_T_186
- U4 pad A11: unconnected-(U4B-IOT_187-PadA11) -> /ICE40HX/ICE_T_187
- U4 pad A15: unconnected-(U4B-IOT_177-PadA15) -> /ICE40HX/ICE_T_177
- U4 pad A16: unconnected-(U4B-IOT_176-PadA16) -> /ICE40HX/ICE_T_176
- U4 pad A2: unconnected-(U4B-IOT_218-PadA2) -> /ICE40HX/ICE_T_218
- U4 pad A5: unconnected-(U4B-IOT_213-PadA5) -> /ICE40HX/ICE_T_213
- U4 pad A6: unconnected-(U4B-IOT_211-PadA6) -> /ICE40HX/ICE_T_211
- U4 pad A7: unconnected-(U4B-IOT_205-PadA7) -> /ICE40HX/ICE_T_205
- U4 pad A9: unconnected-(U4B-IOT_194-PadA9) -> /ICE40HX/ICE_T_194
- U4 pad B10: unconnected-(U4B-IOT_183-PadB10) -> /ICE40HX/ICE_T_183
- U4 pad B11: unconnected-(U4B-IOT_184-PadB11) -> /ICE40HX/ICE_T_184
- U4 pad B12: unconnected-(U4B-IOT_182-PadB12) -> /ICE40HX/ICE_T_182
- U4 pad B13: unconnected-(U4B-IOT_178-PadB13) -> /ICE40HX/ICE_T_178
- U4 pad B14: unconnected-(U4B-IOT_171-PadB14) -> /ICE40HX/ICE_T_171
- U4 pad B15: unconnected-(U4B-IOT_169-PadB15) -> /ICE40HX/ICE_T_169
- U4 pad B16: unconnected-(U4C-IOR_165-PadB16) -> /ICE40HX/ICE_R_165
- U4 pad B3: unconnected-(U4B-IOT_223-PadB3) -> /ICE40HX/ICE_T_223
- U4 pad B4: unconnected-(U4B-IOT_216-PadB4) -> /ICE40HX/ICE_T_216
- U4 pad B5: unconnected-(U4B-IOT_214-PadB5) -> /ICE40HX/ICE_T_214
- U4 pad B6: unconnected-(U4B-IOT_208-PadB6) -> /ICE40HX/ICE_T_208
- U4 pad B7: unconnected-(U4B-IOT_207-PadB7) -> /ICE40HX/ICE_T_207
- U4 pad B8: unconnected-(U4B-IOT_203-PadB8) -> /ICE40HX/ICE_T_203
- U4 pad B9: unconnected-(U4B-IOT_199-PadB9) -> /ICE40HX/ICE_T_199
- U4 pad C16: unconnected-(U4C-IOR_161-PadC16) -> /ICE40HX/ICE_R_161
- U4 pad D15: unconnected-(U4C-IOR_157-PadD15) -> /ICE40HX/ICE_R_157
- U4 pad D16: unconnected-(U4C-IOR_153-PadD16) -> /ICE40HX/ICE_R_153
- U4 pad D8: unconnected-(U4B-IOT_200-PadD8) -> /ICE40HX/ICE_T_200
- U4 pad E14: unconnected-(U4C-IOR_160-PadE14) -> /ICE40HX/ICE_R_160
- U4 pad E16: unconnected-(U4C-IOR_151-PadE16) -> /ICE40HX/ICE_R_151
- U4 pad F15: unconnected-(U4C-IOR_149-PadF15) -> /ICE40HX/ICE_R_149
- U4 pad F16: unconnected-(U4C-IOR_147-PadF16) -> /ICE40HX/ICE_R_147
- U4 pad G15: unconnected-(U4C-IOR_145-PadG15) -> /ICE40HX/ICE_R_145
- U4 pad G16: unconnected-(U4C-IOR_143-PadG16) -> /ICE40HX/ICE_R_143
- U4 pad J15: unconnected-(U4C-IOR_130-PadJ15) -> /ICE40HX/ICE_R_130
- U4 pad J16: unconnected-(U4C-IOR_138-PadJ16) -> /ICE40HX/ICE_R_138
- U4 pad K15: unconnected-(U4C-IOR_131-PadK15) -> /ICE40HX/ICE_R_131
- U4 pad K16: unconnected-(U4C-IOR_133-PadK16) -> /ICE40HX/ICE_R_133
- U4 pad L14: unconnected-(U4C-IOR_119-PadL14) -> /ICE40HX/ICE_R_119
- U4 pad L16: unconnected-(U4C-IOR_127-PadL16) -> /ICE40HX/ICE_R_127
- U4 pad M15: unconnected-(U4C-IOR_123-PadM15) -> /ICE40HX/ICE_R_123
- U4 pad M16: unconnected-(U4C-IOR_121-PadM16) -> /ICE40HX/ICE_R_121
- U4 pad N16: unconnected-(U4C-IOR_117-PadN16) -> /ICE40HX/ICE_R_117
- U4 pad P15: unconnected-(U4C-IOR_112-PadP15) -> /ICE40HX/ICE_R_112
- U4 pad P16: unconnected-(U4C-IOR_113-PadP16) -> /ICE40HX/ICE_R_113
Routing:
- net /ICE40HX/ICE_R_112: track 0.00 -> 40.7 mm
- net /ICE40HX/ICE_T_169: track 0.00 -> 39.6 mm
- net /ICE40HX/ICE_R_117: track 0.00 -> 39.2 mm
- net /ICE40HX/ICE_T_171: track 0.00 -> 38.9 mm
- net /ICE40HX/ICE_T_216: track 0.00 -> 38.8 mm
- net /ICE40HX/ICE_R_161: track 0.00 -> 38.6 mm
- net /ICE40HX/ICE_T_182: track 0.00 -> 38.5 mm
- net /ICE40HX/ICE_R_121: track 0.00 -> 38.4 mm
- net /ICE40HX/ICE_T_218: track 0.00 -> 38.4 mm
- net /ICE40HX/ICE_R_153: track 0.00 -> 37.9 mm
- net /ICE40HX/ICE_R_127: track 0.00 -> 37.7 mm
- net /ICE40HX/ICE_T_213: track 0.00 -> 37.3 mm
- net /ICE40HX/ICE_R_151: track 0.00 -> 37.2 mm
- net /ICE40HX/ICE_R_133: track 0.00 -> 37.0 mm
- net /ICE40HX/ICE_T_187: track 0.00 -> 37.0 mm
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
Commit message: added again some traces
Connections:
- J9 pad 1: unconnected-(J9-Pad1) -> /ICE40HX/ICE_R_136
- J9 pad 10: unconnected-(J9-Pad10) -> /ICE40HX/ICE_R_116
- J9 pad 11: unconnected-(J9-Pad11) -> /ICE40HX/ICE_R_118
- J9 pad 12: unconnected-(J9-Pad12) -> /ICE40HX/ICE_R_128
- J9 pad 13: unconnected-(J9-Pad13) -> /ICE40HX/ICE_R_129
- J9 pad 14: unconnected-(J9-Pad14) -> /ICE40HX/ICE_R_137
- J9 pad 15: unconnected-(J9-Pad15) -> /ICE40HX/ICE_R_134
- J9 pad 2: unconnected-(J9-Pad2) -> /ICE40HX/ICE_R_126
- J9 pad 3: unconnected-(J9-Pad3) -> /ICE40HX/ICE_R_122
- J9 pad 37: unconnected-(J9-Pad37) -> /ICE40HX/ICE_R_150
- J9 pad 38: unconnected-(J9-Pad38) -> /ICE40HX/ICE_R_142
- J9 pad 39: unconnected-(J9-Pad39) -> /ICE40HX/ICE_R_155
- J9 pad 4: unconnected-(J9-Pad4) -> /ICE40HX/ICE_R_120
- J9 pad 40: unconnected-(J9-Pad40) -> /ICE40HX/ICE_R_152
- J9 pad 41: unconnected-(J9-Pad41) -> /ICE40HX/ICE_R_166
- J9 pad 42: unconnected-(J9-Pad42) -> /ICE40HX/ICE_R_162
- J9 pad 43: unconnected-(J9-Pad43) -> /ICE40HX/ICE_R_154
- J9 pad 44: unconnected-(J9-Pad44) -> /ICE40HX/ICE_R_167
- J9 pad 45: unconnected-(J9-Pad45) -> /ICE40HX/ICE_R_146
- J9 pad 46: unconnected-(J9-Pad46) -> /ICE40HX/ICE_R_156
- J9 pad 48: unconnected-(J9-Pad48) -> /ICE40HX/ICE_R_158
- J9 pad 5: unconnected-(J9-Pad5) -> /ICE40HX/ICE_R_110
- J9 pad 6: unconnected-(J9-Pad6) -> /ICE40HX/ICE_R_109
- J9 pad 7: unconnected-(J9-Pad7) -> /ICE40HX/ICE_R_111
- J9 pad 8: unconnected-(J9-Pad8) -> /ICE40HX/ICE_R_114
- J9 pad 9: unconnected-(J9-Pad9) -> /ICE40HX/ICE_R_115
- U4 pad D14: unconnected-(U4C-IOR_167-PadD14) -> /ICE40HX/ICE_R_167
- U4 pad E13: unconnected-(U4C-IOR_166-PadE13) -> /ICE40HX/ICE_R_166
- U4 pad F11: unconnected-(U4C-IOR_158-PadF11) -> /ICE40HX/ICE_R_158
- U4 pad F12: unconnected-(U4C-IOR_156-PadF12) -> /ICE40HX/ICE_R_156
- U4 pad F13: unconnected-(U4C-IOR_162-PadF13) -> /ICE40HX/ICE_R_162
- U4 pad F14: unconnected-(U4C-IOR_155-PadF14) -> /ICE40HX/ICE_R_155
- U4 pad G10: unconnected-(U4C-IOR_146-PadG10) -> /ICE40HX/ICE_R_146
- U4 pad G12: unconnected-(U4C-IOR_154-PadG12) -> /ICE40HX/ICE_R_154
- U4 pad G13: unconnected-(U4C-IOR_152-PadG13) -> /ICE40HX/ICE_R_152
- U4 pad G14: unconnected-(U4C-IOR_150-PadG14) -> /ICE40HX/ICE_R_150
- U4 pad H14: unconnected-(U4C-IOR_142-PadH14) -> /ICE40HX/ICE_R_142
- U4 pad J10: unconnected-(U4C-IOR_122-PadJ10) -> /ICE40HX/ICE_R_122
- U4 pad J11: unconnected-(U4C-IOR_126-PadJ11) -> /ICE40HX/ICE_R_126
- U4 pad J12: unconnected-(U4C-IOR_136-PadJ12) -> /ICE40HX/ICE_R_136
- U4 pad J13: unconnected-(U4C-IOR_137-PadJ13) -> /ICE40HX/ICE_R_137
- U4 pad J14: unconnected-(U4C-IOR_134-PadJ14) -> /ICE40HX/ICE_R_134
- U4 pad K12: unconnected-(U4C-IOR_120-PadK12) -> /ICE40HX/ICE_R_120
- U4 pad K13: unconnected-(U4C-IOR_128-PadK13) -> /ICE40HX/ICE_R_128
- U4 pad K14: unconnected-(U4C-IOR_129-PadK14) -> /ICE40HX/ICE_R_129
- U4 pad L12: unconnected-(U4C-IOR_116-PadL12) -> /ICE40HX/ICE_R_116
- U4 pad L13: unconnected-(U4C-IOR_118-PadL13) -> /ICE40HX/ICE_R_118
- U4 pad M13: unconnected-(U4C-IOR_114-PadM13) -> /ICE40HX/ICE_R_114
- U4 pad M14: unconnected-(U4C-IOR_115-PadM14) -> /ICE40HX/ICE_R_115
- U4 pad P14: unconnected-(U4C-IOR_111-PadP14) -> /ICE40HX/ICE_R_111
- U4 pad R14: unconnected-(U4C-IOR_109-PadR14) -> /ICE40HX/ICE_R_109
- U4 pad R15: unconnected-(U4C-IOR_110-PadR15) -> /ICE40HX/ICE_R_110
Routing:
- net /ICE40HX/ICE_R_120: track 0.00 -> 50.7 mm, vias 0 -> 1
- net /ICE40HX/ICE_R_122: track 0.00 -> 50.1 mm, vias 0 -> 1
- net /ICE40HX/ICE_R_156: track 0.00 -> 48.1 mm, vias 0 -> 1
- net /ICE40HX/ICE_R_116: track 0.00 -> 47.2 mm, vias 0 -> 1
- net /ICE40HX/ICE_R_114: track 0.00 -> 47.2 mm, vias 0 -> 1
- net /ICE40HX/ICE_R_109: track 0.00 -> 46.7 mm, vias 0 -> 1
- net /ICE40HX/ICE_R_126: track 0.00 -> 46.5 mm, vias 0 -> 1
- net /ICE40HX/ICE_R_136: track 0.00 -> 46.0 mm, vias 0 -> 1
- net /ICE40HX/ICE_R_158: track 0.00 -> 45.9 mm, vias 0 -> 1
- net /ICE40HX/ICE_R_128: track 0.00 -> 45.7 mm, vias 0 -> 1
- net /ICE40HX/ICE_R_162: track 0.00 -> 45.1 mm, vias 0 -> 1
- net /ICE40HX/ICE_R_137: track 0.00 -> 45.0 mm, vias 0 -> 1
- net /ICE40HX/ICE_R_154: track 0.00 -> 44.8 mm, vias 0 -> 1
- net /ICE40HX/ICE_R_167: track 0.00 -> 44.7 mm, vias 0 -> 1
- net /ICE40HX/ICE_R_152: track 0.00 -> 44.4 mm, vias 0 -> 1
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
Commit message: preps for crosslink and DDR3
Parts:
- added U15: LIFMD60006UMG64I, Custom:LIFMD60006UMG64I, F.Cu at (-11.5, 9.82)
Connections:
- net /ENCODER/ICE_RE10_A renamed /ROTARY_ENCODER/ICE_RE10_A
- net /ENCODER/ICE_RE10_B renamed /ROTARY_ENCODER/ICE_RE10_B
- net /ENCODER/ICE_RE10_C renamed /ROTARY_ENCODER/ICE_RE10_C
- net /ENCODER/ICE_RE1_A renamed /ROTARY_ENCODER/ICE_RE1_A
- net /ENCODER/ICE_RE1_B renamed /ROTARY_ENCODER/ICE_RE1_B
- net /ENCODER/ICE_RE1_C renamed /ROTARY_ENCODER/ICE_RE1_C
- net /ENCODER/ICE_RE2_A renamed /ROTARY_ENCODER/ICE_RE2_A
- net /ENCODER/ICE_RE2_B renamed /ROTARY_ENCODER/ICE_RE2_B
- net /ENCODER/ICE_RE2_C renamed /ROTARY_ENCODER/ICE_RE2_C
- net /ENCODER/ICE_RE3_A renamed /ROTARY_ENCODER/ICE_RE3_A
- net /ENCODER/ICE_RE3_B renamed /ROTARY_ENCODER/ICE_RE3_B
- net /ENCODER/ICE_RE3_C renamed /ROTARY_ENCODER/ICE_RE3_C
- net /ENCODER/ICE_RE4_A renamed /ROTARY_ENCODER/ICE_RE4_A
- net /ENCODER/ICE_RE4_B renamed /ROTARY_ENCODER/ICE_RE4_B
- net /ENCODER/ICE_RE4_C renamed /ROTARY_ENCODER/ICE_RE4_C
- net /ENCODER/ICE_RE5_A renamed /ROTARY_ENCODER/ICE_RE5_A
- net /ENCODER/ICE_RE5_B renamed /ROTARY_ENCODER/ICE_RE5_B
- net /ENCODER/ICE_RE5_C renamed /ROTARY_ENCODER/ICE_RE5_C
- net /ENCODER/ICE_RE6_A renamed /ROTARY_ENCODER/ICE_RE6_A
- net /ENCODER/ICE_RE6_B renamed /ROTARY_ENCODER/ICE_RE6_B
- net /ENCODER/ICE_RE6_C renamed /ROTARY_ENCODER/ICE_RE6_C
- net /ENCODER/ICE_RE7_A renamed /ROTARY_ENCODER/ICE_RE7_A
- net /ENCODER/ICE_RE7_B renamed /ROTARY_ENCODER/ICE_RE7_B
- net /ENCODER/ICE_RE7_C renamed /ROTARY_ENCODER/ICE_RE7_C
- net /ENCODER/ICE_RE8_A renamed /ROTARY_ENCODER/ICE_RE8_A
- net /ENCODER/ICE_RE8_B renamed /ROTARY_ENCODER/ICE_RE8_B
- net /ENCODER/ICE_RE8_C renamed /ROTARY_ENCODER/ICE_RE8_C
- net /ENCODER/ICE_RE9_A renamed /ROTARY_ENCODER/ICE_RE9_A
- net /ENCODER/ICE_RE9_B renamed /ROTARY_ENCODER/ICE_RE9_B
- net /ENCODER/ICE_RE9_C renamed /ROTARY_ENCODER/ICE_RE9_C
- net /ICE40HX/ICE_B2_100 renamed /ENCODER_CTRL/ENCODER_CTRL_B_100
- net /ICE40HX/ICE_B2_101 renamed /ENCODER_CTRL/ENCODER_CTRL_B_101
- net /ICE40HX/ICE_B2_102 renamed /ENCODER_CTRL/ENCODER_CTRL_B_102
- net /ICE40HX/ICE_B2_52 renamed /ENCODER_CTRL/ENCODER_CTRL_B_52
- net /ICE40HX/ICE_B2_53 renamed /ENCODER_CTRL/ENCODER_CTRL_B_53
- net /ICE40HX/ICE_B2_54 renamed /ENCODER_CTRL/ENCODER_CTRL_B_54
- net /ICE40HX/ICE_B2_55 renamed /ENCODER_CTRL/ENCODER_CTRL_B_55
- net /ICE40HX/ICE_B2_56 renamed /ENCODER_CTRL/ENCODER_CTRL_B_56
- net /ICE40HX/ICE_B2_57 renamed /ENCODER_CTRL/ENCODER_CTRL_B_57
- net /ICE40HX/ICE_B2_58 renamed /ENCODER_CTRL/ENCODER_CTRL_B_58
- net /ICE40HX/ICE_B2_59 renamed /ENCODER_CTRL/ENCODER_CTRL_B_59
- net /ICE40HX/ICE_B2_60 renamed /ENCODER_CTRL/ENCODER_CTRL_B_60
- net /ICE40HX/ICE_B2_61 renamed /ENCODER_CTRL/ENCODER_CTRL_B_61
- net /ICE40HX/ICE_B2_63 renamed /ENCODER_CTRL/ENCODER_CTRL_B_63
- net /ICE40HX/ICE_B2_64 renamed /ENCODER_CTRL/ENCODER_CTRL_B_64
- net /ICE40HX/ICE_B2_66 renamed /ENCODER_CTRL/ENCODER_CTRL_B_66
- net /ICE40HX/ICE_B2_67 renamed /ENCODER_CTRL/ENCODER_CTRL_B_67
- net /ICE40HX/ICE_B2_68 renamed /ENCODER_CTRL/ENCODER_CTRL_B_68
- net /ICE40HX/ICE_B2_69 renamed /ENCODER_CTRL/ENCODER_CTRL_B_69
- net /ICE40HX/ICE_B2_71 renamed /ENCODER_CTRL/ENCODER_CTRL_B_71
- net /ICE40HX/ICE_B2_72 renamed /ENCODER_CTRL/ENCODER_CTRL_B_72
- net /ICE40HX/ICE_B2_73 renamed /ENCODER_CTRL/ENCODER_CTRL_B_73
- net /ICE40HX/ICE_B2_74 renamed /ENCODER_CTRL/ENCODER_CTRL_B_74
- net /ICE40HX/ICE_B2_75 renamed /ENCODER_CTRL/ENCODER_CTRL_B_75
- net /ICE40HX/ICE_B2_76 renamed /ENCODER_CTRL/ENCODER_CTRL_B_76
- net /ICE40HX/ICE_B2_77 renamed /ENCODER_CTRL/ENCODER_CTRL_B_77
- net /ICE40HX/ICE_B2_78 renamed /ENCODER_CTRL/ENCODER_CTRL_B_78
- net /ICE40HX/ICE_B2_79 renamed /ENCODER_CTRL/ENCODER_CTRL_B_79
- net /ICE40HX/ICE_B2_80 renamed /ENCODER_CTRL/ENCODER_CTRL_B_80
- net /ICE40HX/ICE_B2_83 renamed /ENCODER_CTRL/ENCODER_CTRL_B_83
- net /ICE40HX/ICE_B2_84 renamed /ENCODER_CTRL/ENCODER_CTRL_B_84
- net /ICE40HX/ICE_B2_85 renamed /ENCODER_CTRL/ENCODER_CTRL_B_85
- net /ICE40HX/ICE_B2_86 renamed /ENCODER_CTRL/ENCODER_CTRL_B_86
- net /ICE40HX/ICE_B2_87 renamed /ENCODER_CTRL/ENCODER_CTRL_B_87
- net /ICE40HX/ICE_B2_88 renamed /ENCODER_CTRL/ENCODER_CTRL_B_88
- net /ICE40HX/ICE_B2_89 renamed /ENCODER_CTRL/ENCODER_CTRL_B_89
- net /ICE40HX/ICE_B2_91 renamed /ENCODER_CTRL/ENCODER_CTRL_B_91
- net /ICE40HX/ICE_B2_92 renamed /ENCODER_CTRL/ENCODER_CTRL_B_92
- net /ICE40HX/ICE_B2_93 renamed /ENCODER_CTRL/ENCODER_CTRL_B_93
- net /ICE40HX/ICE_B2_94 renamed /ENCODER_CTRL/ENCODER_CTRL_B_94
- net /ICE40HX/ICE_B2_98 renamed /ENCODER_CTRL/ENCODER_CTRL_B_98
- net /ICE40HX/ICE_B2_99 renamed /ENCODER_CTRL/ENCODER_CTRL_B_99
- net /ICE40HX/ICE_B3_10A renamed /ENCODER_CTRL/ENCODER_CTRL_L_10A
- net /ICE40HX/ICE_B3_10B renamed /ENCODER_CTRL/ENCODER_CTRL_L_10B
- net /ICE40HX/ICE_B3_11A renamed /ENCODER_CTRL/ENCODER_CTRL_L_11A
- net /ICE40HX/ICE_B3_11B renamed /ENCODER_CTRL/ENCODER_CTRL_L_11B
- net /ICE40HX/ICE_B3_12A renamed /ENCODER_CTRL/ENCODER_CTRL_L_12A
- net /ICE40HX/ICE_B3_12B renamed /ENCODER_CTRL/ENCODER_CTRL_L_12B
- net /ICE40HX/ICE_B3_13A renamed /ENCODER_CTRL/ENCODER_CTRL_L_13A
- net /ICE40HX/ICE_B3_14B renamed /ENCODER_CTRL/ENCODER_CTRL_L_14B
- net /ICE40HX/ICE_B3_15A renamed /ENCODER_CTRL/ENCODER_CTRL_L_15A
- net /ICE40HX/ICE_B3_15B renamed /ENCODER_CTRL/ENCODER_CTRL_L_15B
- net /ICE40HX/ICE_B3_16A renamed /ENCODER_CTRL/ENCODER_CTRL_L_16A
- net /ICE40HX/ICE_B3_16B renamed /ENCODER_CTRL/ENCODER_CTRL_L_16B
- net /ICE40HX/ICE_B3_17A renamed /ENCODER_CTRL/ENCODER_CTRL_L_17A
- net /ICE40HX/ICE_B3_17B renamed /ENCODER_CTRL/ENCODER_CTRL_L_17B
- net /ICE40HX/ICE_B3_18A renamed /ENCODER_CTRL/ENCODER_CTRL_L_18A
- net /ICE40HX/ICE_B3_18B renamed /ENCODER_CTRL/ENCODER_CTRL_L_18B
- net /ICE40HX/ICE_B3_19A renamed /ENCODER_CTRL/ENCODER_CTRL_L_19A
- net /ICE40HX/ICE_B3_19B renamed /ENCODER_CTRL/ENCODER_CTRL_L_19B
- net /ICE40HX/ICE_B3_1A renamed /ENCODER_CTRL/ENCODER_CTRL_L_1A
- net /ICE40HX/ICE_B3_1B renamed /ENCODER_CTRL/ENCODER_CTRL_L_1B
- net /ICE40HX/ICE_B3_20A renamed /ENCODER_CTRL/ENCODER_CTRL_L_20A
- net /ICE40HX/ICE_B3_20B renamed /ENCODER_CTRL/ENCODER_CTRL_L_20B
- net /ICE40HX/ICE_B3_21A renamed /ENCODER_CTRL/ENCODER_CTRL_L_21A
- net /ICE40HX/ICE_B3_21B renamed /ENCODER_CTRL/ENCODER_CTRL_L_21B
- net /ICE40HX/ICE_B3_22A renamed /ENCODER_CTRL/ENCODER_CTRL_L_22A
- net /ICE40HX/ICE_B3_22B renamed /ENCODER_CTRL/ENCODER_CTRL_L_22B
- net /ICE40HX/ICE_B3_23A renamed /ENCODER_CTRL/ENCODER_CTRL_L_23A
- net /ICE40HX/ICE_B3_23B renamed /ENCODER_CTRL/ENCODER_CTRL_L_23B
- net /ICE40HX/ICE_B3_24A renamed /ENCODER_CTRL/ENCODER_CTRL_L_24A
- net /ICE40HX/ICE_B3_24B renamed /ENCODER_CTRL/ENCODER_CTRL_L_24B
- net /ICE40HX/ICE_B3_25A renamed /ENCODER_CTRL/ENCODER_CTRL_L_25A
- net /ICE40HX/ICE_B3_25B renamed /ENCODER_CTRL/ENCODER_CTRL_L_25B
- net /ICE40HX/ICE_B3_26A renamed /ENCODER_CTRL/ENCODER_CTRL_L_26A
- net /ICE40HX/ICE_B3_26B renamed /ENCODER_CTRL/ENCODER_CTRL_L_26B
- net /ICE40HX/ICE_B3_2A renamed /ENCODER_CTRL/ENCODER_CTRL_L_2A
- net /ICE40HX/ICE_B3_2B renamed /ENCODER_CTRL/ENCODER_CTRL_L_2B
- net /ICE40HX/ICE_B3_3A renamed /ENCODER_CTRL/ENCODER_CTRL_L_3A
- net /ICE40HX/ICE_B3_3B renamed /ENCODER_CTRL/ENCODER_CTRL_L_3B
- net /ICE40HX/ICE_B3_4A renamed /ENCODER_CTRL/ENCODER_CTRL_L_4A
- net /ICE40HX/ICE_B3_4B renamed /ENCODER_CTRL/ENCODER_CTRL_L_4B
- net /ICE40HX/ICE_B3_5A renamed /ENCODER_CTRL/ENCODER_CTRL_L_5A
- net /ICE40HX/ICE_B3_5B renamed /ENCODER_CTRL/ENCODER_CTRL_L_5B
- net /ICE40HX/ICE_B3_6A renamed /ENCODER_CTRL/ENCODER_CTRL_L_6A
- net /ICE40HX/ICE_B3_6B renamed /ENCODER_CTRL/ENCODER_CTRL_L_6B
- net /ICE40HX/ICE_B3_7A renamed /ENCODER_CTRL/ENCODER_CTRL_L_7A
- net /ICE40HX/ICE_B3_7B renamed /ENCODER_CTRL/ENCODER_CTRL_L_7B
- net /ICE40HX/ICE_B3_8A renamed /ENCODER_CTRL/ENCODER_CTRL_L_8A
- net /ICE40HX/ICE_B3_8B renamed /ENCODER_CTRL/ENCODER_CTRL_L_8B
- net /ICE40HX/ICE_B3_9A renamed /ENCODER_CTRL/ENCODER_CTRL_L_9A
- net /ICE40HX/ICE_B3_9B renamed /ENCODER_CTRL/ENCODER_CTRL_L_9B
- net /ICE40HX/ICE_CDONE renamed /ENCODER_CTRL/ENCODER_CTRL_CDONE
- net /ICE40HX/ICE_CRESET_B renamed /ENCODER_CTRL/ENCODER_CTRL_CRESET_B
- net /ICE40HX/ICE_JTAG_SCK renamed /ENCODER_CTRL/ENCODER_CTRL_JTAG_SCK
- net /ICE40HX/ICE_JTAG_SDI renamed /ENCODER_CTRL/ENCODER_CTRL_JTAG_SDI
- net /ICE40HX/ICE_JTAG_SDO renamed /ENCODER_CTRL/ENCODER_CTRL_JTAG_SDO
- net /ICE40HX/ICE_JTAG_SS renamed /ENCODER_CTRL/ENCODER_CTRL_JTAG_SS
- net /ICE40HX/ICE_JTAG_TRST renamed /ENCODER_CTRL/ENCODER_CTRL_JTAG_TRST
- net /ICE40HX/ICE_JTAG_VCC renamed /ENCODER_CTRL/ENCODER_CTRL_JTAG_VCC
- net /ICE40HX/ICE_R_109 renamed /ENCODER_CTRL/ENCODER_CTRL_R_109
- net /ICE40HX/ICE_R_110 renamed /ENCODER_CTRL/ENCODER_CTRL_R_110
- net /ICE40HX/ICE_R_111 renamed /ENCODER_CTRL/ENCODER_CTRL_R_111
- net /ICE40HX/ICE_R_112 renamed /ENCODER_CTRL/ENCODER_CTRL_R_112
- net /ICE40HX/ICE_R_113 renamed /ENCODER_CTRL/ENCODER_CTRL_R_113
- net /ICE40HX/ICE_R_114 renamed /ENCODER_CTRL/ENCODER_CTRL_R_114
- net /ICE40HX/ICE_R_115 renamed /ENCODER_CTRL/ENCODER_CTRL_R_115
- net /ICE40HX/ICE_R_116 renamed /ENCODER_CTRL/ENCODER_CTRL_R_116
- net /ICE40HX/ICE_R_117 renamed /ENCODER_CTRL/ENCODER_CTRL_R_117
- net /ICE40HX/ICE_R_118 renamed /ENCODER_CTRL/ENCODER_CTRL_R_118
- net /ICE40HX/ICE_R_119 renamed /ENCODER_CTRL/ENCODER_CTRL_R_119
- net /ICE40HX/ICE_R_121 renamed /ENCODER_CTRL/ENCODER_CTRL_R_121
- net /ICE40HX/ICE_R_123 renamed /ENCODER_CTRL/ENCODER_CTRL_R_123
- net /ICE40HX/ICE_R_127 renamed /ENCODER_CTRL/ENCODER_CTRL_R_127
- net /ICE40HX/ICE_R_128 renamed /ENCODER_CTRL/ENCODER_CTRL_R_128
- net /ICE40HX/ICE_R_129 renamed /ENCODER_CTRL/ENCODER_CTRL_R_129
- net /ICE40HX/ICE_R_130 renamed /ENCODER_CTRL/ENCODER_CTRL_R_130
- net /ICE40HX/ICE_R_131 renamed /ENCODER_CTRL/ENCODER_CTRL_R_131
- net /ICE40HX/ICE_R_133 renamed /ENCODER_CTRL/ENCODER_CTRL_R_133
- net /ICE40HX/ICE_R_134 renamed /ENCODER_CTRL/ENCODER_CTRL_R_134
- net /ICE40HX/ICE_R_137 renamed /ENCODER_CTRL/ENCODER_CTRL_R_137
- net /ICE40HX/ICE_R_138 renamed /ENCODER_CTRL/ENCODER_CTRL_R_138
- net /ICE40HX/ICE_R_143 renamed /ENCODER_CTRL/ENCODER_CTRL_R_143
- net /ICE40HX/ICE_R_145 renamed /ENCODER_CTRL/ENCODER_CTRL_R_145
- net /ICE40HX/ICE_R_147 renamed /ENCODER_CTRL/ENCODER_CTRL_R_147
- net /ICE40HX/ICE_R_149 renamed /ENCODER_CTRL/ENCODER_CTRL_R_149
- net /ICE40HX/ICE_R_151 renamed /ENCODER_CTRL/ENCODER_CTRL_R_151
- net /ICE40HX/ICE_R_153 renamed /ENCODER_CTRL/ENCODER_CTRL_R_153
- net /ICE40HX/ICE_R_157 renamed /ENCODER_CTRL/ENCODER_CTRL_R_157
- net /ICE40HX/ICE_R_160 renamed /ENCODER_CTRL/ENCODER_CTRL_R_160
- net /ICE40HX/ICE_R_161 renamed /ENCODER_CTRL/ENCODER_CTRL_R_161
- net /ICE40HX/ICE_R_165 renamed /ENCODER_CTRL/ENCODER_CTRL_R_165
- net /ICE40HX/ICE_T_169 renamed /ENCODER_CTRL/ENCODER_CTRL_T_169
- net /ICE40HX/ICE_T_171 renamed /ENCODER_CTRL/ENCODER_CTRL_T_171
- net /ICE40HX/ICE_T_176 renamed /ENCODER_CTRL/ENCODER_CTRL_T_176
- net /ICE40HX/ICE_T_177 renamed /ENCODER_CTRL/ENCODER_CTRL_T_177
- net /ICE40HX/ICE_T_178 renamed /ENCODER_CTRL/ENCODER_CTRL_T_178
- net /ICE40HX/ICE_T_182 renamed /ENCODER_CTRL/ENCODER_CTRL_T_182
- net /ICE40HX/ICE_T_183 renamed /ENCODER_CTRL/ENCODER_CTRL_T_183
- net /ICE40HX/ICE_T_184 renamed /ENCODER_CTRL/ENCODER_CTRL_T_184
- net /ICE40HX/ICE_T_186 renamed /ENCODER_CTRL/ENCODER_CTRL_T_186
- net /ICE40HX/ICE_T_187 renamed /ENCODER_CTRL/ENCODER_CTRL_T_187
- net /ICE40HX/ICE_T_194 renamed /ENCODER_CTRL/ENCODER_CTRL_T_194
- net /ICE40HX/ICE_T_199 renamed /ENCODER_CTRL/ENCODER_CTRL_T_199
- net /ICE40HX/ICE_T_200 renamed /ENCODER_CTRL/ENCODER_CTRL_T_200
- net /ICE40HX/ICE_T_203 renamed /ENCODER_CTRL/ENCODER_CTRL_T_203
- net /ICE40HX/ICE_T_205 renamed /ENCODER_CTRL/ENCODER_CTRL_T_205
- net /ICE40HX/ICE_T_207 renamed /ENCODER_CTRL/ENCODER_CTRL_T_207
- net /ICE40HX/ICE_T_208 renamed /ENCODER_CTRL/ENCODER_CTRL_T_208
- net /ICE40HX/ICE_T_211 renamed /ENCODER_CTRL/ENCODER_CTRL_T_211
- net /ICE40HX/ICE_T_213 renamed /ENCODER_CTRL/ENCODER_CTRL_T_213
- net /ICE40HX/ICE_T_214 renamed /ENCODER_CTRL/ENCODER_CTRL_T_214
- net /ICE40HX/ICE_T_216 renamed /ENCODER_CTRL/ENCODER_CTRL_T_216
- net /ICE40HX/ICE_T_218 renamed /ENCODER_CTRL/ENCODER_CTRL_T_218
- net /ICE40HX/ICE_T_220 renamed /ENCODER_CTRL/ENCODER_CTRL_T_220
- net /ICE40HX/ICE_T_223 renamed /ENCODER_CTRL/ENCODER_CTRL_T_223
- net /STM32F4/STM_A0 renamed /MIDI_CTRL/STM_A0
- net /STM32F4/STM_A1 renamed /MIDI_CTRL/STM_A1
- net /STM32F4/STM_A10 renamed /MIDI_CTRL/STM_A10
- net /STM32F4/STM_A11 renamed /MIDI_CTRL/STM_A11
- net /STM32F4/STM_A12 renamed /MIDI_CTRL/STM_A12
- net /STM32F4/STM_A13 renamed /MIDI_CTRL/STM_A13
- net /STM32F4/STM_A14 renamed /MIDI_CTRL/STM_A14
- net /STM32F4/STM_A15 renamed /MIDI_CTRL/STM_A15
- net /STM32F4/STM_A2 renamed /MIDI_CTRL/STM_A2
- net /STM32F4/STM_A3 renamed /MIDI_CTRL/STM_A3
- net /STM32F4/STM_A4 renamed /MIDI_CTRL/STM_A4
- net /STM32F4/STM_A5 renamed /MIDI_CTRL/STM_A5
- net /STM32F4/STM_A6 renamed /MIDI_CTRL/STM_A6
- net /STM32F4/STM_A7 renamed /MIDI_CTRL/STM_A7
- net /STM32F4/STM_A8 renamed /MIDI_CTRL/STM_A8
- net /STM32F4/STM_A9 renamed /MIDI_CTRL/STM_A9
- net /STM32F4/STM_B0 renamed /MIDI_CTRL/STM_B0
- net /STM32F4/STM_B1 renamed /MIDI_CTRL/STM_B1
- net /STM32F4/STM_B10 renamed /MIDI_CTRL/STM_B10
- net /STM32F4/STM_B11 renamed /MIDI_CTRL/STM_B11
- net /STM32F4/STM_B12 renamed /MIDI_CTRL/STM_B12
- net /STM32F4/STM_B13 renamed /MIDI_CTRL/STM_B13
- net /STM32F4/STM_B14 renamed /MIDI_CTRL/STM_B14
- net /STM32F4/STM_B15 renamed /MIDI_CTRL/STM_B15
- net /STM32F4/STM_B2 renamed /MIDI_CTRL/STM_B2
- net /STM32F4/STM_B3 renamed /MIDI_CTRL/STM_B3
- net /STM32F4/STM_B4 renamed /MIDI_CTRL/STM_B4
- net /STM32F4/STM_B5 renamed /MIDI_CTRL/STM_B5
- net /STM32F4/STM_B6 renamed /MIDI_CTRL/STM_B6
- net /STM32F4/STM_B7 renamed /MIDI_CTRL/STM_B7
- net /STM32F4/STM_B8 renamed /MIDI_CTRL/STM_B8
- net /STM32F4/STM_B9 renamed /MIDI_CTRL/STM_B9
- net /STM32F4/STM_C0 renamed /MIDI_CTRL/STM_C0
- net /STM32F4/STM_C1 renamed /MIDI_CTRL/STM_C1
- net /STM32F4/STM_C10 renamed /MIDI_CTRL/STM_C10
- net /STM32F4/STM_C11 renamed /MIDI_CTRL/STM_C11
- net /STM32F4/STM_C12 renamed /MIDI_CTRL/STM_C12
- net /STM32F4/STM_C13 renamed /MIDI_CTRL/STM_C13
- net /STM32F4/STM_C14 renamed /MIDI_CTRL/STM_C14
- net /STM32F4/STM_C15 renamed /MIDI_CTRL/STM_C15
- net /STM32F4/STM_C2 renamed /MIDI_CTRL/STM_C2
- net /STM32F4/STM_C3 renamed /MIDI_CTRL/STM_C3
- net /STM32F4/STM_C4 renamed /MIDI_CTRL/STM_C4
- net /STM32F4/STM_C5 renamed /MIDI_CTRL/STM_C5
- net /STM32F4/STM_C6 renamed /MIDI_CTRL/STM_C6
- net /STM32F4/STM_C7 renamed /MIDI_CTRL/STM_C7
- net /STM32F4/STM_C8 renamed /MIDI_CTRL/STM_C8
- net /STM32F4/STM_C9 renamed /MIDI_CTRL/STM_C9
- net /STM32F4/STM_D0 renamed /MIDI_CTRL/STM_D0
- net /STM32F4/STM_D1 renamed /MIDI_CTRL/STM_D1
- net /STM32F4/STM_D10 renamed /MIDI_CTRL/STM_D10
- net /STM32F4/STM_D11 renamed /MIDI_CTRL/STM_D11
- net /STM32F4/STM_D12 renamed /MIDI_CTRL/STM_D12
- net /STM32F4/STM_D13 renamed /MIDI_CTRL/STM_D13
- net /STM32F4/STM_D14 renamed /MIDI_CTRL/STM_D14
- net /STM32F4/STM_D15 renamed /MIDI_CTRL/STM_D15
- net /STM32F4/STM_D2 renamed /MIDI_CTRL/STM_D2
- net /STM32F4/STM_D3 renamed /MIDI_CTRL/STM_D3
- net /STM32F4/STM_D4 renamed /MIDI_CTRL/STM_D4
- net /STM32F4/STM_D5 renamed /MIDI_CTRL/STM_D5
- net /STM32F4/STM_D6 renamed /MIDI_CTRL/STM_D6
- net /STM32F4/STM_D7 renamed /MIDI_CTRL/STM_D7
- net /STM32F4/STM_D8 renamed /MIDI_CTRL/STM_D8
- net /STM32F4/STM_D9 renamed /MIDI_CTRL/STM_D9
- net /STM32F4/STM_E0 renamed /MIDI_CTRL/STM_E0
- net /STM32F4/STM_E1 renamed /MIDI_CTRL/STM_E1
- net /STM32F4/STM_E10 renamed /MIDI_CTRL/STM_E10
- net /STM32F4/STM_E11 renamed /MIDI_CTRL/STM_E11
- net /STM32F4/STM_E12 renamed /MIDI_CTRL/STM_E12
- net /STM32F4/STM_E13 renamed /MIDI_CTRL/STM_E13
- net /STM32F4/STM_E14 renamed /MIDI_CTRL/STM_E14
- net /STM32F4/STM_E15 renamed /MIDI_CTRL/STM_E15
- net /STM32F4/STM_E2 renamed /MIDI_CTRL/STM_E2
- net /STM32F4/STM_E3 renamed /MIDI_CTRL/STM_E3
- net /STM32F4/STM_E4 renamed /MIDI_CTRL/STM_E4
- net /STM32F4/STM_E5 renamed /MIDI_CTRL/STM_E5
- net /STM32F4/STM_E6 renamed /MIDI_CTRL/STM_E6
- net /STM32F4/STM_E7 renamed /MIDI_CTRL/STM_E7
- net /STM32F4/STM_E8 renamed /MIDI_CTRL/STM_E8
- net /STM32F4/STM_E9 renamed /MIDI_CTRL/STM_E9
- net /STM32F4/STM_USB_OTG_FS_DN renamed /MIDI_CTRL/STM_USB_OTG_FS_DN
- net /STM32F4/STM_USB_OTG_FS_DP renamed /MIDI_CTRL/STM_USB_OTG_FS_DP
- J6 pad 1: unconnected-(J6-Pad1) -> /ENCODER_CTRL/ENCODER_CTRL_T_173
- J6 pad 10: unconnected-(J6-Pad10) -> /ENCODER_CTRL/ENCODER_CTRL_T_185
- J6 pad 11: unconnected-(J6-Pad11) -> /ENCODER_CTRL/ENCODER_CTRL_T_193
- J6 pad 12: unconnected-(J6-Pad12) -> /ENCODER_CTRL/ENCODER_CTRL_T_191
- J6 pad 2: unconnected-(J6-Pad2) -> /ENCODER_CTRL/ENCODER_CTRL_T_179
- J6 pad 3: unconnected-(J6-Pad3) -> /ENCODER_CTRL/ENCODER_CTRL_T_168
- J6 pad 37: unconnected-(J6-Pad37) -> /ENCODER_CTRL/ENCODER_CTRL_T_210
- J6 pad 38: unconnected-(J6-Pad38) -> /ENCODER_CTRL/ENCODER_CTRL_T_206
- J6 pad 39: unconnected-(J6-Pad39) -> /ENCODER_CTRL/ENCODER_CTRL_T_212
- J6 pad 4: unconnected-(J6-Pad4) -> /ENCODER_CTRL/ENCODER_CTRL_T_170
- J6 pad 40: unconnected-(J6-Pad40) -> /ENCODER_CTRL/ENCODER_CTRL_T_209
- J6 pad 41: unconnected-(J6-Pad41) -> /ENCODER_CTRL/ENCODER_CTRL_T_219
- J6 pad 42: unconnected-(J6-Pad42) -> /ENCODER_CTRL/ENCODER_CTRL_T_221
- J6 pad 43: unconnected-(J6-Pad43) -> /ENCODER_CTRL/ENCODER_CTRL_T_224
- J6 pad 44: unconnected-(J6-Pad44) -> /ENCODER_CTRL/ENCODER_CTRL_T_222
- J6 pad 45: unconnected-(J6-Pad45) -> /ENCODER_CTRL/ENCODER_CTRL_T_226
- J6 pad 46: unconnected-(J6-Pad46) -> /ENCODER_CTRL/ENCODER_CTRL_T_227
- J6 pad 47: unconnected-(J6-Pad47) -> /ENCODER_CTRL/ENCODER_CTRL_T_196
- J6 pad 48: unconnected-(J6-Pad48) -> /ENCODER_CTRL/ENCODER_CTRL_T_192
- J6 pad 49: unconnected-(J6-Pad49) -> /ENCODER_CTRL/ENCODER_CTRL_T_225
- J6 pad 5: unconnected-(J6-Pad5) -> /ENCODER_CTRL/ENCODER_CTRL_T_174
- J6 pad 50: unconnected-(J6-Pad50) -> /ENCODER_CTRL/ENCODER_CTRL_T_215
- J6 pad 6: unconnected-(J6-Pad6) -> /ENCODER_CTRL/ENCODER_CTRL_T_172
- J6 pad 7: unconnected-(J6-Pad7) -> /ENCODER_CTRL/ENCODER_CTRL_T_181
- J6 pad 8: unconnected-(J6-Pad8) -> /ENCODER_CTRL/ENCODER_CTRL_T_180
- J6 pad 9: unconnected-(J6-Pad9) -> /ENCODER_CTRL/ENCODER_CTRL_T_190
- J9 pad 1: /ICE40HX/ICE_R_136 -> /ENCODER_CTRL/ENCODER_CTRL_R_122
- J9 pad 2: /ICE40HX/ICE_R_126 -> /ENCODER_CTRL/ENCODER_CTRL_R_120
- J9 pad 3: /ICE40HX/ICE_R_122 -> /ENCODER_CTRL/ENCODER_CTRL_R_126
- J9 pad 37: /ICE40HX/ICE_R_150 -> /ENCODER_CTRL/ENCODER_CTRL_R_144
- J9 pad 38: /ICE40HX/ICE_R_142 -> /ENCODER_CTRL/ENCODER_CTRL_R_148
- J9 pad 39: /ICE40HX/ICE_R_155 -> /ENCODER_CTRL/ENCODER_CTRL_R_142
- J9 pad 4: /ICE40HX/ICE_R_120 -> /ENCODER_CTRL/ENCODER_CTRL_R_136
- J9 pad 40: /ICE40HX/ICE_R_152 -> /ENCODER_CTRL/ENCODER_CTRL_R_139
- J9 pad 41: /ICE40HX/ICE_R_166 -> /ENCODER_CTRL/ENCODER_CTRL_R_152
- J9 pad 42: /ICE40HX/ICE_R_162 -> /ENCODER_CTRL/ENCODER_CTRL_R_150
- J9 pad 43: /ICE40HX/ICE_R_154 -> /ENCODER_CTRL/ENCODER_CTRL_R_162
- J9 pad 44: /ICE40HX/ICE_R_167 -> /ENCODER_CTRL/ENCODER_CTRL_R_155
- J9 pad 45: /ICE40HX/ICE_R_146 -> /ENCODER_CTRL/ENCODER_CTRL_R_167
- J9 pad 46: /ICE40HX/ICE_R_156 -> /ENCODER_CTRL/ENCODER_CTRL_R_166
- J9 pad 47: unconnected-(J9-Pad47) -> /ENCODER_CTRL/ENCODER_CTRL_R_146
- J9 pad 48: /ICE40HX/ICE_R_158 -> /ENCODER_CTRL/ENCODER_CTRL_R_154
- J9 pad 49: unconnected-(J9-Pad49) -> /ENCODER_CTRL/ENCODER_CTRL_R_158
- J9 pad 50: unconnected-(J9-Pad50) -> /ENCODER_CTRL/ENCODER_CTRL_R_156
- U4 pad C10: unconnected-(U4B-IOT_185-PadC10) -> /ENCODER_CTRL/ENCODER_CTRL_T_185
- U4 pad C11: unconnected-(U4B-IOT_180-PadC11) -> /ENCODER_CTRL/ENCODER_CTRL_T_180
- U4 pad C12: unconnected-(U4B-IOT_172-PadC12) -> /ENCODER_CTRL/ENCODER_CTRL_T_172
- U4 pad C13: unconnected-(U4B-IOT_174-PadC13) -> /ENCODER_CTRL/ENCODER_CTRL_T_174
- U4 pad C14: unconnected-(U4B-IOT_168-PadC14) -> /ENCODER_CTRL/ENCODER_CTRL_T_168
- U4 pad C3: unconnected-(U4B-IOT_227-PadC3) -> /ENCODER_CTRL/ENCODER_CTRL_T_227
- U4 pad C4: unconnected-(U4B-IOT_222-PadC4) -> /ENCODER_CTRL/ENCODER_CTRL_T_222
- U4 pad C5: unconnected-(U4B-IOT_221-PadC5) -> /ENCODER_CTRL/ENCODER_CTRL_T_221
- U4 pad C6: unconnected-(U4B-IOT_209-PadC6) -> /ENCODER_CTRL/ENCODER_CTRL_T_209
- U4 pad C7: unconnected-(U4B-IOT_206-PadC7) -> /ENCODER_CTRL/ENCODER_CTRL_T_206
- U4 pad C9: unconnected-(U4B-IOT_191-PadC9) -> /ENCODER_CTRL/ENCODER_CTRL_T_191
- U4 pad D10: unconnected-(U4B-IOT_190-PadD10) -> /ENCODER_CTRL/ENCODER_CTRL_T_190
- U4 pad D11: unconnected-(U4B-IOT_181-PadD11) -> /ENCODER_CTRL/ENCODER_CTRL_T_181
- U4 pad D13: unconnected-(U4B-IOT_170-PadD13) -> /ENCODER_CTRL/ENCODER_CTRL_T_170
- U4 pad D14: /ICE40HX/ICE_R_167 -> /ENCODER_CTRL/ENCODER_CTRL_R_167
- U4 pad D3: unconnected-(U4B-IOT_226-PadD3) -> /ENCODER_CTRL/ENCODER_CTRL_T_226
- U4 pad D4: unconnected-(U4B-IOT_224-PadD4) -> /ENCODER_CTRL/ENCODER_CTRL_T_224
- U4 pad D5: unconnected-(U4B-IOT_219-PadD5) -> /ENCODER_CTRL/ENCODER_CTRL_T_219
- U4 pad D6: unconnected-(U4B-IOT_212-PadD6) -> /ENCODER_CTRL/ENCODER_CTRL_T_212
- U4 pad D7: unconnected-(U4B-IOT_210-PadD7) -> /ENCODER_CTRL/ENCODER_CTRL_T_210
- U4 pad D9: unconnected-(U4B-IOT_193-PadD9) -> /ENCODER_CTRL/ENCODER_CTRL_T_193
- U4 pad E10: unconnected-(U4B-IOT_179-PadE10) -> /ENCODER_CTRL/ENCODER_CTRL_T_179
- U4 pad E11: unconnected-(U4B-IOT_173-PadE11) -> /ENCODER_CTRL/ENCODER_CTRL_T_173
- U4 pad E13: /ICE40HX/ICE_R_166 -> /ENCODER_CTRL/ENCODER_CTRL_R_166
- U4 pad E5: unconnected-(U4B-IOT_225-PadE5) -> /ENCODER_CTRL/ENCODER_CTRL_T_225
- U4 pad E6: unconnected-(U4B-IOT_215-PadE6) -> /ENCODER_CTRL/ENCODER_CTRL_T_215
- U4 pad E9: unconnected-(U4B-IOT_192-PadE9) -> /ENCODER_CTRL/ENCODER_CTRL_T_192
- U4 pad F11: /ICE40HX/ICE_R_158 -> /ENCODER_CTRL/ENCODER_CTRL_R_158
- U4 pad F12: /ICE40HX/ICE_R_156 -> /ENCODER_CTRL/ENCODER_CTRL_R_156
- U4 pad F13: /ICE40HX/ICE_R_162 -> /ENCODER_CTRL/ENCODER_CTRL_R_162
- U4 pad F14: /ICE40HX/ICE_R_155 -> /ENCODER_CTRL/ENCODER_CTRL_R_155
- U4 pad F9: unconnected-(U4B-IOT_196-PadF9) -> /ENCODER_CTRL/ENCODER_CTRL_T_196
- U4 pad G10: /ICE40HX/ICE_R_146 -> /ENCODER_CTRL/ENCODER_CTRL_R_146
- U4 pad G11: unconnected-(U4C-IOR_148-PadG11) -> /ENCODER_CTRL/ENCODER_CTRL_R_148
- U4 pad G12: /ICE40HX/ICE_R_154 -> /ENCODER_CTRL/ENCODER_CTRL_R_154
- U4 pad G13: /ICE40HX/ICE_R_152 -> /ENCODER_CTRL/ENCODER_CTRL_R_152
- U4 pad G14: /ICE40HX/ICE_R_150 -> /ENCODER_CTRL/ENCODER_CTRL_R_150
- U4 pad H12: unconnected-(U4C-IOR_144-PadH12) -> /ENCODER_CTRL/ENCODER_CTRL_R_144
- U4 pad H13: unconnected-(U4C-IOR_139-PadH13) -> /ENCODER_CTRL/ENCODER_CTRL_R_139
- U4 pad H14: /ICE40HX/ICE_R_142 -> /ENCODER_CTRL/ENCODER_CTRL_R_142
- U4 pad J10: /ICE40HX/ICE_R_122 -> /ENCODER_CTRL/ENCODER_CTRL_R_122
- U4 pad J11: /ICE40HX/ICE_R_126 -> /ENCODER_CTRL/ENCODER_CTRL_R_126
- U4 pad J12: /ICE40HX/ICE_R_136 -> /ENCODER_CTRL/ENCODER_CTRL_R_136
- U4 pad K12: /ICE40HX/ICE_R_120 -> /ENCODER_CTRL/ENCODER_CTRL_R_120
Routing:
- net /ENCODER_CTRL/ENCODER_CTRL_R_120: track 0.00 -> 51.8 mm, vias 0 -> 1
- net /ENCODER_CTRL/ENCODER_CTRL_R_122: track 0.00 -> 51.2 mm, vias 0 -> 1
- net /ENCODER_CTRL/ENCODER_CTRL_R_136: track 0.00 -> 51.0 mm, vias 0 -> 1
- net /ICE40HX/ICE_R_120: track 50.7 -> 0.00 mm, vias 1 -> 0
- net /ENCODER_CTRL/ENCODER_CTRL_T_192: track 0.00 -> 50.6 mm, vias 0 -> 1
- net /ENCODER_CTRL/ENCODER_CTRL_T_215: track 0.00 -> 50.3 mm, vias 0 -> 1
- net /ENCODER_CTRL/ENCODER_CTRL_R_156: track 0.00 -> 50.2 mm, vias 0 -> 1
- net /ICE40HX/ICE_R_122: track 50.1 -> 0.00 mm, vias 1 -> 0
- net /ENCODER_CTRL/ENCODER_CTRL_T_179: track 0.00 -> 50.0 mm, vias 0 -> 1
- net /ENCODER_CTRL/ENCODER_CTRL_R_154: track 0.00 -> 49.4 mm, vias 0 -> 1
- net /ENCODER_CTRL/ENCODER_CTRL_R_126: track 0.00 -> 49.3 mm, vias 0 -> 1
- net /ENCODER_CTRL/ENCODER_CTRL_T_196: track 0.00 -> 48.8 mm, vias 0 -> 1
- net /ENCODER_CTRL/ENCODER_CTRL_R_146: track 0.00 -> 48.5 mm, vias 0 -> 1
- net /ENCODER_CTRL/ENCODER_CTRL_R_158: track 0.00 -> 48.4 mm, vias 0 -> 1
- net /ICE40HX/ICE_R_156: track 48.1 -> 0.00 mm, vias 1 -> 0
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
Commit message: kekw
Parts:
- removed C1, C10, C21, C3, C35, C36, C43, C7: 10u, Capacitor_SMD:C_0603_1608Metric_Pad1.08x0.95mm_HandSolder
- removed C11, C14: 22u, Capacitor_SMD:C_0603_1608Metric_Pad1.08x0.95mm_HandSolder
- removed C12, C20, C34, C38, C39, C40, C41, C45, C47, C48, C49, C51, C52, C56, C57, C58, C59, C60: 100n, Capacitor_SMD:C_0603_1608Metric_Pad1.08x0.95mm_HandSolder
- removed C13: 4u7, Capacitor_SMD:C_0603_1608Metric_Pad1.08x0.95mm_HandSolder
- removed C15, C4: 20p, Capacitor_SMD:C_0603_1608Metric_Pad1.08x0.95mm_HandSolder
- removed C16, C17, C18, C19, C22, C23, C24, C25, C26, C27, C28, C29, C30, C31, C32, C33: 100p, Capacitor_SMD:C_0603_1608Metric_Pad1.08x0.95mm_HandSolder
- removed C2: 30p, Capacitor_SMD:C_0603_1608Metric_Pad1.08x0.95mm_HandSolder
- removed C37, C44, C54, C55, C61: 1u, Capacitor_SMD:C_0603_1608Metric_Pad1.08x0.95mm_HandSolder
- removed C42, C46, C8, C9: 10n, Capacitor_SMD:C_0603_1608Metric_Pad1.08x0.95mm_HandSolder
- removed C5, C6: 2u2, Capacitor_SMD:C_0603_1608Metric_Pad1.08x0.95mm_HandSolder
- removed C50, C53: 2p2, Capacitor_SMD:C_0603_1608Metric_Pad1.08x0.95mm_HandSolder
- removed D1: CUS10S40H3F, Custom:CUS10S40H3F
- removed D2, D3, D4, D5: LED, LED_SMD:LED_0603_1608Metric
- removed D6: CDSU4148, Diode_SMD:D_0603_1608Metric_Pad1.05x0.95mm_HandSolder
- removed FB1, FB2, FB3, FB4, FB5: 600R 500mA, Inductor_SMD:L_0603_1608Metric_Pad1.05x0.95mm_HandSolder
- removed J1: UJ31CHG2SMTTR, Custom:UJ31CHG2SMTTR
- removed J10, J11, J6, J9: 901301150, Custom:901301150
- removed J12: 901301240, Custom:901301240
- removed J2, J3, J4, J5, J7: 702462004, Custom:702462004
- removed J8: 61301611121, Custom:61301611121
- removed L1: 10u, Inductor_SMD:L_0603_1608Metric_Pad1.05x0.95mm_HandSolder
- removed R1, R2: 5k1, Resistor_SMD:R_0603_1608Metric_Pad0.98x0.95mm_HandSolder
- removed R10, R12, R19, R24: 100, Resistor_SMD:R_0603_1608Metric_Pad0.98x0.95mm_HandSolder
- removed R11, R13: 100m, Resistor_SMD:R_0603_1608Metric_Pad0.98x0.95mm_HandSolder
- removed R14, R18, R21, R22, R23: 1, Resistor_SMD:R_0603_1608Metric_Pad0.98x0.95mm_HandSolder
- removed R15: 2k4, Resistor_SMD:R_0603_1608Metric_Pad0.98x0.95mm_HandSolder
- removed R16: 825, Resistor_SMD:R_0603_1608Metric_Pad0.98x0.95mm_HandSolder
- removed R17: 300, Resistor_SMD:R_0603_1608Metric_Pad0.98x0.95mm_HandSolder
- removed R20, R25, R29, R30, R31, R32, R33, R34, R35, R36, R37, R38, R39, R40, R41, R42, R43, R44, R45, R46, R47, R48, R49, R50, R51, R52, R53, R54, R55, R56, R57, R58, R59, R61: 10k, Resistor_SMD:R_0603_1608Metric_Pad0.98x0.95mm_HandSolder
- removed R26: 649, Resistor_SMD:R_0603_1608Metric_Pad0.98x0.95mm_HandSolder
- removed R27, R28: 0, Resistor_SMD:R_0603_1608Metric_Pad0.98x0.95mm_HandSolder
- removed R3: 873k3, Resistor_SMD:R_0603_1608Metric_Pad0.98x0.95mm_HandSolder
- removed R4: 100k, Resistor_SMD:R_0603_1608Metric_Pad0.98x0.95mm_HandSolder
- removed R5: 1k, Resistor_SMD:R_0603_1608Metric_Pad0.98x0.95mm_HandSolder
- removed R6, R7: 1M, Resistor_SMD:R_0603_1608Metric_Pad0.98x0.95mm_HandSolder
- removed R60: 47, Resistor_SMD:R_0603_1608Metric_Pad0.98x0.95mm_HandSolder
- removed R8: 357k, Resistor_SMD:R_0603_1608Metric_Pad0.98x0.95mm_HandSolder
- removed R9: 210k, Resistor_SMD:R_0603_1608Metric_Pad0.98x0.95mm_HandSolder
- removed TP1, TP10, TP11, TP2, TP3, TP4, TP5, TP6, TP7, TP8, TP9: TestPoint, TestPoint:TestPoint_Pad_D3.0mm
- removed U1: TPS61040DBVR, Custom:TPS61040DBVR
- removed U10, U11, U12, U13, U14, U5, U6, U7, U8, U9: EC11E183440C, Custom:EC11E183440C
- removed U15: LIFMD60006UMG64I, Custom:LIFMD60006UMG64I
- removed U2: LT3030EFETRPBF, Custom:LT8302ES8ETRPBF
- removed U3: STM32F407VGTx, Package_QFP:LQFP-100_14x14mm_P0.5mm
- removed U4: ICE40HX8KCT256, Custom:ICE40HX8KCT256
- removed X1: STDCSU18M, Custom:STDCSU18M
Routing:
- net GND: track 111.4 -> 0.00 mm, vias 28 -> 0
- net /ENCODER_CTRL/ENCODER_CTRL_B_74: track 54.8 -> 0.00 mm, vias 1 -> 0
- net /ENCODER_CTRL/ENCODER_CTRL_B_68: track 54.0 -> 0.00 mm, vias 1 -> 0
- net /ENCODER_CTRL/ENCODER_CTRL_L_22A: track 53.3 -> 0.00 mm, vias 1 -> 0
- net /ENCODER_CTRL/ENCODER_CTRL_L_21A: track 52.4 -> 0.00 mm, vias 1 -> 0
- net /ENCODER_CTRL/ENCODER_CTRL_L_19A: track 52.1 -> 0.00 mm, vias 1 -> 0
- net /ENCODER_CTRL/ENCODER_CTRL_R_120: track 51.8 -> 0.00 mm, vias 1 -> 0
- net /ENCODER_CTRL/ENCODER_CTRL_L_7A: track 51.2 -> 0.00 mm, vias 1 -> 0
- net /ENCODER_CTRL/ENCODER_CTRL_B_85: track 51.2 -> 0.00 mm, vias 1 -> 0
- net /ENCODER_CTRL/ENCODER_CTRL_B_64: track 51.2 -> 0.00 mm, vias 1 -> 0
- net /ENCODER_CTRL/ENCODER_CTRL_R_122: track 51.2 -> 0.00 mm, vias 1 -> 0
- net /ENCODER_CTRL/ENCODER_CTRL_B_80: track 51.1 -> 0.00 mm, vias 1 -> 0
- net /ENCODER_CTRL/ENCODER_CTRL_R_136: track 51.0 -> 0.00 mm, vias 1 -> 0
- net /ENCODER_CTRL/ENCODER_CTRL_L_24B: track 51.0 -> 0.00 mm, vias 1 -> 0
- net /ENCODER_CTRL/ENCODER_CTRL_L_4A: track 50.8 -> 0.00 mm, vias 1 -> 0
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- removed copper zone on In2.Cu, net +1V2
- removed copper zone on In2.Cu, net +3V3
- removed copper zone on In3.Cu, net GND
Other:
- board outline removed
- copper layers 6 -> 2
- board text removed: "U1"
