File: FuseBox/ENCODER_CTRL.kicad_sch (KiCad schematic)
At the start: 47 parts, among them J10 901301150, J11 901301150, J6 901301150, J8 61301611121, J9 901301150, U4 ICE40HX8KCT256

Commit message: preps for crosslink and DDR3
Connections:
- net ENCODER_CTRL_T_185: now reaches U4.C10 (IOT_185)
- net ENCODER_CTRL_T_185: now also J6.10
- net ENCODER_CTRL_T_180: now reaches U4.C11 (IOT_180)
- net ENCODER_CTRL_T_180: now also J6.8
- net ENCODER_CTRL_T_172: now reaches U4.C12 (IOT_172)
- net ENCODER_CTRL_T_172: now also J6.6
- net ENCODER_CTRL_T_174: now reaches U4.C13 (IOT_174)
- net ENCODER_CTRL_T_174: now also J6.5
- net ENCODER_CTRL_T_168: now reaches U4.C14 (IOT_168)
- net ENCODER_CTRL_T_168: now also J6.3
- net ENCODER_CTRL_T_227: now reaches U4.C3 (IOT_227)
- net ENCODER_CTRL_T_227: now also J6.46
- net ENCODER_CTRL_T_222: now reaches U4.C4 (IOT_222)
- net ENCODER_CTRL_T_222: now also J6.44
- net ENCODER_CTRL_T_221: now reaches U4.C5 (IOT_221)
- net ENCODER_CTRL_T_221: now also J6.42
- net ENCODER_CTRL_T_209: now reaches U4.C6 (IOT_209)
- net ENCODER_CTRL_T_209: now also J6.40
- net ENCODER_CTRL_T_206: now reaches U4.C7 (IOT_206)
- net ENCODER_CTRL_T_206: now also J6.38
- net ENCODER_CTRL_T_191: now reaches U4.C9 (IOT_191)
- net ENCODER_CTRL_T_191: now also J6.12
- net ENCODER_CTRL_T_190: now reaches U4.D10 (IOT_190)
- net ENCODER_CTRL_T_190: now also J6.9
- net ENCODER_CTRL_T_181: now reaches U4.D11 (IOT_181)
- net ENCODER_CTRL_T_181: now also J6.7
- net ENCODER_CTRL_T_170: now reaches U4.D13 (IOT_170)
- net ENCODER_CTRL_T_170: now also J6.4
- net ENCODER_CTRL_T_226: now reaches U4.D3 (IOT_226)
- net ENCODER_CTRL_T_226: now also J6.45
- net ENCODER_CTRL_T_224: now reaches U4.D4 (IOT_224)
- net ENCODER_CTRL_T_224: now also J6.43
- net ENCODER_CTRL_T_219: now reaches U4.D5 (IOT_219)
- net ENCODER_CTRL_T_219: now also J6.41
- net ENCODER_CTRL_T_212: now reaches U4.D6 (IOT_212)
- net ENCODER_CTRL_T_212: now also J6.39
- net ENCODER_CTRL_T_210: now reaches U4.D7 (IOT_210)
- net ENCODER_CTRL_T_210: now also J6.37
- net ENCODER_CTRL_T_193: now reaches U4.D9 (IOT_193)
- net ENCODER_CTRL_T_193: now also J6.11
- net ENCODER_CTRL_T_179: now reaches U4.E10 (IOT_179)
- net ENCODER_CTRL_T_179: now also J6.2
- net ENCODER_CTRL_T_173: now reaches U4.E11 (IOT_173)
- net ENCODER_CTRL_T_173: now also J6.1
- net ENCODER_CTRL_T_225: now reaches U4.E5 (IOT_225)
- net ENCODER_CTRL_T_225: now also J6.49
- net ENCODER_CTRL_T_215: now reaches U4.E6 (IOT_215)
- net ENCODER_CTRL_T_215: now also J6.50
- net ENCODER_CTRL_T_192: now reaches U4.E9 (IOT_192)
- net ENCODER_CTRL_T_192: now also J6.48
- net ENCODER_CTRL_T_196: now reaches U4.F9 (IOT_196)
- net ENCODER_CTRL_T_196: now also J6.47
- net ENCODER_CTRL_R_148: now reaches U4.G11 (IOR_148)
- net ENCODER_CTRL_R_148: now also J9.38
- net ENCODER_CTRL_R_144: now reaches U4.H12 (IOR_144)
- net ENCODER_CTRL_R_144: now also J9.37
- net ENCODER_CTRL_R_139: now reaches U4.H13 (IOR_139)
- net ENCODER_CTRL_R_139: now also J9.40
- net ENCODER_CTRL_R_146: now reaches J9.47
- net ENCODER_CTRL_R_146: now also U4.G10 (IOR_146)
- net ENCODER_CTRL_R_158: now reaches J9.49
- net ENCODER_CTRL_R_158: now also U4.F11 (IOR_158)
- net ENCODER_CTRL_R_156: now reaches J9.50
- net ENCODER_CTRL_R_156: now also U4.F12 (IOR_156)
- net ICE_B2_100 renamed ENCODER_CTRL_B_100
- net ICE_B2_101 renamed ENCODER_CTRL_B_101
- net ICE_B2_102 renamed ENCODER_CTRL_B_102
- net ICE_B2_52 renamed ENCODER_CTRL_B_52
- net ICE_B2_53 renamed ENCODER_CTRL_B_53
- net ICE_B2_54 renamed ENCODER_CTRL_B_54
- net ICE_B2_55 renamed ENCODER_CTRL_B_55
- net ICE_B2_56 renamed ENCODER_CTRL_B_56
- net ICE_B2_57 renamed ENCODER_CTRL_B_57
- net ICE_B2_58 renamed ENCODER_CTRL_B_58
- net ICE_B2_59 renamed ENCODER_CTRL_B_59
- net ICE_B2_60 renamed ENCODER_CTRL_B_60
- net ICE_B2_61 renamed ENCODER_CTRL_B_61
- net ICE_B2_63 renamed ENCODER_CTRL_B_63
- net ICE_B2_64 renamed ENCODER_CTRL_B_64
- net ICE_B2_66 renamed ENCODER_CTRL_B_66
- net ICE_B2_67 renamed ENCODER_CTRL_B_67
- net ICE_B2_68 renamed ENCODER_CTRL_B_68
- net ICE_B2_69 renamed ENCODER_CTRL_B_69
- net ICE_B2_71 renamed ENCODER_CTRL_B_71
- net ICE_B2_72 renamed ENCODER_CTRL_B_72
- net ICE_B2_73 renamed ENCODER_CTRL_B_73
- net ICE_B2_74 renamed ENCODER_CTRL_B_74
- net ICE_B2_75 renamed ENCODER_CTRL_B_75
- net ICE_B2_76 renamed ENCODER_CTRL_B_76
- net ICE_B2_77 renamed ENCODER_CTRL_B_77
- net ICE_B2_78 renamed ENCODER_CTRL_B_78
- net ICE_B2_79 renamed ENCODER_CTRL_B_79
- net ICE_B2_80 renamed ENCODER_CTRL_B_80
- net ICE_B2_83 renamed ENCODER_CTRL_B_83
- net ICE_B2_84 renamed ENCODER_CTRL_B_84
- net ICE_B2_85 renamed ENCODER_CTRL_B_85
- net ICE_B2_86 renamed ENCODER_CTRL_B_86
- net ICE_B2_87 renamed ENCODER_CTRL_B_87
- net ICE_B2_88 renamed ENCODER_CTRL_B_88
- net ICE_B2_89 renamed ENCODER_CTRL_B_89
- net ICE_B2_91 renamed ENCODER_CTRL_B_91
- net ICE_B2_92 renamed ENCODER_CTRL_B_92
- net ICE_B2_93 renamed ENCODER_CTRL_B_93
- net ICE_B2_94 renamed ENCODER_CTRL_B_94
- net ICE_B2_98 renamed ENCODER_CTRL_B_98
- net ICE_B2_99 renamed ENCODER_CTRL_B_99
- net ICE_B3_10A renamed ENCODER_CTRL_L_10A
- net ICE_B3_10B renamed ENCODER_CTRL_L_10B
- net ICE_B3_11A renamed ENCODER_CTRL_L_11A
- net ICE_B3_11B renamed ENCODER_CTRL_L_11B
- net ICE_B3_12A renamed ENCODER_CTRL_L_12A
- net ICE_B3_12B renamed ENCODER_CTRL_L_12B
- net ICE_B3_13A renamed ENCODER_CTRL_L_13A
- net ICE_B3_14B renamed ENCODER_CTRL_L_14B
- net ICE_B3_15A renamed ENCODER_CTRL_L_15A
- net ICE_B3_15B renamed ENCODER_CTRL_L_15B
- net ICE_B3_16A renamed ENCODER_CTRL_L_16A
- net ICE_B3_16B renamed ENCODER_CTRL_L_16B
- net ICE_B3_17A renamed ENCODER_CTRL_L_17A
- net ICE_B3_17B renamed ENCODER_CTRL_L_17B
- net ICE_B3_18A renamed ENCODER_CTRL_L_18A
- net ICE_B3_18B renamed ENCODER_CTRL_L_18B
- net ICE_B3_19A renamed ENCODER_CTRL_L_19A
- net ICE_B3_19B renamed ENCODER_CTRL_L_19B
- net ICE_B3_1A renamed ENCODER_CTRL_L_1A
- net ICE_B3_1B renamed ENCODER_CTRL_L_1B
- net ICE_B3_20A renamed ENCODER_CTRL_L_20A
- net ICE_B3_20B renamed ENCODER_CTRL_L_20B
- net ICE_B3_21A renamed ENCODER_CTRL_L_21A
- net ICE_B3_21B renamed ENCODER_CTRL_L_21B
- net ICE_B3_22A renamed ENCODER_CTRL_L_22A
- net ICE_B3_22B renamed ENCODER_CTRL_L_22B
- net ICE_B3_23A renamed ENCODER_CTRL_L_23A
- net ICE_B3_23B renamed ENCODER_CTRL_L_23B
- net ICE_B3_24A renamed ENCODER_CTRL_L_24A
- net ICE_B3_24B renamed ENCODER_CTRL_L_24B
- net ICE_B3_25A renamed ENCODER_CTRL_L_25A
- net ICE_B3_25B renamed ENCODER_CTRL_L_25B
- net ICE_B3_26A renamed ENCODER_CTRL_L_26A
- net ICE_B3_26B renamed ENCODER_CTRL_L_26B
- net ICE_B3_2A renamed ENCODER_CTRL_L_2A
- net ICE_B3_2B renamed ENCODER_CTRL_L_2B
- net ICE_B3_3A renamed ENCODER_CTRL_L_3A
- net ICE_B3_3B renamed ENCODER_CTRL_L_3B
- net ICE_B3_4A renamed ENCODER_CTRL_L_4A
- net ICE_B3_4B renamed ENCODER_CTRL_L_4B
- net ICE_B3_5A renamed ENCODER_CTRL_L_5A
- net ICE_B3_5B renamed ENCODER_CTRL_L_5B
- net ICE_B3_6A renamed ENCODER_CTRL_L_6A
- net ICE_B3_6B renamed ENCODER_CTRL_L_6B
- net ICE_B3_7A renamed ENCODER_CTRL_L_7A
- net ICE_B3_7B renamed ENCODER_CTRL_L_7B
- net ICE_B3_8A renamed ENCODER_CTRL_L_8A
- net ICE_B3_8B renamed ENCODER_CTRL_L_8B
- net ICE_B3_9A renamed ENCODER_CTRL_L_9A
- net ICE_B3_9B renamed ENCODER_CTRL_L_9B
- net ICE_CDONE renamed ENCODER_CTRL_CDONE
- net ICE_CRESET_B renamed ENCODER_CTRL_CRESET_B
- net ICE_JTAG_SCK renamed ENCODER_CTRL_JTAG_SCK
- net ICE_JTAG_SDI renamed ENCODER_CTRL_JTAG_SDI
- net ICE_JTAG_SDO renamed ENCODER_CTRL_JTAG_SDO
- net ICE_JTAG_SS renamed ENCODER_CTRL_JTAG_SS
- net ICE_JTAG_TRST renamed ENCODER_CTRL_JTAG_TRST
- net ICE_JTAG_VCC renamed ENCODER_CTRL_JTAG_VCC
- net ICE_R_109 renamed ENCODER_CTRL_R_109
- net ICE_R_110 renamed ENCODER_CTRL_R_110
- net ICE_R_111 renamed ENCODER_CTRL_R_111
- net ICE_R_112 renamed ENCODER_CTRL_R_112
- net ICE_R_113 renamed ENCODER_CTRL_R_113
- net ICE_R_114 renamed ENCODER_CTRL_R_114
- net ICE_R_115 renamed ENCODER_CTRL_R_115
- net ICE_R_116 renamed ENCODER_CTRL_R_116
- net ICE_R_117 renamed ENCODER_CTRL_R_117
- net ICE_R_118 renamed ENCODER_CTRL_R_118
- net ICE_R_119 renamed ENCODER_CTRL_R_119
- net ICE_R_120 renamed ENCODER_CTRL_R_120
- net ENCODER_CTRL_R_120: now also J9.2; no longer J9.4
- net ICE_R_121 renamed ENCODER_CTRL_R_121
- net ICE_R_122 renamed ENCODER_CTRL_R_122
- net ENCODER_CTRL_R_122: now also J9.1; no longer J9.3
- net ICE_R_123 renamed ENCODER_CTRL_R_123
- net ICE_R_126 renamed ENCODER_CTRL_R_126
- net ENCODER_CTRL_R_126: now also J9.3; no longer J9.2
- net ICE_R_127 renamed ENCODER_CTRL_R_127
- net ICE_R_128 renamed ENCODER_CTRL_R_128
- net ICE_R_129 renamed ENCODER_CTRL_R_129
- net ICE_R_130 renamed ENCODER_CTRL_R_130
- net ICE_R_131 renamed ENCODER_CTRL_R_131
- net ICE_R_133 renamed ENCODER_CTRL_R_133
- net ICE_R_134 renamed ENCODER_CTRL_R_134
- net ICE_R_136 renamed ENCODER_CTRL_R_136
- net ENCODER_CTRL_R_136: now also J9.4; no longer J9.1
- net ICE_R_137 renamed ENCODER_CTRL_R_137
- net ICE_R_138 renamed ENCODER_CTRL_R_138
- net ICE_R_142 renamed ENCODER_CTRL_R_142
- net ENCODER_CTRL_R_142: now also J9.39; no longer J9.38
- net ICE_R_143 renamed ENCODER_CTRL_R_143
- net ICE_R_145 renamed ENCODER_CTRL_R_145
- net ICE_R_146 renamed ENCODER_CTRL_R_167
- net ENCODER_CTRL_R_167: now also U4.D14 (IOR_167); no longer U4.G10 (IOR_146)
- net ICE_R_147 renamed ENCODER_CTRL_R_147
- net ICE_R_149 renamed ENCODER_CTRL_R_149
- net ICE_R_150 renamed ENCODER_CTRL_R_150
- net ENCODER_CTRL_R_150: now also J9.42; no longer J9.37
- net ICE_R_151 renamed ENCODER_CTRL_R_151
- net ICE_R_152 renamed ENCODER_CTRL_R_152
- net ENCODER_CTRL_R_152: now also J9.41; no longer J9.40
- net ICE_R_153 renamed ENCODER_CTRL_R_153
- net ICE_R_154 renamed ENCODER_CTRL_R_154
- net ENCODER_CTRL_R_154: now also J9.48; no longer J9.43
- net ICE_R_155 renamed ENCODER_CTRL_R_155
- net ENCODER_CTRL_R_155: now also J9.44; no longer J9.39
- net ICE_R_156 renamed ENCODER_CTRL_R_166
- net ENCODER_CTRL_R_166: now also U4.E13 (IOR_166); no longer U4.F12 (IOR_156)
- net ICE_R_157 renamed ENCODER_CTRL_R_157
- removed net ICE_R_158: J9.48, U4.F11 (IOR_158)
- net ICE_R_160 renamed ENCODER_CTRL_R_160
- net ICE_R_161 renamed ENCODER_CTRL_R_161
- net ICE_R_162 renamed ENCODER_CTRL_R_162
- net ENCODER_CTRL_R_162: now also J9.43; no longer J9.42
- net ICE_R_165 renamed ENCODER_CTRL_R_165
- removed net ICE_R_166: J9.41, U4.E13 (IOR_166)
- removed net ICE_R_167: J9.44, U4.D14 (IOR_167)
- net ICE_T_169 renamed ENCODER_CTRL_T_169
- net ICE_T_171 renamed ENCODER_CTRL_T_171
- net ICE_T_176 renamed ENCODER_CTRL_T_176
- net ICE_T_177 renamed ENCODER_CTRL_T_177
- net ICE_T_178 renamed ENCODER_CTRL_T_178
- net ICE_T_182 renamed ENCODER_CTRL_T_182
- net ICE_T_183 renamed ENCODER_CTRL_T_183
- net ICE_T_184 renamed ENCODER_CTRL_T_184
- net ICE_T_186 renamed ENCODER_CTRL_T_186
- net ICE_T_187 renamed ENCODER_CTRL_T_187
- net ICE_T_194 renamed ENCODER_CTRL_T_194
- net ICE_T_199 renamed ENCODER_CTRL_T_199
- net ICE_T_200 renamed ENCODER_CTRL_T_200
- net ICE_T_203 renamed ENCODER_CTRL_T_203
- net ICE_T_205 renamed ENCODER_CTRL_T_205
- net ICE_T_207 renamed ENCODER_CTRL_T_207
- net ICE_T_208 renamed ENCODER_CTRL_T_208
- net ICE_T_211 renamed ENCODER_CTRL_T_211
- net ICE_T_213 renamed ENCODER_CTRL_T_213
- net ICE_T_214 renamed ENCODER_CTRL_T_214
- net ICE_T_216 renamed ENCODER_CTRL_T_216
- net ICE_T_218 renamed ENCODER_CTRL_T_218
- net ICE_T_220 renamed ENCODER_CTRL_T_220
- net ICE_T_223 renamed ENCODER_CTRL_T_223
Other:
- note added: "Bank Bottom"
- note added: "Bank Left"
- note added: "Bank Right"
- note added: "Bank Top"
- note removed: "Bank 0"
- note removed: "Bank 1"
- note removed: "Bank 2"
- note removed: "Bank 3"
- moved on the sheet: C16, C17, C18, C19, C20, C21, C22, C23, C24, C25, C26, C27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
