File: FuseBox/FUSEBOX.kicad_sch (KiCad schematic)
At the start: 0 parts

Commit message: changes
Other:
- removed sheet USB_SPI
Changed lines of the file:
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@@
 	(paper "A4")
-	(sheet
-		(at 22.86 60.96)
-		(size 27.94 6.35)
-		(exclude_from_sim no)
-		(in_bom yes)
-		(on_board yes)
-		(dnp no)
-		(fields_autoplaced yes)
-		(stroke
-			(width 0.1524)
-			(type solid)
-		)
-		(fill
-			(color 0 0 0 0.0000)
-		)
-		(property "Sheetname" "USB_SPI"
-			(at 22.86 60.2484 0)
-			(effects
-				(font
-					(size 1.27 1.27)
-				)
-				(justify left bottom)
-			)
-		)
-		(property "Sheetfile" "USB_SPI.kicad_sch"
-			(at 22.86 67.8946 0)
-			(effects
-				(font
-					(size 1.27 1.27)
-				)
-				(justify left top)
-			)
-		)
-		(instances
-			(project "FUSEBOX"
-				(path "/7cec0856-4a31-46c4-b6e3-cba19fcff38c"
-					(page "5")
-				)
-			)
-		)
-	)
 	(sheet
 		(at 22.86 22.86)

Commit message: finished schematic
Other:
- added sheet ENCODER (ENCODER.kicad_sch)
Changed lines of the file:
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@@
+	)
+	(sheet
+		(at 22.86 60.96)
+		(size 27.94 6.35)
+		(exclude_from_sim no)
+		(in_bom yes)
+		(on_board yes)
+		(dnp no)
+		(fields_autoplaced yes)
+		(stroke
+			(width 0.1524)
+			(type solid)
+		)
+		(fill
+			(color 0 0 0 0.0000)
+		)
+		(property "Sheetname" "ENCODER"
+			(at 22.86 60.2484 0)
+			(effects
+				(font
+					(size 1.27 1.27)
+				)
+				(justify left bottom)
+			)
+		)
+		(property "Sheetfile" "ENCODER.kicad_sch"
+			(at 22.86 67.8946 0)
+			(effects
+				(font
+					(size 1.27 1.27)
+				)
+				(justify left top)
+			)
+		)
+		(instances
+			(project "FUSEBOX"
+				(path "/7cec0856-4a31-46c4-b6e3-cba19fcff38c"
+					(page "5")
+				)
+			)
+		)
 	)
 	(sheet

Commit message: preps for crosslink and DDR3
Other:
- sheet ENCODER renamed ROTARY_ENCODER
- sheet ICE40HX renamed ENCODER_CTRL
- sheet STM32F4 renamed MIDI_CTRL
- added sheet DISPLAY_DRIVER (DISPLAY_DRIVER.kicad_sch)
- sheet ENCODER_CTRL: file ICE40HX.kicad_sch -> ENCODER_CTRL.kicad_sch
- sheet MIDI_CTRL: file STM32F4.kicad_sch -> MIDI_CTRL.kicad_sch
- sheet ROTARY_ENCODER: file ENCODER.kicad_sch -> ROTARY_ENCODER.kicad_sch
Changed lines of the file:
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@@
 			(color 0 0 0 0.0000)
 		)
-		(property "Sheetname" "ENCODER"
+		(property "Sheetname" "ROTARY_ENCODER"
 			(at 22.86 60.2484 0)
 			(effects
@@
 			)
 		)
-		(property "Sheetfile" "ENCODER.kicad_sch"
+		(property "Sheetfile" "ROTARY_ENCODER.kicad_sch"
 			(at 22.86 67.8946 0)
 			(effects
@@
 				(path "/7cec0856-4a31-46c4-b6e3-cba19fcff38c"
 					(page "5")
+				)
+			)
+		)
+	)
+	(sheet
+		(at 22.86 73.66)
+		(size 27.94 6.35)
+		(exclude_from_sim no)
+		(in_bom yes)
+		(on_board yes)
+		(dnp no)
+		(fields_autoplaced yes)
+		(stroke
+			(width 0.1524)
+			(type solid)
+		)
+		(fill
+			(color 0 0 0 0.0000)
+		)
+		(property "Sheetname" "DISPLAY_DRIVER"
+			(at 22.86 72.9484 0)
+			(effects
+				(font
+					(size 1.27 1.27)
+				)
+				(justify left bottom)
+			)
+		)
+		(property "Sheetfile" "DISPLAY_DRIVER.kicad_sch"
+			(at 22.86 80.5946 0)
+			(effects
+				(font
+					(size 1.27 1.27)
+				)
+				(justify left top)
+			)
+		)
+		(instances
+			(project "FUSEBOX"
+				(path "/7cec0856-4a31-46c4-b6e3-cba19fcff38c"
+					(page "6")
 				)
 			)
@@
 			(color 0 0 0 0.0000)
 		)
-		(property "Sheetname" "ICE40HX"
+		(property "Sheetname" "ENCODER_CTRL"
 			(at 22.86 47.5484 0)
 			(effects
@@
 			)
 		)
-		(property "Sheetfile" "ICE40HX.kicad_sch"
+		(property "Sheetfile" "ENCODER_CTRL.kicad_sch"
 			(at 22.86 55.1946 0)
 			(effects
@@
 			(color 0 0 0 0.0000)
 		)
-		(property "Sheetname" "STM32F4"
+		(property "Sheetname" "MIDI_CTRL"
 			(at 22.86 34.8484 0)
 			(effects
@@
 			)
 		)
-		(property "Sheetfile" "STM32F4.kicad_sch"
+		(property "Sheetfile" "MIDI_CTRL.kicad_sch"
 			(at 22.86 42.4946 0)
 			(effects

Commit message: kekw
Other:
- removed sheet DISPLAY_DRIVER
- added sheet ADC (ADC.kicad_sch)
- added sheet DAC (DAC.kicad_sch)
- added sheet LED (LED.kicad_sch)
Changed lines of the file:
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@@
 	(paper "A4")
+	(sheet
+		(at 22.86 73.66)
+		(size 27.94 6.35)
+		(exclude_from_sim no)
+		(in_bom yes)
+		(on_board yes)
+		(dnp no)
+		(fields_autoplaced yes)
+		(stroke
+			(width 0.1524)
+			(type solid)
+		)
+		(fill
+			(color 0 0 0 0.0000)
+		)
+		(property "Sheetname" "ADC"
+			(at 22.86 72.9484 0)
+			(effects
+				(font
+					(size 1.27 1.27)
+				)
+				(justify left bottom)
+			)
+		)
+		(property "Sheetfile" "ADC.kicad_sch"
+			(at 22.86 80.5946 0)
+			(effects
+				(font
+					(size 1.27 1.27)
+				)
+				(justify left top)
+			)
+		)
+		(instances
+			(project "FUSEBOX"
+				(path "/7cec0856-4a31-46c4-b6e3-cba19fcff38c"
+					(page "7")
+				)
+			)
+		)
+	)
+	(sheet
+		(at 22.86 86.36)
+		(size 27.94 6.35)
+		(exclude_from_sim no)
+		(in_bom yes)
+		(on_board yes)
+		(dnp no)
+		(fields_autoplaced yes)
+		(stroke
+			(width 0.1524)
+			(type solid)
+		)
+		(fill
+			(color 0 0 0 0.0000)
+		)
+		(property "Sheetname" "DAC"
+			(at 22.86 85.6484 0)
+			(effects
+				(font
+					(size 1.27 1.27)
+				)
+				(justify left bottom)
+			)
+		)
+		(property "Sheetfile" "DAC.kicad_sch"
+			(at 22.86 93.2946 0)
+			(effects
+				(font
+					(size 1.27 1.27)
+				)
+				(justify left top)
+			)
+		)
+		(instances
+			(project "FUSEBOX"
+				(path "/7cec0856-4a31-46c4-b6e3-cba19fcff38c"
+					(page "8")
+				)
+			)
+		)
+	)
 	(sheet
 		(at 22.86 22.86)
@@
 	)
 	(sheet
-		(at 22.86 73.66)
-		(size 27.94 6.35)
-		(exclude_from_sim no)
-		(in_bom yes)
-		(on_board yes)
-		(dnp no)
-		(fields_autoplaced yes)
-		(stroke
-			(width 0.1524)
-			(type solid)
-		)
-		(fill
-			(color 0 0 0 0.0000)
-		)
-		(property "Sheetname" "DISPLAY_DRIVER"
-			(at 22.86 72.9484 0)
-			(effects
-				(font
-					(size 1.27 1.27)
-				)
-				(justify left bottom)
-			)
-		)
-		(property "Sheetfile" "DISPLAY_DRIVER.kicad_sch"
-			(at 22.86 80.5946 0)
-			(effects
-				(font
-					(size 1.27 1.27)
-				)
-				(justify left top)
-			)
-		)
-		(instances
-			(project "FUSEBOX"
-				(path "/7cec0856-4a31-46c4-b6e3-cba19fcff38c"
-					(page "6")
-				)
-			)
+		(at 22.86 99.06)
+		(size 27.94 6.35)
+		(exclude_from_sim no)
+		(in_bom yes)
+		(on_board yes)
+		(dnp no)
+		(fields_autoplaced yes)
+		(stroke
+			(width 0.1524)
+			(type solid)
+		)
+		(fill
+			(color 0 0 0 0.0000)
+		)
+		(property "Sheetname" "LED"
+			(at 22.86 98.3484 0)
+			(effects
+				(font
+					(size 1.27 1.27)
+				)
+				(justify left bottom)
+			)
+		)
+		(property "Sheetfile" "LED.kicad_sch"
+			(at 22.86 105.9946 0)
+			(effects
+				(font
+					(size 1.27 1.27)
+				)
+				(justify left top)
+			)
+		)
+		(instances
+			(project "FUSEBOX"
+				(path "/7cec0856-4a31-46c4-b6e3-cba19fcff38c"
+					(page "7")
+				)
+			)

Commit message: changuz
Other:
- sheet ENCODER_CTRL renamed FPGA
- sheet MIDI_CTRL renamed MCU
- sheet FPGA: file ENCODER_CTRL.kicad_sch -> FPGA.kicad_sch
- sheet MCU: file MIDI_CTRL.kicad_sch -> MCU.kicad_sch
Changed lines of the file:
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@@
 			(color 0 0 0 0.0000)
 		)
-		(property "Sheetname" "ENCODER_CTRL"
+		(property "Sheetname" "FPGA"
 			(at 22.86 47.5484 0)
 			(effects
@@
 			)
 		)
-		(property "Sheetfile" "ENCODER_CTRL.kicad_sch"
+		(property "Sheetfile" "FPGA.kicad_sch"
 			(at 22.86 55.1946 0)
 			(effects
@@
 			(color 0 0 0 0.0000)
 		)
-		(property "Sheetname" "MIDI_CTRL"
+		(property "Sheetname" "MCU"
 			(at 22.86 34.8484 0)
 			(effects
@@
 			)
 		)
-		(property "Sheetfile" "MIDI_CTRL.kicad_sch"
+		(property "Sheetfile" "MCU.kicad_sch"
 			(at 22.86 42.4946 0)
 			(effects
