File: FuseBox/LED.kicad_sch (KiCad schematic)
At the start: 40 parts

Commit message: changuz
Parts:
- removed U18, U19, U20, U21, U22, U23, U24, U25, U26, U27, U28, U29, U30, U31, U32, U33, U34, U35, U37, U38, U39, U40, U41, U42, U43, U44, U45, U46, U47, U48, U49, U50, U51, U52, U53, U54, U55: ~, Custom:APA1202020, symbol Custom:APA1022020
Connections:
- new net: U17. (DO), U36. (DO) (x2)
- new net: U16. (DO), U17. (DO) (x2)
Other:
- moved on the sheet: U36
