File: FuseBox/MCU.kicad_sch (KiCad schematic)
At the start: 30 parts, among them J2 702462004, J3 702462004, J4 702462004, J5 702462004, J7 702462004, U3 STM32F407VGTx, X1 STDCSU18M

Commit message: changuz
Connections:
- net VDD renamed 3V3
Other:
- moved on the sheet: C54, C55, C57, C58, FB5, R60
