File: FuseBox/USB_PWR.kicad_sch (KiCad schematic)
At the start: 54 parts, among them J1 UJ31CHG2SMTTR, U1 TPS61040DBVR, U2 LT3030EFETRPBF

Commit message: changes
Connections:
- net +12V: now also TP7.1; no longer R15.2, TP10.1
- net +1V2: now also TP5.1; no longer R17.2, TP8.1
- net +1V22: now also TP3.1; no longer TP5.1
- net +3V3: now also TP10.1; no longer TP7.1
- net +3V31: now also TP8.1; no longer TP4.1
- net +5V: now also TP2.1; no longer TP1.1
- net VBUS: now also TP1.1; no longer TP2.1
- net VCC_12V: now also TP6.1; no longer C2.1, TP9.1
- net VCC_1V2: now also TP4.1; no longer TP6.1
- net VCC_3V3: now also TP9.1; no longer C12.1, TP3.1
Other:
- note added: "Testpoints"
- note removed: "GND Testpoint"
- moved on the sheet: C5, C6, D2, FB2, R5, TP1

Commit message: changes
Connections:
- net USB_OTG_FS_DN renamed STM_USB_OTG_FS_DN
- net USB_OTG_FS_DP renamed STM_USB_OTG_FS_DP
Other:
- moved on the sheet: J1, R1, R2

Commit message: finished schematic
Parts:
- C1, C10, C11, C12, C13, C14, C2, C3, C5, C6, C7, C8, C9: footprint (none) -> Capacitor_SMD:C_0603_1608Metric_Pad1.08x0.95mm_HandSolder
- D2, D3, D4, D5: footprint (none) -> LED_SMD:LED_0603_1608Metric
- FB1, FB2, FB3, FB4, L1: footprint (none) -> Inductor_SMD:L_0603_1608Metric_Pad1.05x0.95mm_HandSolder
- R1, R10, R11, R12, R13, R14, R15, R16, R17, R2, R3, R4, R5, R6, R7, R8, R9: footprint (none) -> Resistor_SMD:R_0603_1608Metric_Pad0.98x0.95mm_HandSolder
Connections:
- net VCC_12V: now also C2.1
Changed lines of the file:
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@@
 	)
 	(junction
+		(at 222.25 41.91)
+		(diameter 0)
+		(color 0 0 0 0)
+	)
+	(junction
 		(at 215.9 111.76)
 		(diameter 0)
@@
 	(wire
 		(pts
+			(xy 222.25 41.91) (xy 222.25 43.18)
+		)
+		(stroke
+			(width 0)
+			(type default)
+		)
+	)
+	(wire
+		(pts
 			(xy 99.06 184.15) (xy 99.06 185.42)
 		)
@@
 	(wire
 		(pts
+			(xy 222.25 41.91) (xy 237.49 41.91)
+		)
+		(stroke
+			(width 0)
+			(type default)
+		)
+	)
+	(wire
+		(pts
 			(xy 140.97 102.87) (xy 140.97 101.6)
 		)
@@
 	(wire
 		(pts
-			(xy 210.82 41.91) (xy 237.49 41.91)
+			(xy 210.82 41.91) (xy 222.25 41.91)
 		)
 		(stroke
@@
 			)
 		)
-		(property "Footprint" ""
+		(property "Footprint" "Resistor_SMD:R_0603_1608Metric_Pad0.98x0.95mm_HandSolder"
 			(at 184.658 106.68 90)
 			(effects
@@
 			)
 		)
-		(property "Footprint" ""
+		(property "Footprint" "Resistor_SMD:R_0603_1608Metric_Pad0.98x0.95mm_HandSolder"
 			(at 184.658 128.27 90)
 			(effects
@@
 			)
 		)
-		(property "Footprint" ""
+		(property "Footprint" "Inductor_SMD:L_0603_1608Metric_Pad1.05x0.95mm_HandSolder"
 			(at 162.56 31.75 0)
 			(effects
@@
 			)
 		)
-		(property "Footprint" ""
+		(property "Footprint" "Resistor_SMD:R_0603_1608Metric_Pad0.98x0.95mm_HandSolder"
 			(at 263.398 46.99 90)
 			(effects
@@
 			)
 		)
-		(property "Footprint" ""
+		(property "Footprint" "Resistor_SMD:R_0603_1608Metric_Pad0.98x0.95mm_HandSolder"
 			(at 194.31 121.412 90)
 			(effects
@@
 			)
 		)
-		(property "Footprint" ""
+		(property "Footprint" "Resistor_SMD:R_0603_1608Metric_Pad0.98x0.95mm_HandSolder"
 			(at 16.002 53.34 90)
 			(effects
@@
 			)
 		)
-		(property "Footprint" ""
+		(property "Footprint" "Capacitor_SMD:C_0603_1608Metric_Pad1.08x0.95mm_HandSolder"
 			(at 238.4552 50.8 0)
 			(effects
@@
 			)
 		)
-		(property "Footprint" ""
+		(property "Footprint" "Capacitor_SMD:C_0603_1608Metric_Pad1.08x0.95mm_HandSolder"
 			(at 141.9352 110.49 0)
 			(effects
@@
 			)
 		)
-		(property "Footprint" ""
+		(property "Footprint" "Capacitor_SMD:C_0603_1608Metric_Pad1.08x0.95mm_HandSolder"
 			(at 136.8552 53.34 0)
 			(effects
@@
 			)
 		)
-		(property "Footprint" ""
+		(property "Footprint" "Resistor_SMD:R_0603_1608Metric_Pad0.98x0.95mm_HandSolder"
 			(at 253.238 128.27 90)
 			(effects
@@
 			)
 		)
-		(property "Footprint" ""
+		(property "Footprint" "LED_SMD:LED_0603_1608Metric"
 			(at 261.62 55.88 0)
 			(effects
@@
 			)
 		)
-		(property "Footprint" ""
+		(property "Footprint" "Capacitor_SMD:C_0603_1608Metric_Pad1.08x0.95mm_HandSolder"
 			(at 169.8752 110.49 0)
 			(effects
@@
 			)
 		)
-		(property "Footprint" ""
+		(property "Footprint" "Capacitor_SMD:C_0603_1608Metric_Pad1.08x0.95mm_HandSolder"
 			(at 141.9352 132.08 0)
 			(effects
@@
 			)
 		)
-		(property "Footprint" ""
+		(property "Footprint" "Capacitor_SMD:C_0603_1608Metric_Pad1.08x0.95mm_HandSolder"
 			(at 55.5752 113.03 0)
 			(effects
@@
 			)
 		)
-		(property "Footprint" ""
+		(property "Footprint" "Inductor_SMD:L_0603_1608Metric_Pad1.05x0.95mm_HandSolder"
 			(at 232.41 103.378 90)
 			(effects
@@
 			)
 		)
-		(property "Footprint" ""
+		(property "Footprint" "Resistor_SMD:R_0603_1608Metric_Pad0.98x0.95mm_HandSolder"
 			(at 161.29 109.982 90)
 			(effects
@@
 			)
 		)
-		(property "Footprint" ""
+		(property "Footprint" "Resistor_SMD:R_0603_1608Metric_Pad0.98x0.95mm_HandSolder"
 			(at 66.548 109.22 90)
 			(effects
@@
 			)
 		)
-		(property "Footprint" ""
+		(property "Footprint" "Inductor_SMD:L_0603_1608Metric_Pad1.05x0.95mm_HandSolder"
 			(at 45.72 164.338 90)
 			(effects
@@
 			)
 		)
-		(property "Footprint" ""
+		(property "Footprint" "Resistor_SMD:R_0603_1608Metric_Pad0.98x0.95mm_HandSolder"
 			(at 152.908 106.68 90)
 			(effects
@@
 			)
 		)
-		(property "Footprint" ""
+		(property "Footprint" "Capacitor_SMD:C_0603_1608Metric_Pad1.08x0.95mm_HandSolder"
 			(at 58.1152 171.45 0)
 			(effects
@@
 			)
 		)
-		(property "Footprint" ""
+		(property "Footprint" "Inductor_SMD:L_0603_1608Metric_Pad1.05x0.95mm_HandSolder"
 			(at 232.41 124.968 90)
 			(effects
@@
 			)
 		)
-		(property "Footprint" ""
+		(property "Footprint" "Inductor_SMD:L_0603_1608Metric_Pad1.05x0.95mm_HandSolder"
 			(at 251.46 43.688 90)
 			(effects
@@
 			)
 		)
-		(property "Footprint" ""
+		(property "Footprint" "Capacitor_SMD:C_0603_1608Metric_Pad1.08x0.95mm_HandSolder"
 			(at 216.8652 110.49 0)
 			(effects
@@
 			)
 		)
-		(property "Footprint" ""
+		(property "Footprint" "LED_SMD:LED_0603_1608Metric"
 			(at 251.46 137.16 0)
 			(effects
@@
 			)
 		)
-		(property "Footprint" ""
+		(property "Footprint" "Capacitor_SMD:C_0603_1608Metric_Pad1.08x0.95mm_HandSolder"
 			(at 152.0952 132.08 0)
 			(effects
@@
 			)
 		)
-		(property "Footprint" ""
+		(property "Footprint" "Capacitor_SMD:C_0603_1608Metric_Pad1.08x0.95mm_HandSolder"
 			(at 205.4352 110.49 0)
 			(effects
@@
 			)
 		)
-		(property "Footprint" ""
+		(property "Footprint" "Resistor_SMD:R_0603_1608Metric_Pad0.98x0.95mm_HandSolder"
 			(at 243.84 121.412 90)
 			(effects
@@
 			)
 		)
-		(property "Footprint" ""
+		(property "Footprint" "Resistor_SMD:R_0603_1608Metric_Pad0.98x0.95mm_HandSolder"
 			(at 71.628 167.64 90)
 			(effects
@@
 			)
 		)
-		(property "Footprint" ""
+		(property "Footprint" "Resistor_SMD:R_0603_1608Metric_Pad0.98x0.95mm_HandSolder"
 			(at 249.682 96.52 90)
 			(effects
@@
 			)
 		)
-		(property "Footprint" ""
+		(property "Footprint" "Capacitor_SMD:C_0603_1608Metric_Pad1.08x0.95mm_HandSolder"
 			(at 205.4352 132.08 0)
 			(effects
@@
 			)
 		)
-		(property "Footprint" ""
+		(property "Footprint" "Capacitor_SMD:C_0603_1608Metric_Pad1.08x0.95mm_HandSolder"
 			(at 223.2152 50.8 0)
 			(effects
@@
 			)
 		)
-		(property "Footprint" ""
+		(property "Footprint" "Resistor_SMD:R_0603_1608Metric_Pad0.98x0.95mm_HandSolder"
 			(at 209.042 46.99 90)
 			(effects
@@
 			)
 		)
-		(property "Footprint" ""
+		(property "Footprint" "Resistor_SMD:R_0603_1608Metric_Pad0.98x0.95mm_HandSolder"
 			(at 194.31 99.822 90)
 			(effects
@@
 			)
 		)
-		(property "Footprint" ""
+		(property "Footprint" "Resistor_SMD:R_0603_1608Metric_Pad0.98x0.95mm_HandSolder"
 			(at 111.252 48.26 90)
 			(effects
@@
 			)
 		)
-		(property "Footprint" ""
+		(property "Footprint" "LED_SMD:LED_0603_1608Metric"
 			(at 251.46 87.63 0)
 			(effects
@@
 			)
 		)
-		(property "Footprint" ""
+		(property "Footprint" "LED_SMD:LED_0603_1608Metric"
 			(at 69.85 176.53 0)
 			(effects
@@
 			)
 		)
-		(property "Footprint" ""
+		(property "Footprint" "Resistor_SMD:R_0603_1608Metric_Pad0.98x0.95mm_HandSolder"
 			(at 187.452 58.42 90)
 			(effects
@@
 			)
 		)
-		(property "Footprint" ""
+		(property "Footprint" "Capacitor_SMD:C_0603_1608Metric_Pad1.08x0.95mm_HandSolder"
 			(at 31.4452 171.45 0)
 			(effects
@@
 			)
 		)
-		(property "Footprint" ""
+		(property "Footprint" "Resistor_SMD:R_0603_1608Metric_Pad0.98x0.95mm_HandSolder"
 			(at 76.708 109.22 90)
 			(effects

Commit message: changes
Parts:
- TP1, TP10, TP11, TP2, TP3, TP4, TP5, TP6, TP7, TP8, TP9: footprint (none) -> TestPoint:TestPoint_Pad_D3.0mm
Changed lines of the file:
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@@
 			)
 		)
-		(property "Footprint" ""
+		(property "Footprint" "TestPoint:TestPoint_Pad_D3.0mm"
 			(at 104.14 162.56 0)
 			(effects
@@
 			)
 		)
-		(property "Footprint" ""
+		(property "Footprint" "TestPoint:TestPoint_Pad_D3.0mm"
 			(at 124.46 162.56 0)
 			(effects
@@
 			)
 		)
-		(property "Footprint" ""
+		(property "Footprint" "TestPoint:TestPoint_Pad_D3.0mm"
 			(at 144.78 162.56 0)
 			(effects
@@
 			)
 		)
-		(property "Footprint" ""
+		(property "Footprint" "TestPoint:TestPoint_Pad_D3.0mm"
 			(at 134.62 162.56 0)
 			(effects
@@
 			)
 		)
-		(property "Footprint" ""
+		(property "Footprint" "TestPoint:TestPoint_Pad_D3.0mm"
 			(at 104.14 184.15 0)
 			(effects
@@
 			)
 		)
-		(property "Footprint" ""
+		(property "Footprint" "TestPoint:TestPoint_Pad_D3.0mm"
 			(at 144.78 184.15 0)
 			(effects
@@
 			)
 		)
-		(property "Footprint" ""
+		(property "Footprint" "TestPoint:TestPoint_Pad_D3.0mm"
 			(at 124.46 184.15 0)
 			(effects
@@
 			)
 		)
-		(property "Footprint" ""
+		(property "Footprint" "TestPoint:TestPoint_Pad_D3.0mm"
 			(at 114.3 184.15 0)
 			(effects
@@
 			)
 		)
-		(property "Footprint" ""
+		(property "Footprint" "TestPoint:TestPoint_Pad_D3.0mm"
 			(at 158.75 173.99 0)
 			(effects
@@
 			)
 		)
-		(property "Footprint" ""
+		(property "Footprint" "TestPoint:TestPoint_Pad_D3.0mm"
 			(at 114.3 162.56 0)
 			(effects
@@
 			)
 		)
-		(property "Footprint" ""
+		(property "Footprint" "TestPoint:TestPoint_Pad_D3.0mm"
 			(at 134.62 184.15 0)
 			(effects

Commit message: layout
Connections:
- net +12V: now also R15.2
- net +1V2: now also R17.2
- net VCC_3V3: now also C12.1

Commit message: keeeek
Other:
- moved on the sheet: C10, C11, C12, C13, C14, C5, C6, C7, C8, C9, D2, D4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

Commit message: more kekw
Connections:
- net +1V22: now also U2.9 (BYP2); no longer U2.10 (ADJ2)
- net GND: now also U2.EPAD
- net at C9.2: now also U2.10 (ADJ2); no longer U2.9 (BYP2)
- no-connect marks 11 -> 10

Commit message: changuz
Parts:
- removed C10: 10u, Capacitor_SMD:C_0603_1608Metric_Pad1.08x0.95mm_HandSolder, symbol Device:C
- removed C11, C14: 22u, Capacitor_SMD:C_0603_1608Metric_Pad1.08x0.95mm_HandSolder, symbol Device:C
- removed C12: 100n, Capacitor_SMD:C_0603_1608Metric_Pad1.08x0.95mm_HandSolder, symbol Device:C
- removed C13: 4u7, Capacitor_SMD:C_0603_1608Metric_Pad1.08x0.95mm_HandSolder, symbol Device:C
- removed D1: CUS10S40H3F, Custom:CUS10S40H3F, symbol Custom:CUS10S40H3F
- removed D3, D5: LED, LED_SMD:LED_0603_1608Metric, symbol Device:LED
- removed FB1, FB4: 600R 500mA, Inductor_SMD:L_0603_1608Metric_Pad1.05x0.95mm_HandSolder, symbol Device:FerriteBead
- removed L1: 10u, Inductor_SMD:L_0603_1608Metric_Pad1.05x0.95mm_HandSolder, symbol Device:L
- removed R10, R12: 100, Resistor_SMD:R_0603_1608Metric_Pad0.98x0.95mm_HandSolder, symbol Device:R
- removed R11, R13: 100m, Resistor_SMD:R_0603_1608Metric_Pad0.98x0.95mm_HandSolder, symbol Device:R
- removed R14: 1, Resistor_SMD:R_0603_1608Metric_Pad0.98x0.95mm_HandSolder, symbol Device:R
- removed R15: 2k4, Resistor_SMD:R_0603_1608Metric_Pad0.98x0.95mm_HandSolder, symbol Device:R
- removed R17: 300, Resistor_SMD:R_0603_1608Metric_Pad0.98x0.95mm_HandSolder, symbol Device:R
- removed R9: 210k, Resistor_SMD:R_0603_1608Metric_Pad0.98x0.95mm_HandSolder, symbol Device:R
- removed TP10, TP11, TP7, TP8, TP9: TestPoint, TestPoint:TestPoint_Pad_D3.0mm, symbol Connector:TestPoint
- removed U1: TPS61040DBVR, Custom:TPS61040DBVR, symbol Custom:TPS61040DBVR
- removed U2: LT3030EFETRPBF, Custom:LT8302ES8ETRPBF, symbol Custom:LT3030EFETRPBF
- added D1: LED, LED_SMD:LED_0603_1608Metric, symbol Device:LED
- added FB2: 600R 500mA, Inductor_SMD:L_0603_1608Metric_Pad1.05x0.95mm_HandSolder, symbol Device:FerriteBead
- added J13, J14: 61300211121, Custom:61300211121, symbol Custom:61300211121
- added TP4: TestPoint, TestPoint:TestPoint_Pad_D3.0mm, symbol Connector:TestPoint
- added U1, U2: MAX8902BATA/V+T, Custom:MAX8902BATAVT, symbol Custom:MAX8902BATAVT
- C2: value 30p -> 10n
- C9: value 10n -> 10u
- R3: value 873k3 -> 120k
- R4: value 100k -> 540k
- R6, R7: value 1M -> 120k
- R8: value 357k -> 300
- renumbered D4 to D3, FB2 to FB1, R16 to R15, TP4 to TP7
Connections:
- net +1V2 is gone; now on net GND: TP5.1
- net +1V22 is gone; now on an unnamed net: C9.1, TP3.1
- net +3V31 is gone; now on an unnamed net: C8.1, R8.2
- net VCC_1V2 is gone; now on an unnamed net: TP7.1
- net VCC_3V3 is gone; now on an unnamed net: FB3.1
- net GND: now also C9.2, R7.2, D1.1 (K), U1.2 (GND), U1.4 (GS), U1.9 (EPAD), U2.2 (GND), U2.4 (GS), U2.9 (EPAD)
- net VBUS: now also FB2.1; no longer FB1.1
- net at C8.2: now also U2.7 (BYP)
- net at R3.2, R4.1: now also U1.6 (FB); no longer C2.2
- net at R8.1: now also D1.2 (A)
- net at R6.1: now also U2.8 (OUT)
- net at R7.1: now also R6.2, U2.6 (FB)
- net +3V3: no longer names the net of R15.2
- net +3V3: now also C2.1, C3.1, FB1.1, R3.1, U1.8 (OUT); no longer FB3.2
- net +5V renamed 5V
- net 5V: now also FB2.2, U1.1 (IN), U1.3 (EN), U2.1 (IN), U2.3 (EN); no longer FB1.2, R6.2, R7.2
- removed net VCC_12V: C2.1, C3.1, R3.1, TP6.1
- new net: FB1.2, J13.2, TP4.1
- new net: FB3.2, J14.2, TP6.1
- new net: C2.2, U1.7 (BYP)
- new net 1V2: J14.1
- new net 3V3: J13.1
- no-connect marks 10 -> 12
Other:
- note removed: "Boost Converter"
- note removed: "Testpoints"
- note removed: "V(out)=1.233V*(1+Rhi/Rlo)=12V"
- moved on the sheet: C5, C6, D2, D3, FB1, J1, R1, R15, R2, R5, TP1, TP5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
