File: FuseBox/ADC.kicad_sch (KiCad schematic)
At the start: 0 parts

Commit message: keeeek
Parts:
- added U15: OPA1612AIDRGR, Custom:OPA1612AIDRGR, symbol Custom:OPA1612AIDRGR
- added U56: PCM1803ADB, Custom:PCM1803ADB, symbol Custom:PCM1803ADB
Changed lines of the file:
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@@
 	(generator_version "9.0")
 	(paper "A4")
+	(symbol
+		(lib_id "Custom:OPA1612AIDRGR")
+		(at 53.34 44.45 0)
+		(unit 1)
+		(exclude_from_sim no)
+		(in_bom yes)
+		(on_board yes)
+		(dnp no)
+		(property "Reference" "U15"
+			(at 55.372 42.418 0)
+			(effects
+				(font
+					(size 1.524 1.524)
+				)
+			)
+		)
+		(property "Value" "OPA1612AIDRGR"
+			(at 62.23 61.722 0)
+			(effects
+				(font
+					(size 1.524 1.524)
+				)
+			)
+		)
+		(property "Footprint" "Custom:OPA1612AIDRGR"
+			(at 61.976 37.084 0)
+			(effects
+				(font
+					(size 1.27 1.27)
+					(italic yes)
+				)
+				(hide yes)
+			)
+		)
+		(property "Datasheet" "https://www.ti.com/lit/gpn/opa1612"
+			(at 61.468 39.878 0)
+			(effects
+				(font
+					(size 1.27 1.27)
+					(italic yes)
+				)
+				(hide yes)
+			)
+		)
+		(property "Description" ""
+			(at 53.34 44.45 0)
+			(effects
+				(font
+					(size 1.27 1.27)
+				)
+				(hide yes)
+			)
+		)
+		(pin "3"
+		)
+		(pin "1"
+		)
+		(pin "2"
+		)
+		(pin "8"
+		)
+		(pin "6"
+		)
+		(pin "5"
+		)
+		(pin "7"
+		)
+		(pin "4"
+		)
+		(pin "9"
+		)
+		(instances
+			(project ""
+				(path "/7cec0856-4a31-46c4-b6e3-cba19fcff38c/04957fa5-f37a-4410-94fa-538e764c5756"
+					(reference "U15")
+					(unit 1)
+				)
+			)
+		)
+	)
+	(symbol
+		(lib_id "Custom:PCM1803ADB")
+		(at 135.89 44.45 0)
+		(unit 1)
+		(exclude_from_sim no)
+		(in_bom yes)
+		(on_board yes)
+		(dnp no)
+		(property "Reference" "U56"
+			(at 138.43 42.672 0)
+			(effects
+				(font
+					(size 1.524 1.524)
+				)
+			)
+		)
+		(property "Value" "PCM1803ADB"
+			(at 143.51 97.79 0)
+			(effects
+				(font
+					(size 1.524 1.524)
+				)
+			)
+		)
+		(property "Footprint" "Custom:PCM1803ADB"
+			(at 149.86 35.56 0)
+			(effects
+				(font
+					(size 1.27 1.27)
+					(italic yes)
+				)
+				(hide yes)
+			)
+		)
+		(property "Datasheet" "https://www.ti.com/lit/gpn/pcm1803a"
+			(at 149.098 38.354 0)
+			(effects
+				(font
+					(size 1.27 1.27)
+					(italic yes)
+				)
+				(hide yes)
+			)
+		)
+		(property "Description" ""
+			(at 135.89 44.45 0)
+			(effects
+				(font
+					(size 1.27 1.27)
+				)
+				(hide yes)
+			)
+		)
+		(pin "5"
+		)
+		(pin "19"
+		)
+		(pin "16"
+		)
+		(pin "4"
+		)
+		(pin "9"
+		)
+		(pin "11"
+		)
+		(pin "12"
+		)
+		(pin "3"
+		)
+		(pin "6"
+		)
+		(pin "1"
+		)
+		(pin "15"
+		)
+		(pin "17"
+		)
+		(pin "18"
+		)
+		(pin "8"
+		)
+		(pin "13"
+		)
+		(pin "2"
+		)
+		(pin "10"
+		)
+		(pin "14"
+		)
+		(pin "7"
+		)
+		(pin "20"
+		)
+		(instances
+			(project ""
+				(path "/7cec0856-4a31-46c4-b6e3-cba19fcff38c/04957fa5-f37a-4410-94fa-538e764c5756"
+					(reference "U56")
+					(unit 1)
+				)
+			)
+		)
+	)
 )

Commit message: stupid analog
Parts:
- removed U56: PCM1803ADB, Custom:PCM1803ADB, symbol Custom:PCM1803ADB
- added C10, C11: 10n, Capacitor_SMD:C_0603_1608Metric_Pad1.08x0.95mm_HandSolder, symbol Device:C
- added C12, C13, C14, C62: 100n, Capacitor_SMD:C_0603_1608Metric_Pad1.08x0.95mm_HandSolder, symbol Device:C
- added J15: SJ63073E, Custom:SJ63073E, symbol Custom:SJ63073E
- added R10, R9: 100, Resistor_SMD:R_0603_1608Metric_Pad0.98x0.95mm_HandSolder, symbol Device:R
- added R11, R12: 1M, Resistor_SMD:R_0603_1608Metric_Pad0.98x0.95mm_HandSolder, symbol Device:R
- added U18: PCM1803ADB, Custom:PCM1803ADB, symbol Custom:PCM1803ADB
Connections:
- net AIN1_FB_R: now reaches U15.1 (OUTA)
- net AIN1_FB_R: now also U15.6 (-INB), R10.1
- net AIN1_FB_L: now reaches U15.2 (-INA)
- net AIN1_FB_L: now also U15.7 (OUTB), R9.1
- net at U15.3 (+INA): now also R11.2
- net GND: now reaches U15.4 (V-)
- net GND: now also U15.9 (EPAD), C10.1, C11.2, C12.2, C13.2, C14.2, C62.2, J15.1 (SLEEVE), U18.13 (DGND), U18.6 (AGND), U18.9 (TEST)
- net at U15.5 (+INB): now also R12.2
- net 5V: now reaches U15.8 (V+)
- net 5V: now also C14.1, U18.5 (VCC)
- new net: C10.2, R9.2, U18.1 (VINL)
- new net: C11.1, R10.2, U18.2 (VINR)
- new net: C12.1, U18.3 (VREF1)
- new net: C13.1, U18.4 (VREF2)
- new net: J15.3 (RING), R12.1
- new net: J15.2 (TIP), R11.1
- new net 3V3: C62.1, U18.14 (VDD)
- new net FPGA_AIN1_BCK: U18.11 (BCK)
- new net FPGA_AIN1_BYPAS: U18.8 (BYPAS)
- new net FPGA_AIN1_DOUT: U18.12 (DOUT)
- new net FPGA_AIN1_FMT0: U18.17 (FMT0)
- new net FPGA_AIN1_FMT1: U18.18 (FMT1)
- new net FPGA_AIN1_LRCK: U18.10 (LRCK)
- new net FPGA_AIN1_MODE0: U18.19 (MODE0)
- new net FPGA_AIN1_MODE1: U18.20 (MODE1)
- new net FPGA_AIN1_OSR: U18.16 (OSR)
- new net FPGA_AIN1_PDWN: U18.7 (PDWN_N)
- new net FPGA_AIN1_SCK: U18.15 (SCKI)
- no-connect marks 0 -> 3
